File: activity_monitor/board_v1.2/activity_monitor_v1.2.brd (EAGLE design)
At the start: 27.9 x 16.5 mm, 36 parts, among them U1 74HC04_HEX_INVERTERTSSOP14

Commit message: move some things around
Parts:
- U1: value 74HC04_HEX_INVERTERTSSOP14 -> (none)
Changed lines of the file:
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@@
 </autorouter>
 <elements>
-<element name="U1" library="kmod" package="TSSOP14" value="74HC04_HEX_INVERTERTSSOP14" x="13.97" y="11.43" rot="MR0"/>
+<element name="U1" library="kmod" package="TSSOP14" value="" x="13.97" y="11.43" rot="MR0"/>
 <element name="JP1" library="SparkFun-Connectors" package="1X08" value="" x="20.32" y="2.54" rot="R180"/>
 <element name="L0A" library="SparkFun-LED" package="LED-0603" value="" x="6.35" y="13.97" rot="R90"/>
