File: activity_monitor/board_v1.2/activity_monitor_v1.2.sch (EAGLE design)
At the start: 36 parts, among them U1 74HC04_HEX_INVERTERTSSOP14

Commit message: move some things around
Changed lines of the file:
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@@
 </classes>
 <parts>
-<part name="U1" library="kmod" deviceset="74HC04_HEX_INVERTER" device="TSSOP14"/>
+<part name="U1" library="kmod" deviceset="74HC04_HEX_INVERTER" device="TSSOP14" value=""/>
 <part name="JP1" library="SparkFun-Connectors" deviceset="M08" device="1X08"/>
 <part name="GND1" library="SparkFun-Aesthetics" deviceset="GND" device=""/>
