File: process_tester/v1/tester.brd (EAGLE design)
At the start: 21.3 x 15.2 mm, 37 parts, among them IC1 7408RGY, IC2 7404TSSOP14, IC3 7408RGY, IC4 7404D

Commit message: some fixes, filling in values
Parts:
- C1, C2: value (none) -> 10uF
- C10, C7, C8, C9: value (none) -> 100nF
- C3, C4, C5, C6: value (none) -> 1uF
- R1, R2, R3, R4, R5, R6, R7, R8, RA1, RA2: value (none) -> 1k
- R10, R9: value (none) -> 10k
Changed lines of the file:
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@@
 <setting verticaltext="up"/>
 </settings>
-<grid distance="0.05" unitdist="inch" unit="inch" style="lines" multiple="1" display="no" altdistance="0.01" altunitdist="inch" altunit="inch"/>
+<grid distance="0.5" unitdist="mm" unit="mm" style="lines" multiple="1" display="yes" altdistance="0.01" altunitdist="mm" altunit="mm"/>
 <layers>
 <layer number="1" name="Top" color="4" fill="1" visible="yes" active="yes"/>
@@
 <element name="CONN1" library="kmod" package="TESTPAD" value="" x="1.27" y="1.27"/>
 <element name="CONN2" library="kmod" package="TESTPAD" value="" x="6.604" y="10.16"/>
-<element name="RA1" library="kmod" package="0603-ARV" value="" x="4.064" y="2.032"/>
-<element name="RA2" library="kmod" package="0603-ARV" value="" x="4.318" y="4.318" rot="R180"/>
-<element name="R1" library="kmod" package="0603-RES" value="" x="1.27" y="7.62" rot="R270"/>
-<element name="R2" library="kmod" package="0603-RES" value="" x="2.54" y="7.62" rot="R270"/>
-<element name="R3" library="kmod" package="0603-RES" value="" x="3.81" y="7.62" rot="R270"/>
-<element name="R4" library="kmod" package="0603-RES" value="" x="5.08" y="7.62" rot="R270"/>
-<element name="R5" library="kmod" package="0402-RES" value="" x="1.27" y="10.795" rot="R270"/>
-<element name="R6" library="kmod" package="0402-RES" value="" x="2.54" y="10.795" rot="R270"/>
-<element name="R7" library="kmod" package="0402-RES" value="" x="3.81" y="10.795" rot="R270"/>
-<element name="R8" library="kmod" package="0402-RES" value="" x="5.08" y="10.795" rot="R270"/>
+<element name="RA1" library="kmod" package="0603-ARV" value="1k" x="4.064" y="2.032"/>
+<element name="RA2" library="kmod" package="0603-ARV" value="1k" x="4.318" y="4.318" rot="R180"/>
+<element name="R1" library="kmod" package="0603-RES" value="1k" x="1.27" y="7.62" rot="R270"/>
+<element name="R2" library="kmod" package="0603-RES" value="1k" x="2.54" y="7.62" rot="R270"/>
+<element name="R3" library="kmod" package="0603-RES" value="1k" x="3.81" y="7.62" rot="R270"/>
+<element name="R4" library="kmod" package="0603-RES" value="1k" x="5.08" y="7.62" rot="R270"/>
+<element name="R5" library="kmod" package="0402-RES" value="1k" x="1.27" y="10.795" rot="R270"/>
+<element name="R6" library="kmod" package="0402-RES" value="1k" x="2.54" y="10.795" rot="R270"/>
+<element name="R7" library="kmod" package="0402-RES" value="1k" x="3.81" y="10.795" rot="R270"/>
+<element name="R8" library="kmod" package="0402-RES" value="1k" x="5.08" y="10.795" rot="R270"/>
 <element name="CONN3" library="kmod" package="TESTPAD" value="" x="12.446" y="7.62"/>
-<element name="C1" library="kmod" package="EIA3216" value="" x="16.256" y="6.35" rot="R180"/>
-<element name="C2" library="kmod" package="EIA3216" value="" x="16.256" y="8.89"/>
-<element name="C3" library="SparkFun-Capacitors" package="0805" value="" x="12.7" y="11.43" rot="R270"/>
-<element name="C4" library="SparkFun-Capacitors" package="0805" value="" x="14.351" y="11.43" rot="R270"/>
-<element name="C5" library="SparkFun-Capacitors" package="0805" value="" x="16.002" y="11.43" rot="R270"/>
-<element name="C6" library="SparkFun-Capacitors" package="0805" value="" x="17.526" y="11.43" rot="R270"/>
-<element name="C7" library="SparkFun-Capacitors" package="0402-CAP" value="" x="10.414" y="9.652"/>
-<element name="C8" library="SparkFun-Capacitors" package="0402-CAP" value="" x="10.414" y="10.922"/>
-<element name="C9" library="SparkFun-Capacitors" package="0402-CAP" value="" x="10.414" y="12.192"/>
-<element name="C10" library="SparkFun-Capacitors" package="0402-CAP" value="" x="10.414" y="13.462"/>
+<element name="C1" library="kmod" package="EIA3216" value="10uF" x="16.256" y="6.35" rot="R180"/>
+<element name="C2" library="kmod" package="EIA3216" value="10uF" x="16.256" y="8.89"/>
+<element name="C3" library="SparkFun-Capacitors" package="0805" value="1uF" x="12.7" y="11.43" rot="R270"/>
+<element name="C4" library="SparkFun-Capacitors" package="0805" value="1uF" x="14.351" y="11.43" rot="R270"/>
+<element name="C5" library="SparkFun-Capacitors" package="0805" value="1uF" x="16.002" y="11.43" rot="R270"/>
+<element name="C6" library="SparkFun-Capacitors" package="0805" value="1uF" x="17.526" y="11.43" rot="R270"/>
+<element name="C7" library="SparkFun-Capacitors" package="0402-CAP" value="100nF" x="10.414" y="9.652"/>
+<element name="C8" library="SparkFun-Capacitors" package="0402-CAP" value="100nF" x="10.414" y="10.922"/>
+<element name="C9" library="SparkFun-Capacitors" package="0402-CAP" value="100nF" x="10.414" y="12.192"/>
+<element name="C10" library="SparkFun-Capacitors" package="0402-CAP" value="100nF" x="10.414" y="13.462"/>
 <element name="CONN4" library="kmod" package="TESTPAD" value="" x="13.208" y="13.97" rot="R270"/>
 <element name="JP1" library="SparkFun-Connectors" package="1X01" value="M01PTH" x="10.16" y="1.778"/>
@@
 <element name="IC4" library="kmod" package="SO14" value="7404D" x="14.224" y="10.16" rot="MR0"/>
 <element name="CONN5" library="kmod" package="TESTPAD" value="" x="1.778" y="5.08"/>
-<element name="R9" library="kmod" package="0402-RES" value="" x="8.89" y="7.62" rot="MR90"/>
+<element name="R9" library="kmod" package="0402-RES" value="10k" x="8.89" y="7.62" rot="MR90"/>
 <element name="CONN6" library="kmod" package="TESTPAD" value="" x="8.89" y="10.16" rot="MR0"/>
-<element name="R10" library="kmod" package="0402-RES" value="" x="20.066" y="11.43" rot="MR270"/>
+<element name="R10" library="kmod" package="0402-RES" value="10k" x="20.066" y="11.43" rot="MR270"/>
 <element name="CONN7" library="kmod" package="TESTPAD" value="" x="20.066" y="13.97" rot="MR0"/>
 </elements>
