File: process_tester/v1/tester.sch (EAGLE design)
At the start: 37 parts, among them IC1 7408RGY, IC2 7404TSSOP14, IC3 7408RGY, IC4 7404D

Commit message: some fixes, filling in values
Parts:
- C1, C2: value (none) -> 10uF
- C10, C7, C8, C9: value (none) -> 100nF
- C3, C4, C5, C6: value (none) -> 1uF
- R1, R2, R3, R4, R5, R6, R7, R8, RA1, RA2: value (none) -> 1k
- R10, R9: value (none) -> 10k
Changed lines of the file:
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@@
 <grid distance="0.1" unitdist="inch" unit="inch" style="lines" multiple="1" display="no" altdistance="0.01" altunitdist="inch" altunit="inch"/>
 <layers>
-<layer number="1" name="Top" color="4" fill="1" visible="yes" active="no"/>
-<layer number="16" name="Bottom" color="1" fill="1" visible="yes" active="no"/>
-<layer number="17" name="Pads" color="2" fill="1" visible="yes" active="no"/>
-<layer number="18" name="Vias" color="2" fill="1" visible="yes" active="no"/>
-<layer number="19" name="Unrouted" color="6" fill="1" visible="yes" active="no"/>
-<layer number="20" name="Dimension" color="15" fill="1" visible="yes" active="no"/>
-<layer number="21" name="tPlace" color="16" fill="1" visible="yes" active="no"/>
-<layer number="22" name="bPlace" color="14" fill="1" visible="yes" active="no"/>
-<layer number="23" name="tOrigins" color="15" fill="1" visible="yes" active="no"/>
-<layer number="24" name="bOrigins" color="15" fill="1" visible="yes" active="no"/>
-<layer number="25" name="tNames" color="7" fill="1" visible="yes" active="no"/>
-<layer number="26" name="bNames" color="7" fill="1" visible="yes" active="no"/>
-<layer number="27" name="tValues" color="7" fill="1" visible="yes" active="no"/>
-<layer number="28" name="bValues" color="7" fill="1" visible="yes" active="no"/>
+<layer number="1" name="Top" color="4" fill="1" visible="no" active="no"/>
+<layer number="16" name="Bottom" color="1" fill="1" visible="no" active="no"/>
+<layer number="17" name="Pads" color="2" fill="1" visible="no" active="no"/>
+<layer number="18" name="Vias" color="2" fill="1" visible="no" active="no"/>
+<layer number="19" name="Unrouted" color="6" fill="1" visible="no" active="no"/>
+<layer number="20" name="Dimension" color="15" fill="1" visible="no" active="no"/>
+<layer number="21" name="tPlace" color="16" fill="1" visible="no" active="no"/>
+<layer number="22" name="bPlace" color="14" fill="1" visible="no" active="no"/>
+<layer number="23" name="tOrigins" color="15" fill="1" visible="no" active="no"/>
+<layer number="24" name="bOrigins" color="15" fill="1" visible="no" active="no"/>
+<layer number="25" name="tNames" color="7" fill="1" visible="no" active="no"/>
+<layer number="26" name="bNames" color="7" fill="1" visible="no" active="no"/>
+<layer number="27" name="tValues" color="7" fill="1" visible="no" active="no"/>
+<layer number="28" name="bValues" color="7" fill="1" visible="no" active="no"/>
 <layer number="29" name="tStop" color="7" fill="3" visible="no" active="no"/>
 <layer number="30" name="bStop" color="7" fill="6" visible="no" active="no"/>
@@
 <layer number="35" name="tGlue" color="7" fill="4" visible="no" active="no"/>
 <layer number="36" name="bGlue" color="7" fill="5" visible="no" active="no"/>
-<layer number="37" name="tTest" color="7" fill="1" visible="yes" active="no"/>
-<layer number="38" name="bTest" color="7" fill="1" visible="yes" active="no"/>
+<layer number="37" name="tTest" color="7" fill="1" visible="no" active="no"/>
+<layer number="38" name="bTest" color="7" fill="1" visible="no" active="no"/>
 <layer number="39" name="tKeepout" color="4" fill="11" visible="no" active="no"/>
 <layer number="40" name="bKeepout" color="1" fill="11" visible="no" active="no"/>
@@
 <layer number="44" name="Drills" color="7" fill="1" visible="no" active="no"/>
 <layer number="45" name="Holes" color="7" fill="1" visible="no" active="no"/>
-<layer number="46" name="Milling" color="3" fill="1" visible="yes" active="no"/>
-<layer number="47" name="Measures" color="7" fill="1" visible="yes" active="no"/>
-<layer number="48" name="Document" color="7" fill="1" visible="yes" active="no"/>
-<layer number="49" name="Reference" color="7" fill="1" visible="yes" active="no"/>
-<layer number="50" name="dxf" color="7" fill="1" visible="yes" active="no"/>
-<layer number="51" name="tDocu" color="6" fill="1" visible="yes" active="no"/>
-<layer number="52" name="bDocu" color="7" fill="1" visible="yes" active="no"/>
-<layer number="53" name="tGND_GNDA" color="7" fill="9" visible="yes" active="no"/>
-<layer number="54" name="bGND_GNDA" color="1" fill="9" visible="yes" active="no"/>
-<layer number="56" name="wert" color="7" fill="1" visible="yes" active="no"/>
+<layer number="46" name="Milling" color="3" fill="1" visible="no" active="no"/>
+<layer number="47" name="Measures" color="7" fill="1" visible="no" active="no"/>
+<layer number="48" name="Document" color="7" fill="1" visible="no" active="no"/>
+<layer number="49" name="Reference" color="7" fill="1" visible="no" active="no"/>
+<layer number="50" name="dxf" color="7" fill="1" visible="no" active="no"/>
+<layer number="51" name="tDocu" color="6" fill="1" visible="no" active="no"/>
+<layer number="52" name="bDocu" color="7" fill="1" visible="no" active="no"/>
+<layer number="53" name="tGND_GNDA" color="7" fill="9" visible="no" active="no"/>
+<layer number="54" name="bGND_GNDA" color="1" fill="9" visible="no" active="no"/>
+<layer number="56" name="wert" color="7" fill="1" visible="no" active="no"/>
 <layer number="91" name="Nets" color="2" fill="1" visible="yes" active="yes"/>
 <layer number="92" name="Busses" color="1" fill="1" visible="yes" active="yes"/>
@@
 <part name="CONN1" library="kmod" deviceset="CONNECTOR" device=""/>
 <part name="CONN2" library="kmod" deviceset="CONNECTOR" device=""/>
-<part name="RA1" library="kmod" deviceset="RESISTOR_ARRAY" device="0603_X4"/>
-<part name="RA2" library="kmod" deviceset="RESISTOR_ARRAY" device="0603_X4"/>
-<part name="R1" library="kmod" deviceset="RESISTOR" device="0603"/>
-<part name="R2" library="kmod" deviceset="RESISTOR" device="0603"/>
-<part name="R3" library="kmod" deviceset="RESISTOR" device="0603"/>
-<part name="R4" library="kmod" deviceset="RESISTOR" device="0603"/>
-<part name="R5" library="kmod" deviceset="RESISTOR" device="0402"/>
-<part name="R6" library="kmod" deviceset="RESISTOR" device="0402"/>
-<part name="R7" library="kmod" deviceset="RESISTOR" device="0402"/>
-<part name="R8" library="kmod" deviceset="RESISTOR" device="0402"/>
+<part name="RA1" library="kmod" deviceset="RESISTOR_ARRAY" device="0603_X4" value="1k"/>
+<part name="RA2" library="kmod" deviceset="RESISTOR_ARRAY" device="0603_X4" value="1k"/>
+<part name="R1" library="kmod" deviceset="RESISTOR" device="0603" value="1k"/>
+<part name="R2" library="kmod" deviceset="RESISTOR" device="0603" value="1k"/>
+<part name="R3" library="kmod" deviceset="RESISTOR" device="0603" value="1k"/>
+<part name="R4" library="kmod" deviceset="RESISTOR" device="0603" value="1k"/>
+<part name="R5" library="kmod" deviceset="RESISTOR" device="0402" value="1k"/>
+<part name="R6" library="kmod" deviceset="RESISTOR" device="0402" value="1k"/>
+<part name="R7" library="kmod" deviceset="RESISTOR" device="0402" value="1k"/>
+<part name="R8" library="kmod" deviceset="RESISTOR" device="0402" value="1k"/>
 <part name="CONN3" library="kmod" deviceset="CONNECTOR" device=""/>
-<part name="C1" library="kmod" deviceset="CAP_POL" device="1206"/>
-<part name="C2" library="kmod" deviceset="CAP_POL" device="1206"/>
-<part name="C3" library="SparkFun-Capacitors" deviceset="CAP" device="0805"/>
-<part name="C4" library="SparkFun-Capacitors" deviceset="CAP" device="0805"/>
-<part name="C5" library="SparkFun-Capacitors" deviceset="CAP" device="0805"/>
-<part name="C6" library="SparkFun-Capacitors" deviceset="CAP" device="0805"/>
-<part name="C7" library="SparkFun-Capacitors" deviceset="CAP" device="0402-CAP"/>
-<part name="C8" library="SparkFun-Capacitors" deviceset="CAP" device="0402-CAP"/>
-<part name="C9" library="SparkFun-Capacitors" deviceset="CAP" device="0402-CAP"/>
-<part name="C10" library="SparkFun-Capacitors" deviceset="CAP" device="0402-CAP"/>
+<part name="C1" library="kmod" deviceset="CAP_POL" device="1206" value="10uF"/>
+<part name="C2" library="kmod" deviceset="CAP_POL" device="1206" value="10uF"/>
+<part name="C3" library="SparkFun-Capacitors" deviceset="CAP" device="0805" value="1uF"/>
+<part name="C4" library="SparkFun-Capacitors" deviceset="CAP" device="0805" value="1uF"/>
+<part name="C5" library="SparkFun-Capacitors" deviceset="CAP" device="0805" value="1uF"/>
+<part name="C6" library="SparkFun-Capacitors" deviceset="CAP" device="0805" value="1uF"/>
+<part name="C7" library="SparkFun-Capacitors" deviceset="CAP" device="0402-CAP" value="100nF"/>
+<part name="C8" library="SparkFun-Capacitors" deviceset="CAP" device="0402-CAP" value="100nF"/>
+<part name="C9" library="SparkFun-Capacitors" deviceset="CAP" device="0402-CAP" value="100nF"/>
+<part name="C10" library="SparkFun-Capacitors" deviceset="CAP" device="0402-CAP" value="100nF"/>
 <part name="CONN4" library="kmod" deviceset="CONNECTOR" device=""/>
 <part name="JP1" library="SparkFun-Connectors" deviceset="M01" device="PTH"/>
@@
 <part name="IC4" library="kmod" deviceset="74*04" device="D" value="7404D"/>
 <part name="CONN5" library="kmod" deviceset="CONNECTOR" device=""/>
-<part name="R9" library="kmod" deviceset="RESISTOR" device="0402"/>
+<part name="R9" library="kmod" deviceset="RESISTOR" device="0402" value="10k"/>
 <part name="CONN6" library="kmod" deviceset="CONNECTOR" device=""/>
-<part name="R10" library="kmod" deviceset="RESISTOR" device="0402"/>
+<part name="R10" library="kmod" deviceset="RESISTOR" device="0402" value="10k"/>
 <part name="CONN7" library="kmod" deviceset="CONNECTOR" device=""/>
 </parts>
