File: copter/controller/board_v1/controller.brd (EAGLE design)
At the start: 45.5 x 45.5 mm, 69 parts, among them Q8 FA-238, U1 ATMEGA168MLF, U2 AAT3221

Commit message: controller changes
Parts:
- LPWR: value RED -> YLW
- R17: value 33k -> 47k
Changed lines of the file:
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@@
 <setting verticaltext="up"/>
 </settings>
-<grid distance="0.166666666667" unitdist="mm" unit="mm" style="lines" multiple="1" display="yes" altdistance="0.01" altunitdist="mil" altunit="mil"/>
+<grid distance="0.5" unitdist="mm" unit="mm" style="lines" multiple="1" display="yes" altdistance="0.01" altunitdist="mm" altunit="mm"/>
 <layers>
 <layer number="1" name="Top" color="4" fill="1" visible="yes" active="yes"/>
@@
 <element name="C9" library="kmod" package="0805" value="10uF" x="28.70985" y="25.957075" rot="R90"/>
 <element name="R14" library="SparkFun-Resistors" package="0603-RES" value="330" x="15.666665625" y="3.333334375" rot="R90"/>
-<element name="LPWR" library="SparkFun-LED" package="LED-0603" value="RED" x="17.333334375" y="3.333334375">
+<element name="LPWR" library="SparkFun-LED" package="LED-0603" value="YLW" x="17.333334375" y="3.333334375">
 <attribute name="PROD_ID" value="DIO-00819" x="59.243334375" y="-65.246665625" size="1.778" layer="27" display="off"/>
 </element>
@@
 <element name="CONN2" library="kmod" package="HOLE_18AWG" value="" x="8" y="2.5"/>
 <element name="CONN3" library="kmod" package="HOLE_18AWG" value="" x="12.5" y="2.5"/>
-<element name="R17" library="kmod" package="0603-RES" value="33k" x="15.436665625" y="12.6466625" rot="R270"/>
+<element name="R17" library="kmod" package="0603-RES" value="47k" x="15.436665625" y="12.6466625" rot="R270"/>
 <element name="R18" library="kmod" package="0603-RES" value="10k" x="15.43666875" y="15.79" rot="R270"/>
 <element name="JP3" library="SparkFun-Connectors" package="1X06" value="" x="43.18" y="7.921665625" rot="R90"/>
