File: modboard/v0.1/board.brd (EAGLE design)
At the start: 100 x 80 mm, 4 parts

Commit message: modboard in progress
Parts:
- removed C0: PCIE-X1EDGE, kmod:PCIE-X1-EDGE
- removed C1, C2, C3: PCIE-X1CONN, kmod:PCIE-X1-CONN
- added C10, C11, C9: PCIE-X1CONN, kmod-connectors:PCIE-X1-CONN
- added C4, C5: 100nF, kmod-passives:0402-CAP
- added C6, C7: 10uF, kmod-passives:0805
- added C8: PCIE-X1EDGE, kmod-connectors:PCIE-X1-EDGE
- added G4, G5, G6, G7: (no value), kmod-testing:SOT363
- added L0, L1, L2, L3: GREEN, kmod-passives:0603_LED
- added R1, R2, R3, R4: 10k, kmod-passives:0603-RES
- added R5, R6, R7, R8: 330, kmod-passives:0603-RES
- added U$1: XC2C{64,128,256}A-VQ100, kmod-xilinx:XILINX_TQ100
Connections:
- removed net G0: C0.B5, C1.B5, C2.B5, C3.B5
- removed net G1: C0.B6, C1.B6, C2.B6, C3.B6
- removed net G2: C0.B7, C1.B7, C2.B7, C3.B7
- removed net G3: C0.B9, C1.B9, C2.B9, C3.B9
- removed net G4: C0.B10, C1.B10, C2.B10, C3.B10
- removed net G5: C0.B11, C1.B11, C2.B11, C3.B11
- removed net N$1: C0.A11
- removed net N$19: C1.A11, C2.B18
- removed net N$2: C0.A10
- removed net N$20: C1.A10, C2.B17
- removed net N$21: C1.A9, C2.B16
- removed net N$22: C1.A7, C2.B14
- removed net N$23: C1.A6, C2.B13
- removed net N$24: C1.A5, C2.B12
- removed net N$25: C1.A18
- removed net N$26: C1.A17
- removed net N$27: C1.A16
- removed net N$28: C1.A14
- removed net N$29: C1.A13
- removed net N$30: C1.A12
- removed net N$31: C0.A18
- removed net N$32: C0.A17
- removed net N$33: C0.A16
- removed net N$34: C0.A14
- removed net N$35: C0.A13
- removed net N$36: C0.A12
- removed net N$37: C2.A11, C3.B18
- removed net N$38: C2.A10, C3.B17
- removed net N$39: C2.A9, C3.B16
- removed net N$4: C0.A7
- removed net N$40: C2.A7, C3.B14
- removed net N$41: C2.A6, C3.B13
- removed net N$42: C2.A5, C3.B12
- removed net N$5: C0.A6
- removed net N$55: C2.A18
- removed net N$56: C2.A17
- removed net N$57: C2.A16
- removed net N$58: C2.A14
- removed net N$59: C2.A13
- removed net N$6: C0.A5
- removed net N$60: C2.A12
- removed net N$61: C3.A18
- removed net N$62: C3.A17
- removed net N$63: C3.A16
- removed net N$64: C3.A14
- removed net N$65: C3.A13
- removed net N$66: C3.A12
- removed net N$67: C1.B18
- removed net N$68: C1.B17
- removed net N$69: C1.B16
- removed net N$70: C1.B14
- removed net N$71: C1.B13
- removed net N$72: C1.B12
- removed net R30: C0.B12, C3.A5
- removed net R31: C0.B13, C3.A6
- removed net R32: C0.B14, C3.A7
- removed net R33: C0.B16, C3.A9
- removed net R34: C0.B17, C3.A10
- removed net R35: C0.B18, C3.A11
- removed net SCL: C0.B2, C1.B2, C2.B2, C3.B2
- removed net SDA: C0.B3, C1.B3, C2.B3, C3.B3
- new net 0A0: U$1.22
- new net 0A1: U$1.23
- new net 0A2: U$1.24
- new net 0A3: U$1.27
- new net 0B0: U$1.28
- new net 0B1: U$1.29
- new net 0B2: U$1.30
- new net 0B3: U$1.32
- new net 0C0: U$1.33
- new net 0C1: U$1.34
- new net 0C2: U$1.35
- new net 0C3: U$1.36
- new net 0D0: U$1.37
- new net 0D1: U$1.39
- new net 0D2: U$1.40
- new net 0D3: U$1.41
- new net 0E0: U$1.42
- new net 0E1: U$1.43
- new net 0E2: U$1.49
- new net 0E3: U$1.50
- new net 1.8V: C5.1, C7.1, U$1.26, U$1.57
- new net 1A0: U$1.97
- new net 1A1: U$1.99
- new net 1A2: U$1.1
- new net 1A3: U$1.2
- new net 1B0: U$1.3
- new net 1B1: U$1.4
- new net 1B2: U$1.6
- new net 1B3: U$1.7
- new net 1C0: U$1.8
- new net 1C1: U$1.9
- new net 1C2: U$1.10
- new net 1C3: U$1.11
- new net 1D0: U$1.12
- new net 1D1: U$1.13
- new net 1D2: U$1.14
- new net 1D3: U$1.15
- new net 1E0: U$1.16
- new net 1E1: U$1.17
- new net 1E2: U$1.18
- new net 1E3: U$1.19
- new net 2A0: U$1.72
- new net 2A1: U$1.74
- new net 2A2: U$1.76
- new net 2A3: U$1.77
- new net 2B0: U$1.78
- new net 2B1: U$1.79
- new net 2B2: U$1.81
- new net 2B3: U$1.89
- new net 2C0: U$1.90
- new net 2C1: U$1.91
- new net 2C2: U$1.92
- new net 2C3: U$1.94
- new net 2D0: U$1.80
- new net 2D1: U$1.82
- new net 2D2: U$1.85
- new net 2D3: U$1.86
- new net 2E0: U$1.87
- new net 2E1: U$1.93
- new net 2E2: U$1.95
- new net 2E3: U$1.96
- new net 3.3V: C4.1, C6.1, G4.5, G5.5, G6.5, G7.5, R1.2, R2.2, R3.2, R4.2, R5.1, R6.1, R7.1, R8.1, U$1.20, U$1.38, U$1.5, U$1.51, U$1.88, U$1.98
- new net 3A0: U$1.52
- new net 3A1: U$1.53
- new net 3A2: U$1.55
- new net 3A3: U$1.56
- new net 3B0: U$1.58
- new net 3B1: U$1.60
- new net 3B2: U$1.61
- new net 3B3: U$1.64
- new net 3C0: U$1.67
- new net 3C1: U$1.68
- new net 3C2: U$1.70
- new net 3C3: U$1.71
- new net 3D0: U$1.44
- new net 3D1: U$1.46
- new net 3D2: U$1.54
- new net 3D3: U$1.59
- new net 3E0: U$1.63
- new net 3E1: U$1.65
- new net 3E2: U$1.66
- new net 3E3: U$1.73
- new net GND: C4.2, C5.2, C6.2, C7.2, G4.2, G5.2, G6.2, G7.2, U$1.100, U$1.21, U$1.25, U$1.31, U$1.62, U$1.69, U$1.75, U$1.84
- new net N$7: L1.A, R6.2
- new net N$8: L2.A, R7.2
- new net N$9: L3.A, R8.2
- new net SENSE0: G4.6, L0.C, R1.1
- new net SENSE1: G5.6, L1.C, R2.1
- new net SENSE2: G6.6, L2.C, R3.1
- new net SENSE3: G7.6, L3.C, R4.1
- new net TDI0/TDOC: G4.1, U$1.83
- new net TDI1: G4.4, G5.1
- new net TDI2: G5.4, G6.1
- new net TDI3: G6.4, G7.1
- new net TDIC: G7.4, U$1.45
- net N$3: now also L0.A, R5.2; no longer C0.A9
- net TCK: now also U$1.48; no longer C0.A3, C1.A3, C2.A3, C3.A3
- net TDO0: now also G4.3; no longer C0.A1, C1.B1
- net TDO1: now also G5.3; no longer C1.A1, C2.B1
- net TDO2: now also G6.3; no longer C2.A1, C3.B1
- net TDO3: now also G7.3; no longer C0.B1, C3.A1
- net TMS: now also U$1.47; no longer C0.A2, C1.A2, C2.A2, C3.A2
Other:
- board size 100 x 80 mm -> 50 x 42 mm
- board text added: "CR2: 64 128 256"
- board text added: "Modboard Backplane-R v1.0 (MB v1.0) 10-6-13"
- board text added: "Serial"
