File: modboard/v0.1/board.sch (EAGLE design)
At the start: 4 parts

Commit message: modboard in progress
Parts:
- removed C0: PCIE-X1EDGE, kmod:PCIE-X1EDGE
- removed C1, C2, C3: PCIE-X1CONN, kmod:PCIE-X1CONN
- added C10, C11, C9: PCIE-X1CONN, kmod-connectors:PCIE-X1CONN
- added C4, C5: 100nF, kmod-passives:CAP0402-CAP
- added C6, C7: 10uF, kmod-passives:CAP0805
- added C8: PCIE-X1EDGE, kmod-connectors:PCIE-X1EDGE
- added G4, G5, G6, G7: (no value), kmod-testing:74G157
- added L0, L1, L2, L3: GREEN, kmod-passives:LED0603
- added R1, R2, R3, R4: 10k, kmod-passives:RESISTOR0603
- added R5, R6, R7, R8: 330, kmod-passives:RESISTOR0603
- added U$1: XC2C{64,128,256}A-VQ100, kmod-xilinx:XC2C{64,128,256}A-VQ100
Connections:
- removed net G0: C0.B5, C1.B5, C2.B5, C3.B5
- removed net G1: C0.B6, C1.B6, C2.B6, C3.B6
- removed net G2: C0.B7, C1.B7, C2.B7, C3.B7
- removed net G3: C0.B9, C1.B9, C2.B9, C3.B9
- removed net G4: C0.B10, C1.B10, C2.B10, C3.B10
- removed net G5: C0.B11, C1.B11, C2.B11, C3.B11
- removed net N$1: C0.A11
- removed net N$19: C1.A11, C2.B18
- removed net N$2: C0.A10
- removed net N$20: C1.A10, C2.B17
- removed net N$21: C1.A9, C2.B16
- removed net N$22: C1.A7, C2.B14
- removed net N$23: C1.A6, C2.B13
- removed net N$24: C1.A5, C2.B12
- removed net N$25: C1.A18
- removed net N$26: C1.A17
- removed net N$27: C1.A16
- removed net N$28: C1.A14
- removed net N$29: C1.A13
- removed net N$30: C1.A12
- removed net N$31: C0.A18
- removed net N$32: C0.A17
- removed net N$33: C0.A16
- removed net N$34: C0.A14
- removed net N$35: C0.A13
- removed net N$36: C0.A12
- removed net N$37: C2.A11, C3.B18
- removed net N$38: C2.A10, C3.B17
- removed net N$39: C2.A9, C3.B16
- removed net N$4: C0.A7
- removed net N$40: C2.A7, C3.B14
- removed net N$41: C2.A6, C3.B13
- removed net N$42: C2.A5, C3.B12
- removed net N$5: C0.A6
- removed net N$55: C2.A18
- removed net N$56: C2.A17
- removed net N$57: C2.A16
- removed net N$58: C2.A14
- removed net N$59: C2.A13
- removed net N$6: C0.A5
- removed net N$60: C2.A12
- removed net N$61: C3.A18
- removed net N$62: C3.A17
- removed net N$63: C3.A16
- removed net N$64: C3.A14
- removed net N$65: C3.A13
- removed net N$66: C3.A12
- removed net N$67: C1.B18
- removed net N$68: C1.B17
- removed net N$69: C1.B16
- removed net N$70: C1.B14
- removed net N$71: C1.B13
- removed net N$72: C1.B12
- removed net R30: C0.B12, C3.A5
- removed net R31: C0.B13, C3.A6
- removed net R32: C0.B14, C3.A7
- removed net R33: C0.B16, C3.A9
- removed net R34: C0.B17, C3.A10
- removed net R35: C0.B18, C3.A11
- removed net SCL: C0.B2, C1.B2, C2.B2, C3.B2
- removed net SDA: C0.B3, C1.B3, C2.B3, C3.B3
- new net 0A0: U$1.P22/GCK0
- new net 0A1: U$1.P23/GCK1
- new net 0A2: U$1.P24/CDRST
- new net 0A3: U$1.P27/GCK2
- new net 0B0: U$1.P28/DGE
- new net 0B1: U$1.P29
- new net 0B2: U$1.P30
- new net 0B3: U$1.P32
- new net 0C0: U$1.P33
- new net 0C1: U$1.P34
- new net 0C2: U$1.P35
- new net 0C3: U$1.P36
- new net 0D0: U$1.P37
- new net 0D1: U$1.P39
- new net 0D2: U$1.P40
- new net 0D3: U$1.P41
- new net 0E0: U$1.P42
- new net 0E1: U$1.P43
- new net 0E2: U$1.P49
- new net 0E3: U$1.P50
- new net 1.8V: C5.1, C7.1, U$1.VCC
- new net 1A0: U$1.P97
- new net 1A1: U$1.P99/GSR
- new net 1A2: U$1.P1/GTS2
- new net 1A3: U$1.P2/GTS3
- new net 1B0: U$1.P3/GTS0
- new net 1B1: U$1.P4/GTS1
- new net 1B2: U$1.P6
- new net 1B3: U$1.P7
- new net 1C0: U$1.P8
- new net 1C1: U$1.P9
- new net 1C2: U$1.P10
- new net 1C3: U$1.P11
- new net 1D0: U$1.P12
- new net 1D1: U$1.P13
- new net 1D2: U$1.P14
- new net 1D3: U$1.P15
- new net 1E0: U$1.P16
- new net 1E1: U$1.P17
- new net 1E2: U$1.P18
- new net 1E3: U$1.P19
- new net 2A0: U$1.P72
- new net 2A1: U$1.P74
- new net 2A2: U$1.P76
- new net 2A3: U$1.P77
- new net 2B0: U$1.P78
- new net 2B1: U$1.P79
- new net 2B2: U$1.P81
- new net 2B3: U$1.P89
- new net 2C0: U$1.P90
- new net 2C1: U$1.P91
- new net 2C2: U$1.P92
- new net 2C3: U$1.P94
- new net 2D0: U$1.P80/NC
- new net 2D1: U$1.P82/NC
- new net 2D2: U$1.P85/NC
- new net 2D3: U$1.P86/NC
- new net 2E0: U$1.P87/NC
- new net 2E1: U$1.P93/NC
- new net 2E2: U$1.P95/NC
- new net 2E3: U$1.P96/NC
- new net 3.3V: C4.1, C6.1, G4G$2.VCC, G5G$2.VCC, G6G$2.VCC, G7G$2.VCC, R1.2, R2.2, R3.2, R4.2, R5.1, R6.1, R7.1, R8.1, U$1.VAUX, U$1.VCCIO1, U$1.VCCIO2
- new net 3A0: U$1.P52
- new net 3A1: U$1.P53
- new net 3A2: U$1.P55
- new net 3A3: U$1.P56
- new net 3B0: U$1.P58
- new net 3B1: U$1.P60
- new net 3B2: U$1.P61
- new net 3B3: U$1.P64
- new net 3C0: U$1.P67
- new net 3C1: U$1.P68
- new net 3C2: U$1.P70
- new net 3C3: U$1.P71
- new net 3D0: U$1.P44/NC
- new net 3D1: U$1.P46/NC
- new net 3D2: U$1.P54/NC
- new net 3D3: U$1.P59/NC
- new net 3E0: U$1.P63/NC
- new net 3E1: U$1.P65/NC
- new net 3E2: U$1.P66/NC
- new net 3E3: U$1.P73/NC
- new net GND: C4.2, C5.2, C6.2, C7.2, G4G$2.GND, G5G$2.GND, G6G$2.GND, G7G$2.GND, U$1.GND
- new net N$7: L1.A, R6.2
- new net N$8: L2.A, R7.2
- new net N$9: L3.A, R8.2
- new net SENSE0: G4G$1.S, L0.C, R1.1
- new net SENSE1: G5G$1.S, L1.C, R2.1
- new net SENSE2: G6G$1.S, L2.C, R3.1
- new net SENSE3: G7G$1.S, L3.C, R4.1
- new net TDI0/TDOC: G4G$1.I1, U$1.TDO
- new net TDI1: G4G$1.Y, G5G$1.I1
- new net TDI2: G5G$1.Y, G6G$1.I1
- new net TDI3: G6G$1.Y, G7G$1.I1
- new net TDIC: G7G$1.Y, U$1.TDI
- net N$3: now also L0.A, R5.2; no longer C0.A9
- net TCK: now also U$1.TCK; no longer C0.A3, C1.A3, C2.A3, C3.A3
- net TDO0: now also G4G$1.I0; no longer C0.A1, C1.B1
- net TDO1: now also G5G$1.I0; no longer C1.A1, C2.B1
- net TDO2: now also G6G$1.I0; no longer C2.A1, C3.B1
- net TDO3: now also G7G$1.I0; no longer C0.B1, C3.A1
- net TMS: now also U$1.TMS; no longer C0.A2, C1.A2, C2.A2, C3.A2
Other:
- note added: "(SENSE)"
