File: modboard/ioboard_v1.0/board.sch (EAGLE design)
At the start: 20 parts, among them J2 POWER_JACKPTH

Commit message: finished the base modboards
Parts:
- removed CONN1, CONN2: (no value), kmod-nonparts:CONNECTOR18AWG
- removed J2: POWER_JACKPTH, SparkFun-Connectors:POWER_JACKPTH
- removed L5: YLW, kmod-passives:LED0603
- removed R1: 2.2k, kmod-passives:RESISTOR0603
- added C1: 100nF, kmod-passives:CAP0402-CAP
- added L10, L7, L8, L9: (no value), kmod-passives:LED0603
- added RA2, RA3: 10k, kmod-passives:RESISTOR_ARRAY0603_X4
- added RA6: 220, kmod-passives:RESISTOR_ARRAY0603_X4
- renumbered L6 to L3V3
Connections:
- removed net 12V: CONN1.P, J2.GNDBREAK, L5.A, U$1.12V@1, U$1.12V@2
- removed net N$1: L5.C, R1.2
- removed net N$10: JP2.2
- removed net N$9: JP2.3
- new net A0: L4.A, U$1.A0
- new net A1: L3.A, U$1.A1
- new net A2: L2.A, U$1.A2
- new net A3: L1.A, U$1.A3
- new net B0: RA2B.2, S3.2, SW1.6, U$1.B0
- new net B1: RA2C.2, S2.2, SW1.7, U$1.B1
- new net B2: RA2D.2, S1.2, SW1.8, U$1.B2
- new net B3: C1.2, U$1.B3
- new net C0: JP2.2, U$1.C0
- new net C1: JP2.3, U$1.C1
- new net C2: L9.A, U$1.C2
- new net C3: L8.A, U$1.C3
- new net D0: RA3C.1, SW1.2, U$1.D0
- new net D1: RA3B.1, SW1.3, U$1.D1
- new net D2: RA3A.1, SW1.4, U$1.D2
- new net D3: RA2A.2, S4.2, SW1.5, U$1.D3
- new net E0: L10.A, U$1.E0
- new net E1: RA3D.1, SW1.1, U$1.E1
- new net E2: L7.A, U$1.E2
- new net E3: U$1.E3
- new net N$14: L7.C, RA6A.1
- new net N$15: L8.C, RA6B.1
- new net N$16: L9.C, RA6C.1
- new net N$17: L10.C, RA6D.1
- new net N$22: U$1.12V@1, U$1.12V@2
- net 3.3V: now also RA2A.1, RA2B.1, RA2C.1, RA2D.1, RA3A.2, RA3B.2, RA3C.2, RA3D.2
- net GND: now also JP2.6, RA6A.2, RA6B.2, RA6C.2, RA6D.2, SW1.10, SW1.11, SW1.12, SW1.13, SW1.14, SW1.15, SW1.16, SW1.9, U$1.MSEN; no longer CONN2.P, J2.PWR, R1.1, S1.4, S2.4, S3.4, S4.4, U$1.TMS
- net N$11: now also C1.1
- net TMS: now also U$1.TMS
Other:
- moved on the sheet: SW1
