File: modboard/mbmega_v1.0/board.brd (EAGLE design)
At the start: 50 x 42 mm, 18 parts, among them U1 ATMEGA328P_PDIP, Y1 16MHz

Commit message: finished the base modboards
Parts:
- removed LD1: GRN, SparkFun-LED:LED-0603
- removed LD13: RED, SparkFun-LED:LED-0603
- added LC2: GRN, SparkFun-LED:LED-0603
- added LPB1: RED, SparkFun-LED:LED-0603
- moved D1 25.7 mm to (19.1, 42.3)
- moved R1 12.1 mm to (38.5, 30.0), turned to 180 degrees
- moved C2 11.4 mm to (14.0, 24.5)
- moved Y1 11.2 mm to (19.0, 22.0)
- moved R3 11.2 mm to (47.5, 30.5), turned to 180 degrees
- moved C1 10.1 mm to (14.0, 22.0)
- moved S1 9.12 mm to (42.2, 44.0)
- moved C3 7.70 mm to (38.5, 31.5), turned to 180 degrees
- moved U1 6.00 mm to (28.4, 30.2)
- moved C4 5.50 mm to (21.5, 30.5)
- moved C5 5.50 mm to (19.5, 30.5)
- moved R5 3.16 mm to (47.5, 15.0), turned to 180 degrees
- moved R4 2.92 mm to (38.5, 28.5)
- moved LPWR 2.83 mm to (6.00, 17.0), turned to 180 degrees
- moved R2 1.58 mm to (8.00, 17.0), turned to 270 degrees
Connections:
- net E3 renamed E1
- removed net C2: R5.2, U$1.A12
- new net A3: R5.2, U$1.A18
- net B0: now also U1.5; no longer U1.2
- net B1: now also U1.4; no longer U1.3
- net B2: now also U1.3; no longer U1.4
- net B3: now also U1.2; no longer U1.5
- net D0: now also U1.25; no longer U1.23
- net D2: now also U1.23; no longer U1.25
- net E0: now also U$1.A9; no longer U$1.A14
- net GND: now also LC2.C, LPB1.C, U$1.A14, U$1.B3; no longer LD1.C, LD13.C, U$1.A9
- net MISO: now also U$1.A13; no longer U$1.A17
- net MOSI: now also U$1.A15; no longer U$1.A16
- net N$2: now also LPB1.A; no longer LD13.A
- net N$7: now also LC2.A; no longer LD1.A
- net N$9: now also U$1.A17; no longer U$1.A13
- net SCK: now also U$1.A12; no longer U$1.A18
- net SS: now also U$1.A16; no longer U$1.A15
Routing:
- net SCL: track 0.00 -> 65.0 mm, vias 0 -> 1
- net SDA: track 0.00 -> 63.4 mm, vias 0 -> 2
- net G0: track 0.00 -> 62.4 mm, vias 0 -> 1
- net 3.3V: track 0.00 -> 60.2 mm, vias 0 -> 1
- net B3: track 0.00 -> 49.1 mm
- net GND: track 0.00 -> 49.0 mm, vias 0 -> 9
- net D0: track 0.00 -> 47.8 mm, vias 0 -> 1
- net N$1: track 0.00 -> 47.2 mm
- net B2: track 0.00 -> 45.8 mm
- net D1: track 0.00 -> 45.0 mm, vias 0 -> 1
- net RST: track 0.00 -> 44.6 mm
- net C0: track 0.00 -> 44.5 mm, vias 0 -> 3
- net B1: track 0.00 -> 43.2 mm
- net D2: track 0.00 -> 42.7 mm, vias 0 -> 3
- net B0: track 0.00 -> 40.7 mm
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- added copper zone on layer 16, net GND
Other:
- board text added: "FABRIC"
- board text added: "MBMega v1.0 MB v1.0 10-21-13"
- board text added: "MEGA"
- board text added: "PWR"
