File: modboard/mbmega_v1.0/board.sch (EAGLE design)
At the start: 18 parts, among them U1 ATMEGA328P_PDIP, Y1 16MHz

Commit message: finished the base modboards
Parts:
- renumbered LD1 to LC2, LD13 to LPB1
Connections:
- removed net C2: R5.2, U$1.C2
- removed net E3: U$1.E3, U1.PD7(AIN1)
- new net A3: R5.2, U$1.A3
- new net E1: U$1.E1, U1.PD7(AIN1)
- net B0: now also U1.PD3(INT1); no longer U1.PD0(RXD)
- net B1: now also U1.PD2(INT0); no longer U1.PD1(TXD)
- net B2: now also U1.PD1(TXD); no longer U1.PD2(INT0)
- net B3: now also U1.PD0(RXD); no longer U1.PD3(INT1)
- net D0: now also U1.PC2(ADC2); no longer U1.PC0(ADC0)
- net D2: now also U1.PC0(ADC0); no longer U1.PC2(ADC2)
- net GND: now also U$1.E3, U$1.MSEN; no longer U$1.E1
- net MISO: now also U$1.C3; no longer U$1.A2
- net MOSI: now also U$1.A0; no longer U$1.A1
- net N$9: now also U$1.A2; no longer U$1.C3
- net SCK: now also U$1.C2; no longer U$1.A3
- net SS: now also U$1.A1; no longer U$1.A0
