File: vga/board_v0.1/board.sch (EAGLE design)
At the start: 1 part

Commit message: finished the base modboards
Parts:
- added R1, R2: 100, kmod-passives:RESISTOR0603
- added R10, R4, R6, R9: 500, kmod-passives:RESISTOR0603
- added R3: 10, kmod-passives:RESISTOR0603
- added R5, R7: 250, kmod-passives:RESISTOR0603
- added U$2: XC3S{50,100,200}A-FT256, kmod-xilinx:XC3S{50,100,200}A-FT256
- added U$4: MCP1700, kmod-ics:VREGSOT23-3
- added X2: (no value), con-subd:HF15H
Connections:
- new net 1.2V: U$2.G7/VCCINT, U$2.G9/VCCINT, U$2.H8/VCCINT, U$2.J9/VCCINT, U$2.K10/VCCINT, U$2.K8/VCCINT, U$4.OUT
- new net 1.8V: U$1.1.8V
- new net 3.3V: U$1.3.3V, U$2.B13/VCCO_0, U$2.B5/VCCO_0, U$2.B9/VCCO_0, U$2.D2/VCCO_3, U$2.E11/VCCAUX, U$2.E15/VCCO_1, U$2.E8/VCCO_0, U$2.F5/VCCAUX, U$2.H12/VCCO_1, U$2.H2/VCCO_3, U$2.J15/VCCO_1, U$2.J5/VCCO_3, U$2.L12/VCCAUX, U$2.M2/VCCO_3, U$2.M6/VCCAUX, U$2.M9/VCCO_2, U$2.N15/VCCO_1, U$2.R12/VCCO_2, U$2.R4/VCCO_2, U$2.R8/VCCO_2, U$4.IN
- new net GND: U$1.DSEN, U$1.GND@1, U$1.GND@2, U$1.MSEN, U$2.A1/GND, U$2.A16/GND, U$2.B11/GND, U$2.B7/GND, U$2.C14/GND, U$2.C3/GND, U$2.E12/GND, U$2.E5/GND, U$2.F2/GND, U$2.F6/GND, U$2.G10/GND, U$2.G15/GND, U$2.G8/GND, U$2.H9/GND, U$2.J8/GND, U$2.K2/GND, U$2.K7/GND, U$2.K9/GND, U$2.L11/GND, U$2.L15/GND, U$2.M12/GND, U$2.M5/GND, U$2.P14/GND, U$2.P3/GND, U$2.R10/GND, U$2.R6/GND, U$2.T1/GND, U$2.T16/GND, U$4.GND, X2.10, X2.5, X2.6, X2.7, X2.8
- new net HSYNC: R2.2
- new net N$1: R1.1, X2.14
- new net N$2: R2.1, X2.13
- new net N$3: X2.1
- new net N$4: X2.2
- new net N$5: X2.3
- new net TCK: U$1.TCK, U$2.A15/TCK
- new net TDI: U$1.TDI, U$2.B1/TDI
- new net TDO: U$1.TDO, U$2.B16/TDO
- new net TMS: U$1.TMS, U$2.B2/TMS
- new net VSYNC: R1.2

Commit message: vga card done -- first 4-layer board!
Parts:
- added C1, C11, C12, C14, C15, C17, C18, C20, C21, C23, C24, C26, C27, C4, C5, C6, C9: 100nF, kmod-passives:CAP0402-CAP
- added C10, C13, C16, C19, C2, C22, C25, C3, C7, C8: 10uF, kmod-passives:CAP0805
- added IC1: AS4C4M16S, memory-micron:MT48LC64M4A2
- added INIT_B: (no value), kmod-nonparts:CONNECTOR1.27
- added JP1: (no value), SparkFun-Connectors:M06SIP
- added L3V3, LDONE: YLW, kmod-passives:LED0603
- added R11: 2k, kmod-passives:RESISTOR0603
- added R12, R13, R14: 3.9k, kmod-passives:RESISTOR0603
- added R15, R16, R17: 8.2k, kmod-passives:RESISTOR0603
- added R18, R19: 220, kmod-passives:RESISTOR0603
- added R8: 1k, kmod-passives:RESISTOR0603
- added U$6: OSCILLATORCTS-636-50MHz, kmod-mechanical:OSCILLATORCTS-636
- added U$7: S25FL, kmod-ics:S25FL
- R10, R9: value 500 -> 2k
- R3: value 10 -> 510
- R4: value 500 -> 510
- R5: value 250 -> 510
- R6: value 500 -> 1k
- R7: value 250 -> 1k
Connections:
- new net 50MHZ: U$2.R7/IO_L09P_2/GCLK12(50:N.C.), U$6.OUT
- new net A0: U$1.A0, U$2.P8/IO_L10P_2/GCLK14
- new net A1: U$1.A1, U$2.R9/IO_L12P_2/GCLK2
- new net A2: U$1.A2, U$2.P16/IO_L03P_1/A0(50:IO_L03P_1)
- new net A3: U$1.A3, U$2.P13/IO_L19N_2(50:N.C.)
- new net B0: U$1.B0, U$2.T11/IO_L15P_2/AWAKE
- new net B1: U$1.B1, U$2.R11/IO_L15N_2/DOUT
- new net B2: U$1.B2, U$2.R13/IO_L18N_2/D1(50:IO_L20P_2/D1)
- new net B3: U$1.B3, U$2.T13/IO_L18P_2/D2
- new net C0: U$1.C0, U$2.T4/IO_L05P_2
- new net C1: U$1.C1, U$2.R5/IO_L05N_2(50:IO_L06P_2)
- new net C2: U$1.C2, U$2.T5/IO_L06P_2/D7(50:IO_L05N_2/D7)
- new net C3: U$1.C3, U$2.T6/IO_L06N_2/D6
- new net CS: JP1.5, U$2.T2/IO_L02N_2/CSO_B, U$7.!CS
- new net D0: U$1.D0, U$2.N7/IO_L07P_2(50:N.C.)
- new net D1: U$1.D1, U$2.T8/IO_L10N_2/GCLK15
- new net D2: U$1.D2, U$2.T9/IO_L12N_2/GCLK3
- new net D3: U$1.D3, U$2.T10/IO_L14P_2(50:IO_L14N_2)
- new net DONE: LDONE.A, U$2.T15/DONE
- new net G0: U$1.G0, U$2.T7/IO_L09N_2/GCLK13(50:N.C.)
- new net GRST: U$1.!GRST, U$2.A2/PROG_B
- new net MA0: IC1G$1.A0, U$2.F16/IO_L16N_1/A11(50:N.C.)
- new net MA1: IC1G$1.A1, U$2.G14/IO_L17N_1/A13(50:N.C.)
- new net MA10: IC1G$1.A10, U$2.F15/IO_L18N_1/A15(50:N.C.)
- new net MA11: IC1G$1.A11, U$2.K14/IO_L11N_1/RHCLK1
- new net MA12: IC1G$1.A12, U$2.R15/IO_L02P_1/LDC1
- new net MA2: IC1G$1.A2, U$2.G16/IO_L16P_1/A10(50:N.C.)
- new net MA3: IC1G$1.A3, U$2.H15/IO_L15P_1/IRDY1/RHCLK6
- new net MA4: IC1G$1.A4, U$2.H16/IO_L15N_1/RHCLK7
- new net MA5: IC1G$1.A5, U$2.H14/IO_L14N_1/RHCLK5
- new net MA6: IC1G$1.A6, U$2.J16/IO_L12N_1/TRDY1/RHCLK3
- new net MA7: IC1G$1.A7, U$2.K16/IO_L12P_1/RHCLK2
- new net MA8: IC1G$1.A8, U$2.J14/IO_L14P_1/RHCLK4
- new net MA9: IC1G$1.A9, U$2.K15/IO_L11P_1/RHCLK0
- new net MBA0: IC1G$1.BA0, U$2.E16/IO_L18P_1/A14(50:N.C.)
- new net MBA1: IC1G$1.BA1, U$2.F14/IO_L19N_1/A17(50:N.C.)
- new net MCAS: IC1G$1.!CAS, U$2.D16/IO_L22P_1/A20(50:IO_L22P_1)
- new net MCKE: IC1G$1.CKE, U$2.N16/IO_L03N_1/A1(50:IO_L03N_1)
- new net MCLK: IC1G$1.CLK, U$2.M14/IO_L05N_1/VREF_1(50:N.C.)
- new net MCS: IC1G$1.\CS, U$2.B15/IO_L02P_0/VREF_0
- new net MDQ0: IC1G$1.DQ0, U$2.D7/IO_L16P_0
- new net MDQ1: IC1G$1.DQ1, U$2.E7/IO_L14N_0/VREF_0(50:N.C.)
- new net MDQ10: IC1G$1.DQ10, U$2.N12/IO_L19P_2(50:N.C.)
- new net MDQ11: IC1G$1.DQ11, U$2.N11/IO_L16N_2
- new net MDQ12: IC1G$1.DQ12, U$2.N10/IO_L13P_2(50:N.C.)
- new net MDQ13: IC1G$1.DQ13, U$2.P9/IO_L11N_2/GCLK1
- new net MDQ14: IC1G$1.DQ14, U$2.N8/IO_L08N_2/D4
- new net MDQ15: IC1G$1.DQ15, U$2.P6/IO_L07N_2(50:N.C.)
- new net MDQ2: IC1G$1.DQ2, U$2.D8/IO_L11N_0/GCLK9
- new net MDQ3: IC1G$1.DQ3, U$2.D9/IO_L09N_0/GCLK5
- new net MDQ4: IC1G$1.DQ4, U$2.D11/IO_L03N_0
- new net MDQ5: IC1G$1.DQ5, U$2.D13/IO_L01P_0
- new net MDQ6: IC1G$1.DQ6, U$2.C13/IO_L01N_0
- new net MDQ7: IC1G$1.DQ7, U$2.B14/IO_L02N_0
- new net MDQ8: IC1G$1.DQ8, U$2.N14/IO_L01N_1/LDC2
- new net MDQ9: IC1G$1.DQ9, U$2.N13/IO_L01P_1/HDC
- new net MDQMH: IC1G$1.DQMH, U$2.M13/IO_L05P_1(50:N.C.)
- new net MDQML: IC1G$1.DQML, U$2.C16/IO_L24P_1/A24(50:IO_L24P_1)
- new net MISO: JP1.3, U$2.T14/IO_L20P_2/D0/DIN/MISO(50:IO_L18N_2/D0/DIN/MISO), U$7.SO
- new net MNC: IC1G$1.NC, U$2.P15/IO_L02N_1/LDC0
- new net MOSI: JP1.2, U$2.P10/IO_L14N_2/MOSI/CSI_B(50:IO_L14P_2/MOSI/CSI_B), U$7.SI
- new net MRAS: IC1G$1.!RAS, U$2.E14/IO_L20P_1/A18(50:IO_L20P_1)
- new net MWE: IC1G$1.!WE, U$2.D15/IO_L22N_1/A21(50:IO_L22N_1)
- new net N$6: L3V3.C, R18.2
- new net N$7: R10.2, R13.2, R16.2, R4.2, R7.2, X2.2
- new net N$8: R11.2, R14.2, R17.2, R5.2, R8.2, X2.1
- new net SCK: JP1.4, U$2.R14/IO_L20N_2/CCLK, U$7.SCK
- new net VB0: R3.1, U$2.A9/IO_L10N_0/GCLK7
- new net VB1: R6.1, U$2.C8/IO_L11P_0/GCLK8
- new net VB2: R9.1, U$2.A10/IO_L08N_0
- new net VB3: R12.1, U$2.A12/IO_L05N_0(50:N.C.)
- new net VB4: R15.1, U$2.A13/IO_L04N_0
- new net VG0: R4.1, U$2.C6/IO_L16N_0
- new net VG1: R7.1, U$2.A6/IO_L15P_0
- new net VG2: R10.1, U$2.B6/IO_L15N_0
- new net VG3: R13.1, U$2.A8/IO_L12P_0/GCLK10
- new net VG4: R16.1, U$2.B8/IO_L12N_0/GCLK11
- new net VR0: R5.1, U$2.B3/IO_L19N_0
- new net VR1: R8.1, U$2.A3/IO_L19P_0
- new net VR2: R11.1, U$2.A4/IO_L18P_0
- new net VR3: R14.1, U$2.B4/IO_L18N_0
- new net VR4: R17.1, U$2.A5/IO_L17P_0
- net 1.2V: now also C24.1, C25.1, C26.1, C27.1, C8.1
- net 3.3V: now also C1.1, C10.1, C11.1, C12.1, C13.1, C14.1, C15.1, C16.1, C17.1, C18.1, C19.1, C2.1, C20.1, C21.1, C22.1, C23.1, C3.1, C4.1, C5.1, C6.1, C7.1, C9.1, IC1P.VDD@1, IC1P.VDD@2, IC1P.VDD@3, IC1P.VDDQ@1, IC1P.VDDQ@2, IC1P.VDDQ@3, IC1P.VDDQ@4, JP1.6, L3V3.A, U$2.N6/IO_L04P_2/VS1(50:IO_L03N_2/VS1), U$2.P4/IO_L01N_2/M0, U$2.P5/IO_L04N_2/VS0, U$2.T3/IO_L03N_2/VS2(50:IO_L04P_2/VS2), U$6.EN, U$6.VCC, U$7.!HOLD, U$7.!WP, U$7.VCC
- net GND: now also C1.2, C10.2, C11.2, C12.2, C13.2, C14.2, C15.2, C16.2, C17.2, C18.2, C19.2, C2.2, C20.2, C21.2, C22.2, C23.2, C24.2, C25.2, C26.2, C27.2, C3.2, C4.2, C5.2, C6.2, C7.2, C8.2, C9.2, IC1P.VSS@1, IC1P.VSS@2, IC1P.VSS@3, IC1P.VSSQ@1, IC1P.VSSQ@2, IC1P.VSSQ@3, IC1P.VSSQ@4, JP1.1, R18.1, R19.1, U$1.E0, U$1.E1, U$1.E2, U$1.E3, U$2.D5/IO_L20N_0/PUDC_B, U$2.N4/IO_L01P_2/M1, U$2.R16/SUSPEND, U$2.R2/IO_L02P_2/M2, U$6.GND, U$7.GND
- net HSYNC: now also U$2.A14/IO_L04P_0
- net N$3: now also LDONE.C, R19.2; no longer X2.1
- net N$4: now also INIT_B.P, U$2.T12/IO_L17P_2/INIT_B; no longer X2.2
- net N$5: now also R12.2, R15.2, R3.2, R6.2, R9.2
- net VSYNC: now also U$2.C9/IO_L10P_0/GCLK6
Other:
- moved on the sheet: R10, R3, R4, R5, R6, R7, R9
