File: jtag/jtagusaur_v0.2/board.brd (EAGLE design)
At the start: 47.7 x 26 mm, 42 parts, among them J1 AVR_SPI_PRG_62X3_LOCK, U1 ATMEGA328P, Y1 16MHz

Commit message: update some of these values for the leds I decided to populate and their respective brightnesses
Parts:
- L1, L2: value (none) -> RED
- L3PWR, LTX: value (none) -> GRN
- L5PWR, LRX: value (none) -> YLW
- R8: value 330 -> 470
- R9: value 220 -> 330
Changed lines of the file:
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@@
 <?xml version="1.0" encoding="utf-8"?>
 <!DOCTYPE eagle SYSTEM "eagle.dtd">
-<eagle version="6.4">
+<eagle version="6.5.0">
 <drawing>
 <settings>
@@
 <setting verticaltext="up"/>
 </settings>
-<grid distance="0.2" unitdist="mm" unit="mm" style="lines" multiple="1" display="yes" altdistance="0.1" altunitdist="mm" altunit="mm"/>
+<grid distance="0.5" unitdist="mm" unit="mm" style="lines" multiple="1" display="yes" altdistance="0.01" altunitdist="mm" altunit="mm"/>
 <layers>
 <layer number="1" name="Top" color="4" fill="1" visible="yes" active="yes"/>
@@
 <layer number="25" name="tNames" color="7" fill="1" visible="no" active="yes"/>
 <layer number="26" name="bNames" color="7" fill="1" visible="no" active="yes"/>
-<layer number="27" name="tValues" color="7" fill="1" visible="no" active="yes"/>
+<layer number="27" name="tValues" color="7" fill="1" visible="yes" active="yes"/>
 <layer number="28" name="bValues" color="7" fill="1" visible="no" active="yes"/>
 <layer number="29" name="tStop" color="7" fill="3" visible="no" active="yes"/>
@@
 <element name="CONN3" library="kmod-nonparts" package="HOLE_22AWG" value="GND" x="8.4" y="2" rot="R180"/>
 <element name="Y1" library="SparkFun-FreqCtrl" package="HC49US" value="16MHz" x="39" y="19.4" rot="R270"/>
-<element name="L1" library="kmod-passives" package="0603_LED" value="" x="2" y="24" rot="R90"/>
-<element name="L2" library="kmod-passives" package="0603_LED" value="" x="2" y="22.5" rot="R90"/>
+<element name="L1" library="kmod-passives" package="0603_LED" value="RED" x="2" y="24" rot="R90"/>
+<element name="L2" library="kmod-passives" package="0603_LED" value="RED" x="2" y="22.5" rot="R90"/>
 <element name="LF" library="kmod-passives" package="0603_LED" value="" x="43.4" y="24" rot="R180"/>
 <element name="R5" library="kmod-passives" package="0603-RES" value="220" x="7" y="24"/>
@@
 <element name="R7" library="kmod-passives" package="0603-RES" value="220" x="45" y="24" rot="R270"/>
 <element name="U$5" library="kmod-testing" package="TSSOP14" value="TXB0104PWR" x="32" y="8.1" rot="R90"/>
-<element name="L5PWR" library="kmod-passives" package="0603_LED" value="" x="2" y="4.6" rot="R270"/>
-<element name="R8" library="kmod-passives" package="0603-RES" value="330" x="9" y="6.7" rot="R180"/>
-<element name="R9" library="kmod-passives" package="0603-RES" value="220" x="7" y="19.5" rot="R180"/>
+<element name="L5PWR" library="kmod-passives" package="0603_LED" value="YLW" x="2" y="4.6" rot="R270"/>
+<element name="R8" library="kmod-passives" package="0603-RES" value="470" x="9" y="6.7" rot="R180"/>
+<element name="R9" library="kmod-passives" package="0603-RES" value="330" x="7" y="19.5" rot="R180"/>
 <element name="R10" library="kmod-passives" package="0603-RES" value="220" x="7" y="18" rot="R180"/>
-<element name="LRX" library="kmod-passives" package="0603_LED" value="" x="2" y="19.5" rot="R270"/>
-<element name="LTX" library="kmod-passives" package="0603_LED" value="" x="2" y="18" rot="R270"/>
+<element name="LRX" library="kmod-passives" package="0603_LED" value="YLW" x="2" y="19.5" rot="R270"/>
+<element name="LTX" library="kmod-passives" package="0603_LED" value="GRN" x="2" y="18" rot="R270"/>
 <element name="C12" library="kmod-passives" package="0402-CAP" value="22pF" x="42.8" y="16.6"/>
 <element name="C13" library="kmod-passives" package="0402-CAP" value="22pF" x="42.8" y="18.2"/>
 <element name="J1" library="SparkFun-Connectors" package="2X3_LOCK" value="AVR_SPI_PRG_62X3_LOCK" x="17.5" y="22.7" smashed="yes" rot="R180"/>
 <element name="RA1" library="kmod-passives" package="0603-ARV" value="100R" x="21" y="22.5" rot="R90"/>
-<element name="L3PWR" library="kmod-passives" package="0603_LED" value="" x="5.2" y="4.6" rot="R270"/>
+<element name="L3PWR" library="kmod-passives" package="0603_LED" value="GRN" x="5.2" y="4.6" rot="R270"/>
 <element name="R11" library="kmod-passives" package="0603-RES" value="220" x="9" y="5" rot="R180"/>
 <element name="C9" library="kmod-passives" package="0402-CAP" value="100nF" x="12.5" y="7"/>
