File: vga/board_v0.2/board.brd (EAGLE design)
At the start: 35 x 44 mm, 70 parts, among them IC1 AS4C4M16S

Commit message: Got a very basic vga thing working, though with some issues -- the blue doesn't seem to be working, and I seem to be missing one of the green bits
Connections:
- net VB0: now also R15.1, U$9.43; no longer R3.1, U$9.47
- net VB1: now also R12.1, U$9.44; no longer R6.1, U$9.46
- net VB3: now also R6.1, U$9.46; no longer R12.1, U$9.44
- net VB4: now also R3.1, U$9.47; no longer R15.1, U$9.43
- net VG0: now also R16.1, U$9.48; no longer R4.1, U$9.56
- net VG1: now also R13.1, U$9.50; no longer R7.1, U$9.55
- net VG3: now also R7.1, U$9.55; no longer R13.1, U$9.50
- net VG4: now also R4.1, U$9.56; no longer R16.1, U$9.48
- net VR0: now also R17.1, U$9.57; no longer R5.1, U$9.67
- net VR1: now also R14.1, U$9.58; no longer R8.1, U$9.66
- net VR3: now also R8.1, U$9.66; no longer R14.1, U$9.58
- net VR4: now also R5.1, U$9.67; no longer R17.1, U$9.57
Routing:
- net VG4: track 4.28 -> 6.31 mm
- net VG0: track 6.31 -> 4.28 mm
- net VR4: track 7.25 -> 8.37 mm
- net VR0: track 8.37 -> 7.25 mm
- net VB4: track 4.93 -> 3.87 mm
- net VB0: track 3.87 -> 4.93 mm
- net VR3: track 8.19 -> 7.43 mm
- net VR1: track 7.43 -> 8.19 mm
- net VB3: track 4.07 -> 3.45 mm
- net VB1: track 3.45 -> 4.07 mm
Changed lines of the file:
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@@
 <?xml version="1.0" encoding="utf-8"?>
 <!DOCTYPE eagle SYSTEM "eagle.dtd">
-<eagle version="6.4">
+<eagle version="6.5.0">
 <drawing>
 <settings>
@@
 <setting verticaltext="up"/>
 </settings>
-<grid distance="0.1" unitdist="mm" unit="mm" style="lines" multiple="1" display="yes" altdistance="0.01" altunitdist="mm" altunit="mm"/>
+<grid distance="0.5" unitdist="mm" unit="mm" style="lines" multiple="1" display="yes" altdistance="0.01" altunitdist="mm" altunit="mm"/>
 <layers>
 <layer number="1" name="Top" color="4" fill="1" visible="yes" active="yes"/>
@@
 <wire x1="12" y1="44.289" x2="13.171" y2="45.46" width="0.2286" layer="1"/>
 </signal>
-<signal name="VB0">
+<signal name="VB4">
 <contactref element="R3" pad="1"/>
 <contactref element="U$9" pad="47"/>
@@
 <wire x1="22.25" y1="38.3" x2="22.25" y2="36.2" width="0.127" layer="1"/>
 </signal>
-<signal name="VG0">
+<signal name="VG4">
 <contactref element="R4" pad="1"/>
 <contactref element="U$9" pad="56"/>
@@
 <wire x1="13.65" y1="39.55" x2="13.5" y2="39.55" width="0.127" layer="1"/>
 </signal>
-<signal name="VR0">
+<signal name="VR4">
 <contactref element="R5" pad="1"/>
 <contactref element="U$9" pad="67"/>
@@
 <wire x1="11.8" y1="37.9" x2="12.25" y2="37.45" width="0.127" layer="1"/>
 </signal>
-<signal name="VG1">
+<signal name="VG3">
 <contactref element="R7" pad="1"/>
 <contactref element="U$9" pad="55"/>
@@
 <wire x1="18.25" y1="37.35" x2="18.25" y2="36.2" width="0.127" layer="1"/>
 </signal>
-<signal name="VR1">
+<signal name="VR3">
 <contactref element="R8" pad="1"/>
 <contactref element="U$9" pad="66"/>
@@
 <wire x1="15.4" y1="37.5" x2="15.9" y2="37.5" width="0.127" layer="1"/>
 </signal>
-<signal name="VG3">
+<signal name="VG1">
 <contactref element="R13" pad="1"/>
 <contactref element="U$9" pad="50"/>
@@
 <wire x1="20.75" y1="37.75" x2="20.75" y2="36.2" width="0.127" layer="1"/>
 </signal>
-<signal name="VR3">
+<signal name="VR1">
 <contactref element="R14" pad="1"/>
 <contactref element="U$9" pad="58"/>
@@
 <wire x1="15.1" y1="38.2" x2="15.5" y2="37.8" width="0.127" layer="1"/>
 </signal>
-<signal name="VG4">
+<signal name="VG0">
 <contactref element="R16" pad="1"/>
 <contactref element="U$9" pad="48"/>
@@
 <wire x1="21.75" y1="37.3" x2="21.75" y2="36.2" width="0.127" layer="1"/>
 </signal>
-<signal name="VR4">
+<signal name="VR0">
 <contactref element="R17" pad="1"/>
 <contactref element="U$9" pad="57"/>
@@
 <wire x1="8.1" y1="8.6" x2="10.4" y2="8.6" width="0.2286" layer="1"/>
 </signal>
-<signal name="VB1">
+<signal name="VB3">
 <contactref element="R6" pad="1"/>
 <contactref element="U$9" pad="46"/>
@@
 <wire x1="23.25" y1="38.8" x2="23.25" y2="36.2" width="0.127" layer="1"/>
 </signal>
-<signal name="VB3">
+<signal name="VB1">
 <contactref element="R12" pad="1"/>
 <contactref element="U$9" pad="44"/>
@@
 <wire x1="23.75" y1="37.8" x2="23.75" y2="36.2" width="0.127" layer="1"/>
 </signal>
-<signal name="VB4">
+<signal name="VB0">
 <contactref element="R15" pad="1"/>
 <contactref element="U$9" pad="43"/>
