File: coven/test_socket/board.brd (EAGLE design)
At the start: 160 x 100 mm, 22 parts, among them J1 ATX24RH

Commit message: Initial coven boards: A13 v0.1 card and test socket
Parts:
- added C10, C11, C6, C9: DNP(15pF), kmod-passives:0402-CAP
- added C12: DNP(0.1uF), kmod-passives:0402-CAP
- added C13, C14: 47pF, kmod-passives:0402-CAP
- added C15, C16, C22, C24, C29: 10uF, kmod-passives:0805
- added C17, C18, C27: 0.1uF, kmod-passives:0402-CAP
- added C19: 3300pF, kmod-passives:0402-CAP
- added C20: 1uF, kmod-passives:0603-CAP
- added C21: 5pF-100pF;optional, kmod-passives:0402-CAP
- added C23: DNP(10uF), kmod-passives:0805
- added C25: 22uF, kmod-passives:0805
- added C26: 4.7uF, kmod-passives:0603-CAP
- added C28: 100uF, kmod-passives:CAP-5-2
- added C5: 22nF, kmod-passives:0402-CAP
- added CONN10: 3.3V, kmod-nonparts:HOLE_22AWG
- added CONN11: GND, kmod-nonparts:HOLE_22AWG
- added CONN12: RESET#, kmod-nonparts:HOLE_22AWG
- added CONN13: UBOOT, kmod-nonparts:HOLE_22AWG
- added CONN14: MOSI, kmod-nonparts:HOLE_22AWG
- added CONN15: MISO, kmod-nonparts:HOLE_22AWG
- added CONN16: CLK, kmod-nonparts:HOLE_22AWG
- added CONN17: CS, kmod-nonparts:HOLE_22AWG
- added CONN3: PWR_ON#, kmod-nonparts:HOLE_22AWG
- added CONN4: I2C_SCL, kmod-nonparts:HOLE_22AWG
- added CONN5: I2C_SDA, kmod-nonparts:HOLE_22AWG
- added CONN6: COM_RX, kmod-nonparts:HOLE_22AWG
- added CONN7: COM_TX, kmod-nonparts:HOLE_22AWG
- added CONN8: 12V, kmod-nonparts:HOLE_22AWG
- added CONN9: 5V, kmod-nonparts:HOLE_22AWG
- added J2: POWER_JACKPTH, SparkFun-Connectors:POWER_JACK_PTH
- added JP2: USB-IDMICRO, kmod-connectors:USB-MICRO
- added L1: 1.5A,3.3uH:NR6028T3R0N, kmod-passives:NR60XX
- added L12V, L5VSTD: RED, kmod-passives:0603_LED
- added LPRSNT, LPWROK, LPWR_ON, LRESET, LRX, LUBOOT: YLW, kmod-passives:0603_LED
- added LTX: GRN, kmod-passives:0603_LED
- added Q1: BSS84, SparkFun-DiscreteSemi:SOT23-3
- added R12, R15, R17, R33: 100k, kmod-passives:0603-RES
- added R13, R16, R18, R19, R9: 330, kmod-passives:0603-RES
- added R14, R24, R25, R27: 4.7k, kmod-passives:0603-RES
- added R20: 220, kmod-passives:0603-RES
- added R21: DNP(330), kmod-passives:0603-RES
- added R22, R23: 27R, kmod-passives:0603-RES
- added R28, R29, R30: 0.01R, kmod-passives:0603-RES
- added R31: 56k 1%, kmod-passives:0603-RES
- added R32: 10k 1%, kmod-passives:0603-RES
- added R4: 10R, kmod-passives:0603-RES
- added R6: 47k, kmod-passives:0603-RES
- added R7: 470, kmod-passives:0603-RES
- added R8: 1k, kmod-passives:0603-RES
- added SB1: RX, kmod-nonparts:TRACE-CUT
- added SB2: TX, kmod-nonparts:TRACE-CUT
- added SB3: 12V_CS, kmod-nonparts:SOLDER-BRIDGE-OPEN-LARGE
- added SB4: 5V_CS, kmod-nonparts:SOLDER-BRIDGE-OPEN-LARGE
- added SB5: 3V3_CS, kmod-nonparts:SOLDER-BRIDGE-OPEN-LARGE
- added SB6: HVB_CS, kmod-nonparts:SOLDER-BRIDGE-OPEN-LARGE
- added SB7: OVB_CS, kmod-nonparts:SOLDER-BRIDGE-OPEN-LARGE
- added SW_ATXON, SW_PWRON: MHPS2283, kmod-mechanical:PUSHBUTTON-2.5-5.4
- added SW_RESET, SW_UBOOT: TAC_SWITCHPTH, kmod-mechanical:TACTILE-PTH
- added U$5: RJ45-ETHERNET, kmod-connectors:RJ45
- added U$6: D1213A-04S, kmod-discretesemi:SOT363
- added U$7: FT230X, kmod-ics:TSSOP16
- added U$8: BD9D321EFJ, kmod-testing:HTSOP8
- added U$9: SPX1117M3-L-3-3, kmod-ics:SOT223
- C1: value 0.1uF/DNP -> DNP(0.1uF)
- C3, C4, C7, C8: value 1uF? -> 1uF
- R1: value 330R?/DNP -> DNP(330)
- U$3: value RJ45-8PTH -> D1213A-04S; device SparkFun-Connectors:RJ45-8 -> kmod-discretesemi:SOT363
- moved U$3 147.2 mm to (60.9, 9.20), turned to 180 degrees
- moved R1 141.3 mm to (69.9, 6.00), turned to 180 degrees
- moved CONN2 134.7 mm to (55.5, 8.50)
- moved R10 131.9 mm to (49.4, 18.6), turned to 90 degrees
- moved U$4 129.8 mm to (48.4, 22.4)
- moved C7 128.7 mm to (44.4, 24.0), turned to 180 degrees
- moved C1 128.2 mm to (69.9, 4.20)
- moved R11 125.5 mm to (44.4, 20.8)
- moved JP1 125.1 mm to (61.0, 1.60)
- moved C8 124.8 mm to (44.4, 22.4), turned to 180 degrees
- moved U$2 119.1 mm to (62.0, 20.2)
- moved J1 112.6 mm to (38.0, 92.0), turned to 180 degrees
- moved CONN1 109.8 mm to (28.3, 9.90)
- moved C2 109.7 mm to (53.5, 22.1)
- moved R26 107.6 mm to (58.2, 20.2)
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Connections:
- removed net N$13: C8.1, R11.2, U$4.1
- removed net N$7: C4.1, R26.2, U$2.1
- removed net PWR_ON#/PRSNT#: U$1.A1, U$1.B8
- new net !RXLED: R19.1, U$7.14
- new net !TXLED: R20.1, U$7.7
- new net 12V_U: J1.10, J1.11, J2.PWR, R29.2, SB3.L1, SB3.L2
- new net 3.3V_U: C25.1, J1.1, J1.12, J1.13, J1.2, R30.2, SB5.L1, SB5.L2, U$9.2, U$9.4
- new net 5V_U: C21.1, C22.1, C23.1, J1.21, J1.22, J1.23, J1.4, J1.6, L1.P$2, R28.2, R31.2, SB4.L1, SB4.L2
- new net COM_RX: CONN6.P, SB1.R1, U$1.A7
- new net COM_TX: CONN7.P, SB2.R1, U$1.A8
- new net FT230X_DM: C13.1, JP2.D-, R23.1
- new net FT230X_DP: C14.1, JP2.D+, R22.1
- new net HOST_VBUS_U: C8.1, R11.2, SB6.L1, SB6.L2, U$4.1
- new net N$14: LPRSNT.C, R9.2
- new net N$15: LPWR_ON.A, R13.1
- new net N$16: LRESET.C, R16.2
- new net N$17: L12V.C, R14.2
- new net N$18: LUBOOT.C, R18.2
- new net N$19: R23.2, U$7.9
- new net N$20: C12.1, JP2.MT1, JP2.MT2, JP2.P$1, JP2.P$2, R21.2
- new net N$21: SB1.L1, U$7.1
- new net N$22: SB2.L1, U$7.4
- new net N$23: R22.2, U$7.8
- new net N$24: L5VSTD.C, R27.2
- new net N$25: J1.9, L5VSTD.A
- new net N$26: C18.1, U$8.7
- new net N$27: C18.2, L1.P$1, U$8.6
- new net N$28: C20.1, U$8.3
- new net N$29: C19.1, U$8.4
- new net N$30: C21.2, R31.1, R32.2, U$8.2
- new net N$4: C5.1, R4.1, U$5.3, U$5.6
- new net N$8: Q1.3, R13.2
- new net N$9: LPWROK.C, R7.2
- new net OTG_VBUS_U: C4.1, R26.2, SB7.L1, SB7.L2, U$2.1
- new net PRSNT#: R8.2, R9.1, U$1.A1
- new net PWR_ON#: CONN3.P, Q1.1, R12.1, R8.1, SW_PWRON.5, U$1.B8
- new net SPI0_CLK: CONN16.P, U$1.B27
- new net SPI0_CS: CONN17.P, U$1.B28
- new net SPI0_MISO: CONN15.P, U$1.B24
- new net SPI0_MOSI: CONN14.P, U$1.B23
- net 12V: now also C15.1, C16.1, C17.1, CONN8.P, L12V.A, R29.1, SB3.R1, SB3.R2, U$8.1, U$8.8; no longer J1.10, J1.11, J1.15, J1.17, J1.18, J1.19, J1.24, J1.3, J1.5, J1.7
- net 3.3V: now also C26.1, C27.1, CONN10.P, LPRSNT.A, LRESET.A, LRX.A, LTX.A, LUBOOT.A, Q1.2, R12.2, R15.2, R17.2, R24.2, R25.2, R30.1, R4.2, R6.2, SB5.R1, SB5.R2, SW_PWRON.4, U$7.10, U$7.12, U$7.3; no longer J1.1, J1.12, J1.13, J1.2
- net 5V: now also C24.1, CONN9.P, R28.1, SB4.R1, SB4.R2, U$9.3; no longer J1.21, J1.22, J1.23, J1.4, J1.6
- net ETH_RXN: now also C6.1, U$5.8
- net ETH_RXP: now also C9.1, U$5.7
- net ETH_TXN: now also C10.1, U$5.2
- net ETH_TXP: now also C11.1, U$5.1
- net GND: now also C10.2, C11.2, C12.2, C13.2, C14.2, C15.2, C16.2, C17.2, C19.2, C20.2, C22.2, C23.2, C24.2, C25.2, C26.2, C27.2, C28.2, C29.2, C5.2, C6.2, C9.2, CONN11.P, J1.15, J1.17, J1.18, J1.19, J1.24, J1.3, J1.5, J1.7, J2.GND, J2.GNDBREAK, JP2.GND, LPWR_ON.C, R14.1, R21.1, R27.1, R32.1, R33.1, R7.1, SW_ATXON.3, SW_RESET.2, SW_UBOOT.2, U$3.2, U$5.S1, U$5.S2, U$6.2, U$7.13, U$7.5, U$7.6, U$8.5, U$8.P$1, U$8.P$2, U$8.P$3, U$8.P$4, U$8.P$5, U$8.PAD, U$9.1
- net HOST_DM: now also U$6.4
- net HOST_DP: now also U$6.6
- net HOST_VBUS: now also C28.1, SB6.R1, SB6.R2, U$6.5
- net I2C_SCL: now also CONN4.P, R24.1
- net I2C_SDA: now also CONN5.P, R25.1
- net N$1: now also SW_ATXON.2
- net N$10: now also LRX.C, R19.2; no longer U$1.A7
- net N$11: now also LTX.C, R20.2; no longer U$1.A8
- net N$2: now also LPWROK.A
- net OTG_DM: now also U$3.4
- net OTG_DP: now also U$3.6
- net OTG_IDDET: now also R6.1, U$3.1
- net OTG_VBUS: now also C29.1, SB7.R1, SB7.R2, U$3.5
- net OTG_VBUSDRV: now also R33.2
- net SYS_RESET#: now also CONN12.P, R15.1, R16.1, SW_RESET.3
- net UBOOT: now also CONN13.P, R17.1, R18.1, SW_UBOOT.3
Routing:
- net 3.3V_U: track 0.00 -> 151.6 mm
- net COM_RX: track 0.00 -> 113.4 mm
- net COM_TX: track 0.00 -> 112.6 mm
- net 5V: track 0.00 -> 107.7 mm, vias 0 -> 6
- net UBOOT: track 0.00 -> 99.4 mm
- net N$2: track 0.00 -> 97.9 mm, vias 0 -> 1
- net N$25: track 0.00 -> 92.5 mm, vias 0 -> 1
- net PRSNT#: track 0.00 -> 85.8 mm, vias 0 -> 3
- net N$1: track 0.00 -> 85.2 mm
- net ETH_TXP: track 0.00 -> 83.9 mm, vias 0 -> 1
- net 5V_U: track 0.00 -> 83.7 mm
- net ETH_TXN: track 0.00 -> 82.5 mm, vias 0 -> 1
- net OTG_IDDET: track 0.00 -> 81.9 mm, vias 0 -> 1
- net PWR_ON#: track 0.00 -> 78.2 mm, vias 0 -> 1
- net ETH_RXP: track 0.00 -> 73.6 mm
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- added copper zone on layer 15, net 12V
- added copper zone on layer 15, net 3.3V
- added copper zone on layer 1, net GND
- added copper zone on layer 2, net GND
Other:
- board size 160 x 100 mm -> 100 x 100 mm
- board text added: "12V"
- board text added: "12V only!"
- board text added: "ATX POWER"
- board text added: "AVAIL"
- board text added: "CARD VREGS"
- board text added: "Coven test socket v1 7-3-14"
- board text added: "OTG"
- board text added: "PGOOD"
- board text added: "PRESENT"
- board text added: "RESET"
- board text added: "RX"
- board text added: "TX"
- board text added: "UART"
- board text added: "UBOOT"
