File: coven/test_socket/board.sch (EAGLE design)
At the start: 22 parts, among them J1 ATX24RH

Commit message: Initial coven boards: A13 v0.1 card and test socket
Parts:
- added C10, C11, C6, C9: DNP(15pF), kmod-passives:CAP0402-CAP
- added C12: DNP(0.1uF), kmod-passives:CAP0402-CAP
- added C13, C14: 47pF, kmod-passives:CAP0402-CAP
- added C15, C16, C22, C24, C29: 10uF, kmod-passives:CAP0805
- added C17, C18, C27: 0.1uF, kmod-passives:CAP0402-CAP
- added C19: 3300pF, kmod-passives:CAP0402-CAP
- added C20: 1uF, kmod-passives:CAP0603
- added C21: 5pF-100pF;optional, kmod-passives:CAP0402-CAP
- added C23: DNP(10uF), kmod-passives:CAP0805
- added C25: 22uF, kmod-passives:CAP0805
- added C26: 4.7uF, kmod-passives:CAP0603
- added C28: 100uF, kmod-passives:CAP_POLPTH-5-2
- added C5: 22nF, kmod-passives:CAP0402-CAP
- added CONN10: 3.3V, kmod-nonparts:CONNECTOR22AWG
- added CONN11: GND, kmod-nonparts:CONNECTOR22AWG
- added CONN12: RESET#, kmod-nonparts:CONNECTOR22AWG
- added CONN13: UBOOT, kmod-nonparts:CONNECTOR22AWG
- added CONN14: MOSI, kmod-nonparts:CONNECTOR22AWG
- added CONN15: MISO, kmod-nonparts:CONNECTOR22AWG
- added CONN16: CLK, kmod-nonparts:CONNECTOR22AWG
- added CONN17: CS, kmod-nonparts:CONNECTOR22AWG
- added CONN3: PWR_ON#, kmod-nonparts:CONNECTOR22AWG
- added CONN4: I2C_SCL, kmod-nonparts:CONNECTOR22AWG
- added CONN5: I2C_SDA, kmod-nonparts:CONNECTOR22AWG
- added CONN6: COM_RX, kmod-nonparts:CONNECTOR22AWG
- added CONN7: COM_TX, kmod-nonparts:CONNECTOR22AWG
- added CONN8: 12V, kmod-nonparts:CONNECTOR22AWG
- added CONN9: 5V, kmod-nonparts:CONNECTOR22AWG
- added J2: POWER_JACKPTH, SparkFun-Connectors:POWER_JACKPTH
- added JP2: USB-IDMICRO, kmod-connectors:USB-IDMICRO
- added L1: 1.5A,3.3uH:NR6028T3R0N, kmod-passives:INDUCTORNR60XX
- added L12V, L5VSTD: RED, kmod-passives:LED0603
- added LPRSNT, LPWROK, LPWR_ON, LRESET, LRX, LUBOOT: YLW, kmod-passives:LED0603
- added LTX: GRN, kmod-passives:LED0603
- added Q1: BSS84, SparkFun-DiscreteSemi:MOSFET-PCHANNELSMD
- added R12, R15, R17, R33: 100k, kmod-passives:RESISTOR0603
- added R13, R16, R18, R19, R9: 330, kmod-passives:RESISTOR0603
- added R14, R24, R25, R27: 4.7k, kmod-passives:RESISTOR0603
- added R20: 220, kmod-passives:RESISTOR0603
- added R21: DNP(330), kmod-passives:RESISTOR0603
- added R22, R23: 27R, kmod-passives:RESISTOR0603
- added R28, R29, R30: 0.01R, kmod-passives:RESISTOR0603
- added R31: 56k 1%, kmod-passives:RESISTOR0603
- added R32: 10k 1%, kmod-passives:RESISTOR0603
- added R4: 10R, kmod-passives:RESISTOR0603
- added R6: 47k, kmod-passives:RESISTOR0603
- added R7: 470, kmod-passives:RESISTOR0603
- added R8: 1k, kmod-passives:RESISTOR0603
- added SB1: RX, kmod-nonparts:TRACE-CUT
- added SB2: TX, kmod-nonparts:TRACE-CUT
- added SB3: 12V_CS, kmod-nonparts:SOLDER-BRIDGEOPEN-WIDE
- added SB4: 5V_CS, kmod-nonparts:SOLDER-BRIDGEOPEN-WIDE
- added SB5: 3V3_CS, kmod-nonparts:SOLDER-BRIDGEOPEN-WIDE
- added SB6: HVB_CS, kmod-nonparts:SOLDER-BRIDGEOPEN-WIDE
- added SB7: OVB_CS, kmod-nonparts:SOLDER-BRIDGEOPEN-WIDE
- added SW_ATXON, SW_PWRON: MHPS2283, kmod-mechanical:SWITCH_DPDTPUSHBUTTON
- added SW_RESET, SW_UBOOT: TAC_SWITCHPTH, kmod-mechanical:TAC_SWITCHPTH
- added U$5: RJ45-ETHERNET, kmod-connectors:RJ45-ETHERNET
- added U$6: D1213A-04S, kmod-discretesemi:TVS_ARRAY
- added U$7: FT230X, kmod-ics:FT230X
- added U$8: BD9D321EFJ, kmod-testing:BD9D321EFJ
- added U$9: SPX1117M3-L-3-3, kmod-ics:VREGSOT223
- C1: value 0.1uF/DNP -> DNP(0.1uF)
- C3, C4, C7, C8: value 1uF? -> 1uF
- R1: value 330R?/DNP -> DNP(330)
- U$3: value RJ45-8PTH -> D1213A-04S; device SparkFun-Connectors:RJ45-8PTH -> kmod-discretesemi:TVS_ARRAY
Connections:
- removed net N$13: C8.1, R11.2, U$4.OUT
- removed net N$7: C4.1, R26.2, U$2.OUT
- removed net PWR_ON#/PRSNT#: U$1.PRSNT#, U$1.PWR_ON#
- new net !RXLED: R19.1, U$7.CBUS1
- new net !TXLED: R20.1, U$7.CBUS2
- new net 12V_U: J1.12V@0, J1.12V@1, J2.PWR, R29.2, SB3.P$1
- new net 3.3V_U: C25.1, J1.3.3V@0, J1.3.3V@1, J1.3.3V@2, J1.3.3V@3, R30.2, SB5.P$1, U$9.OUT
- new net 5V_U: C21.1, C22.1, C23.1, J1.5V@0, J1.5V@1, J1.5V@2, J1.5V@3, J1.5V@4, L1.2, R28.2, R31.2, SB4.P$1
- new net COM_RX: CONN6.P, SB1.P$2, U$1.COM_TX
- new net COM_TX: CONN7.P, SB2.P$2, U$1.COM_RX
- new net FT230X_DM: C13.1, JP2.D-, R23.1
- new net FT230X_DP: C14.1, JP2.D+, R22.1
- new net HOST_VBUS_U: C8.1, R11.2, SB6.P$1, U$4.OUT
- new net N$14: LPRSNT.C, R9.2
- new net N$15: LPWR_ON.A, R13.1
- new net N$16: LRESET.C, R16.2
- new net N$17: L12V.C, R14.2
- new net N$18: LUBOOT.C, R18.2
- new net N$19: R23.2, U$7.D-
- new net N$20: C12.1, JP2.SHELL, R21.2
- new net N$21: SB1.P$1, U$7.TXD
- new net N$22: SB2.P$1, U$7.RXD
- new net N$23: R22.2, U$7.D+
- new net N$24: L5VSTD.C, R27.2
- new net N$25: J1.5V_STDBY, L5VSTD.A
- new net N$26: C18.1, U$8.BOOT
- new net N$27: C18.2, L1.1, U$8.SW
- new net N$28: C20.1, U$8.VREG
- new net N$29: C19.1, U$8.SS
- new net N$30: C21.2, R31.1, R32.2, U$8.FB
- new net N$4: C5.1, R4.1, U$5.COM
- new net N$8: Q1.D, R13.2
- new net N$9: LPWROK.C, R7.2
- new net OTG_VBUS_U: C4.1, R26.2, SB7.P$1, U$2.OUT
- new net PRSNT#: R8.2, R9.1, U$1.PRSNT#
- new net PWR_ON#: CONN3.P, Q1.G, R12.1, R8.1, SW_PWRON.COM1, U$1.PWR_ON#
- new net SPI0_CLK: CONN16.P, U$1.L7_P
- new net SPI0_CS: CONN17.P, U$1.L7_N
- new net SPI0_MISO: CONN15.P, U$1.L5_N
- new net SPI0_MOSI: CONN14.P, U$1.L5_P
- net 12V: now also C15.1, C16.1, C17.1, CONN8.P, L12V.A, R29.1, SB3.P$2, U$8.EN, U$8.VIN; no longer J1.12V@0, J1.12V@1, J1.GND@0, J1.GND@1, J1.GND@2, J1.GND@3, J1.GND@4, J1.GND@5, J1.GND@6, J1.GND@7
- net 3.3V: now also C26.1, C27.1, CONN10.P, LPRSNT.A, LRESET.A, LRX.A, LTX.A, LUBOOT.A, Q1.S, R12.2, R15.2, R17.2, R24.2, R25.2, R30.1, R4.2, R6.2, SB5.P$2, SW_PWRON.NC1, U$7.3.3V/5V, U$7.3V3OUT, U$7.VCCIO; no longer J1.3.3V@0, J1.3.3V@1, J1.3.3V@2, J1.3.3V@3
- net 5V: now also C24.1, CONN9.P, R28.1, SB4.P$2, U$9.IN; no longer J1.5V@0, J1.5V@1, J1.5V@2, J1.5V@3, J1.5V@4
- net ETH_RXN: now also C6.1, U$5.RN
- net ETH_RXP: now also C9.1, U$5.RP
- net ETH_TXN: now also C10.1, U$5.TN
- net ETH_TXP: now also C11.1, U$5.TP
- net GND: now also C10.2, C11.2, C12.2, C13.2, C14.2, C15.2, C16.2, C17.2, C19.2, C20.2, C22.2, C23.2, C24.2, C25.2, C26.2, C27.2, C28.-, C29.2, C5.2, C6.2, C9.2, CONN11.P, J1.GND@0, J1.GND@1, J1.GND@2, J1.GND@3, J1.GND@4, J1.GND@5, J1.GND@6, J1.GND@7, J2.GND, J2.GNDBREAK, JP2.GND, LPWR_ON.C, R14.1, R21.1, R27.1, R32.1, R33.1, R7.1, SW_ATXON.NO0, SW_RESET.2, SW_UBOOT.2, U$3.VN, U$5.SHIELD, U$6.VN, U$7.!CTS, U$7.GND, U$8.GND, U$9.GND
- net HOST_DM: now also U$6.CH3
- net HOST_DP: now also U$6.CH4
- net HOST_VBUS: now also C28.+, SB6.P$2, U$6.VP
- net I2C_SCL: now also CONN4.P, R24.1
- net I2C_SDA: now also CONN5.P, R25.1
- net N$1: now also SW_ATXON.COM0
- net N$10: now also LRX.C, R19.2; no longer U$1.COM_TX
- net N$11: now also LTX.C, R20.2; no longer U$1.COM_RX
- net N$2: now also LPWROK.A
- net OTG_DM: now also U$3.CH3
- net OTG_DP: now also U$3.CH4
- net OTG_IDDET: now also R6.1, U$3.CH1
- net OTG_VBUS: now also C29.1, SB7.P$2, U$3.VP
- net OTG_VBUSDRV: now also R33.2
- net SYS_RESET#: now also CONN12.P, R15.1, R16.1, SW_RESET.3
- net UBOOT: now also CONN13.P, R17.1, R18.1, SW_UBOOT.3
Other:
- note added: "Button unpressed: pulls up to 3.3V card not present: 100k pullup to 3.3V card present and button pressed: prsnt# pulls down with 1k, beats 100k pullup"
- note added: "Note: only populate one of these!"
- note added: "Or TL2201EEYA"
- note added: "VFB = 0.765"
- note added: "vreg rating: 8V <= VIN <= 18V (note: caps only 25V)"
- moved on the sheet: C1, C2, C3, C4, CONN2, J1, R1, R2, R26, R3, R5, U$2
