File: coven/a13_v0.1/board.brd (EAGLE design)
At the start: 50 x 50 mm, 169 parts, among them IC1 256/512 x 8bit, Y1 24MHz, Y2 25MHz

Commit message: work continues on coven boards
Parts:
- added C77: 0.1uF, kmod-passives:0402-CAP
- added C78: 10uF, kmod-passives:0603-CAP
- added C79: 22uF, kmod-passives:0805
- added D3: PMEG2010AEB, SparkFun-DiscreteSemi:SOD-523
- added L9: CIC10J601(750mA,600R), kmod-passives:0603
- added R35: 330R, kmod-passives:0603-RES
- added R36: 10k, kmod-passives:0603-RES
- added R37, R38, R39: 47k, kmod-passives:0603-RES
- added RA13: 47k, kmod-passives:0603-ARV
- added SB12, SB13, SB14, SB15, SB16, SB17: SOLDER-BRIDGEOPEN, kmod-nonparts:SOLDER-BRIDGE-OPEN
- added U$15: Molex 1050270001, kmod-connectors:MICROSD-MOLEX-1050270001
Connections:
- removed net AXP209_IRQ: U$14.048
- removed net AXP209_SCK: U$14.002
- removed net AXP209_SDA: U$14.001
- new net N$108: C78.1, C79.1, L9.2, U$15.P4
- new net N$112: C77.1, R35.2, U$15.SHELL1, U$15.SHELL2, U$15.SHELL3, U$15.SHELL4
- new net N$78: SB12.R1, SB12.R2, U$14.008
- new net N$89: SB15.R1, SB15.R2, SB17.R1, SB17.R2, U$14.017
- new net NMI_N: R39.1, U$1.158, U$14.048
- new net SD_CD: R36.2, U$1.155, U$15.G1
- new net SD_CLK: RA13.4, U$1.110, U$15.P5
- new net SD_CMD: RA13.3, U$1.111, U$15.P3
- new net SD_D0: R38.1, U$1.108, U$15.P7
- new net SD_D1: R37.1, U$1.107, U$15.P8
- new net SD_D2: RA13.1, U$1.113, U$15.P1
- new net SD_D3: RA13.2, U$1.112, U$15.P2
- new net TWI0-SCK: U$1.101, U$14.002
- new net TWI0-SDA: U$1.102, U$14.001
- new net VDDR_SW: L5.1, SB16.L1, SB16.L2, U$12.3
- new net VDDR_U: C60.1, L5.2, R22.2, R26.2, SB17.L1, SB17.L2
- net 3.3V: now also L9.1, R37.2, R38.2, RA13.5, RA13.6, RA13.7, RA13.8
- net GND: now also C77.2, C78.2, C79.2, R35.1, R36.1, U$15.P6
- net N$79: now also SB13.R1, SB13.R2, U$14.010; no longer L5.1, U$12.3
- net N$88: now also SB14.R1, SB14.R2, SB16.R1, SB16.R2, U$14.015; no longer C60.1, L5.2, R22.2, R26.2
- net N$93: now also R39.2; no longer U$1.158
- net VCPU_SW: now also SB12.L1, SB12.L2; no longer U$14.008
- net VCPU_U: now also SB13.L1, SB13.L2; no longer U$14.010
- net VINT_SW: now also SB14.L1, SB14.L2; no longer U$14.015
- net VINT_U: now also SB15.L1, SB15.L2; no longer U$14.017

Commit message: more work on coven
Parts:
- removed D3: PMEG2010AEB, SparkFun-DiscreteSemi:SOD-523
- removed JP1: M13X22X13, SparkFun-Connectors:2X13
- added C80, C84: 0.1uF, kmod-passives:0402-CAP
- added C81, C83: 10uF, kmod-passives:0603-CAP
- added C82: 1uF, kmod-passives:0402-CAP
- added CONN11: UBOOT, kmod-nonparts:HOLE_22AWG
- added CONN12: PWR_ON#, kmod-nonparts:TESTPAD-2MM
- added CONN13: PWR_EN, kmod-nonparts:TESTPAD-2MM
- added D2: RB521S30, kmod-discretesemi:SOD-523
- added D4: B5819WS, kmod-discretesemi:SOD-323
- added D6: PMEG2010AEB, kmod-discretesemi:SOD-523
- added L0: WHT, kmod-passives:0603_LED
- added L12V: YLW, kmod-passives:0603_LED
- added Q1: BSS84, SparkFun-DiscreteSemi:SOT23-3
- added R40: 100k, kmod-passives:0603-RES
- added R41: 200k 1%, kmod-passives:0402-RES
- added R42: 10k, kmod-passives:0402-RES
- added R44: DNP(100k), kmod-passives:0402-RES
- added R45: 2.2k, kmod-passives:0603-RES
- added R46: 470R, kmod-passives:0603-RES
- added R47, R48: 100k, kmod-passives:0402-RES
- added RA14: 10k, kmod-passives:0603-ARV
- added S2: TAC_SWITCHPTH, kmod-mechanical:TACTILE-PTH
- added U$16: CVN-V1EDGE, kmod-connectors:CVN-V1-EDGE
- added U$17: RT9818C-29GV, kmod-ics:SOT23-3
- C77: value 0.1uF -> 0.1uF/DNP
- D1: value PMEG2010AEB -> RB521S30; device SparkFun-DiscreteSemi:SOD-523 -> kmod-discretesemi:SOD-523
- R35: value 330R -> 330R?/DNP
- moved R34 372.8 mm to (80.5, 31.5)
- moved SB10 372.8 mm to (83.0, 36.5)
- moved SB11 372.8 mm to (80.5, 34.0)
- moved SB6 372.8 mm to (83.0, 41.5)
- moved SB9 372.8 mm to (83.0, 39.0)
- moved S1 367.6 mm to (75.5, 56.5)
- moved C69 364.1 mm to (106.0, 41.0)
- moved C70 364.1 mm to (102.5, 41.0)
- moved C71 364.1 mm to (99.5, 33.5)
- moved C72 364.1 mm to (99.5, 30.0)
- moved C73 364.1 mm to (99.5, 27.0)
- moved C74 364.1 mm to (96.5, 27.0)
- moved C75 364.1 mm to (93.5, 27.0)
- moved C76 364.1 mm to (90.0, 27.0)
- moved CONN10 364.1 mm to (109.0, 48.0)
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Connections:
- net N$91 renamed 3.3V_U
- new net N$103: L12V.C, R45.2
- new net N$109: L0.A, R46.1
- new net N$110: R46.2
- new net PRSNT#: U$16.A1, U$16.B49
- new net PWR_EN: CONN13.P, Q1.3, R48.2, U$10.1
- new net PWR_ON#: CONN12.P, Q1.1, R44.2, R47.1, U$16.B8
- new net SVR_ID0: RA14.1, U$16.A5
- new net SVR_ID1: RA14.2, U$16.A6
- new net SVR_ID2: RA14.3, U$16.A9
- new net SVR_ID3: RA14.4, U$16.A10
- new net SVR_ID4: R42.1, U$16.A12
- new net TWI2_SCK: U$1.160, U$16.B5
- new net TWI2_SDA: U$1.161, U$16.B6
- new net UBOOT: CONN11.P, D2.A, R40.1, S2.4, U$1.157
- new net USBOTG_IDDET: U$1.153, U$16.B16
- new net USBOTG_VBUSDET: U$1.154, U$16.B15
- new net USBOTG_VBUSDRV: U$16.A14
- new net VRA2: C83.1, C84.1, R41.2, U$1.082
- net 12V: now also L12V.A, Q1.2, R47.2, U$16.A2, U$16.A3, U$16.B1, U$16.B2, U$16.B3; no longer JP1.4, JP1.6, U$10.1
- net 3.3V: now also D4.A, D6.A, R40.2, R42.2, RA14.5, RA14.6, RA14.7, RA14.8, U$17.3; no longer D1.A
- net ETH_RXN: now also U$16.B44; no longer JP1.10
- net ETH_RXP: now also U$16.B43; no longer JP1.8
- net ETH_TXN: now also U$16.B48; no longer JP1.13
- net ETH_TXP: now also U$16.B47; no longer JP1.11
- net GND: now also C80.1, C81.1, C82.1, C83.2, C84.2, L0.C, R41.1, R44.1, R45.1, R48.1, S2.1, U$16.A15, U$16.A16, U$16.A19, U$16.A20, U$16.A23, U$16.A24, U$16.A27, U$16.A28, U$16.A31, U$16.A32, U$16.A35, U$16.A36, U$16.A39, U$16.A4, U$16.A40, U$16.A43, U$16.A44, U$16.A47, U$16.A48, U$16.B13, U$16.B14, U$16.B17, U$16.B18, U$16.B21, U$16.B22, U$16.B25, U$16.B26, U$16.B29, U$16.B30, U$16.B33, U$16.B34, U$16.B37, U$16.B38, U$16.B4, U$16.B41, U$16.B42, U$16.B45, U$16.B46, U$16.B7, U$17.2
- net N$92: now also D1.C, U$16.B11; no longer U$1.157
- net N$93: now also D4.C
- net N$95: now also C80.2, C81.2
- net N$96: now also D2.C, U$16.A13; no longer U$1.082
- net N$97: now also C82.2
- net N$98: now also D6.C; no longer D1.C
- net RESET_N: now also D1.A, U$17.1
- net UART1_RX: now also U$16.A8; no longer JP1.5
- net UART1_TX: now also U$16.A7; no longer JP1.3
- net USB2DM: now also U$16.B10; no longer JP1.21
- net USB2DP: now also U$16.B9; no longer JP1.19
- net USB3DM: no longer JP1.26
- net USB3DP: no longer JP1.24
- net USBOTG_DM: now also U$16.B20; no longer JP1.18
- net USBOTG_DP: now also U$16.B19; no longer JP1.16
Other:
- board size 50 x 50 mm -> 51 x 62 mm

Commit message: Initial coven boards: A13 v0.1 card and test socket
Parts:
- removed C69: 1uF, kmod-passives:0402-CAP
- removed C77: 0.1uF/DNP, kmod-passives:0402-CAP
- removed JP2: (no value), SparkFun-Connectors:1X04
- removed LPWR: YLW, kmod-passives:0603_LED
- removed R33: 10k, kmod-passives:0603-RES
- removed R35: 330R?/DNP, kmod-passives:0603-RES
- removed S1, S2: TAC_SWITCHPTH, kmod-mechanical:TACTILE-PTH
- removed SB13, SB14, SB15, SB16, SB17, SB2: SOLDER-BRIDGEOPEN, kmod-nonparts:SOLDER-BRIDGE-OPEN
- removed U$14: AXP209, kmod-testing:QFN48
- added C85, C86: 4.7uF, kmod-passives:0603-CAP
- added C87: 0.1uF, kmod-passives:0402-CAP
- added CONN14: !NMI, kmod-nonparts:HOLE_22AWG
- added CONN15: TWI0C, kmod-nonparts:TESTPAD-1.27
- added CONN16: TWI0D, kmod-nonparts:TESTPAD-1.27
- added CONN17: RST_N, kmod-nonparts:HOLE_22AWG
- added CONN18: RX, kmod-nonparts:HOLE_22AWG
- added L10: GRN, kmod-passives:0603_LED
- added L11, L3V3: YLW, kmod-passives:0603_LED
- added SW_UBOOT, S_RESET: TAC_SWITCHSMD_4.5X4.5, kmod-mechanical:TAC_SWITCH_SMD_4.5X4.5
- C10, C11, C12, C13, C14, C15, C16, C17, C18, C19, C20, C22, C24, C26, C27, C28, C29, C30, C32, C33, C34, C35, C36, C45, C5, C53, C55, C57, C6, C61, C62, C63, C64, C65, C66, C67, C9: value 1uF/0.1uF -> 0.1uF
- C25, C31: value 1uF/0.1uF -> 1uF
- C39, C40, C41, C42: value 10pF -> 0.1uF
- C48: device kmod-passives:0402-CAP -> kmod-passives:0603-CAP
- C51: value 22uF -> 4.7uF; device kmod-passives:0805 -> kmod-passives:0603-CAP
- C70: value 1nF -> 0.1uF
- C71, C72, C73, C74: value 1uF -> 0.1uF
- C75: value 10uF -> 0.1uF; device kmod-passives:0603-CAP -> kmod-passives:0402-CAP
- C76: value 1uF -> 4.7uF; device kmod-passives:0402-CAP -> kmod-passives:0603-CAP
- CONN10: value VBUS -> TX
- CONN12: device kmod-nonparts:TESTPAD-2MM -> kmod-nonparts:TESTPAD-1.27
- CONN13: value PWR_EN -> 3V3_EN
- CONN9: value ACIN -> PRTCTL
- DDR3_1: value (none) -> x16, 96FBGA: AS4C{64/128/256}M16D3
- L6: value 2A,120R@100MHz -> DNP(2A,120R@100MHz)
- R10, R11, R18, R19, R20, R21, R22, R23, R24, R25, R3, R4, R41, R42, R44, R47, R48, R5, R6, R7, R8, R9: device kmod-passives:0402-RES -> kmod-passives:0603-RES
- R16, R46: value 470R -> 680R
- R31: value 100R -> 470R
- R32: value 200k 1% -> 470R
- SB1: value SOLDER-BRIDGEOPEN -> NMDIX
- SB10: value TRACE-CUT -> 1V5_CS; device kmod-nonparts:TRACE-CUT -> kmod-nonparts:SOLDER-BRIDGE-OPEN-LARGE
- SB11: value SOLDER-BRIDGEOPEN -> AVCC_CS; device kmod-nonparts:SOLDER-BRIDGE-OPEN -> kmod-nonparts:SOLDER-BRIDGE-OPEN-LARGE
- SB12: value SOLDER-BRIDGEOPEN -> INT_CS; device kmod-nonparts:SOLDER-BRIDGE-OPEN -> kmod-nonparts:SOLDER-BRIDGE-OPEN-LARGE
- SB3: value SOLDER-BRIDGEOPEN -> NCLKEN
- SB4: value TRACE-CUT -> CLKEN
- SB5: value SOLDER-BRIDGEOPEN -> CLKOUT
- SB6: value SOLDER-BRIDGEOPEN -> DET13
- SB7: value SOLDER-BRIDGEOPEN -> DET3; device kmod-nonparts:SOLDER-BRIDGE-OPEN -> kmod-nonparts:TRACE-CUT
- SB8: value TRACE-CUT -> 3V3_CS; device kmod-nonparts:TRACE-CUT -> kmod-nonparts:SOLDER-BRIDGE-OPEN-LARGE
- SB9: value TRACE-CUT -> CPU_CS; device kmod-nonparts:TRACE-CUT -> kmod-nonparts:SOLDER-BRIDGE-OPEN-LARGE
- moved CONN13 251.5 mm to (13.0, 15.5)
- moved R48 250.8 mm to (16.8, 15.8), turned to 180 degrees
- moved CONN12 249.9 mm to (16.4, 13.9), turned to 180 degrees
- moved U$17 249.4 mm to (14.2, 40.3)
- moved Q1 243.0 mm to (9.90, 14.7), turned to 270 degrees
- moved R46 239.8 mm to (3.10, 48.1), flipped to the bottom, turned to 180 degrees
- moved L0 239.4 mm to (3.10, 49.9), flipped to the bottom, turned to 90 degrees
- moved R47 235.3 mm to (7.10, 14.7), turned to 270 degrees
- moved R41 234.9 mm to (41.0, 35.7), flipped to the bottom
- moved D2 233.5 mm to (11.5, 32.8)
- moved C84 232.0 mm to (38.7, 34.9), flipped to the bottom, turned to 90 degrees
- moved C83 230.6 mm to (41.0, 34.2), flipped to the bottom, turned to 180 degrees
- moved R42 228.0 mm to (32.0, 12.8), flipped to the bottom, turned to 180 degrees
- moved RA14 227.9 mm to (33.7, 22.2), flipped to the bottom, turned to 90 degrees
- moved R44 225.6 mm to (13.0, 12.9), turned to 180 degrees
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Connections:
- net N$80 renamed 3.3V_FB
- net N$95 renamed VRP
- net N$97 renamed VRA1
- net PWR_EN renamed 3V3_EN
- removed net AXP209_NOE: R33.1, SB11.L1, SB11.L2, U$14.004
- removed net AXP209_VINT: C74.2, U$14.026, U$14.027
- removed net IPSOUT: C71.1, C72.1, C73.1, C75.1, C76.1, SB6.R1, SB6.R2, U$14.007, U$14.013, U$14.014, U$14.021, U$14.034, U$14.035, U$14.040, U$14.044
- removed net N$100: CONN10.P, U$14.031
- removed net N$101: R32.1, U$14.023
- removed net N$102: C70.2, U$14.047
- removed net N$103: L12V.C, R45.2
- removed net N$104: SB7.R1, SB7.R2, SB8.L1, U$14.043
- removed net N$110: R46.2
- removed net N$112: C77.1, R35.2, U$15.SHELL1, U$15.SHELL2, U$15.SHELL3, U$15.SHELL4
- removed net N$67: R16.2
- removed net N$86: S1.1, SB6.L1, SB6.L2, SB9.R1
- removed net N$87: S1.4, SB10.L1, SB11.R1, SB11.R2
- removed net N$88: SB14.R1, SB14.R2, SB16.R1, SB16.R2, U$14.015
- removed net N$89: SB15.R1, SB15.R2, SB17.R1, SB17.R2, U$14.017
- removed net N$90: R31.1, U$14.037
- removed net N$99: CONN9.P, U$14.032, U$14.033
- removed net USB3DM: U$7.003
- removed net USB3DP: U$7.004
- new net L0: R46.2, U$1.001
- new net L1: R31.2, U$1.012
- new net L2: R32.2, U$1.013
- new net LAN_VBUSDET: SB6.R1, SB6.R2, SB7.R1, U$7.011
- new net LIND: R16.2, U$1.002
- new net N$80: L3V3.A, R17.1
- new net SPI0_CLK: U$1.006, U$16.B27
- new net SPI0_CS: U$1.003, U$16.B28
- new net SPI0_MISO: U$1.007, U$16.B24
- new net SPI0_MOSI: U$1.008, U$16.B23
- new net USBH_VBUSDRV: SB6.L1, SB6.L2, U$1.014
- net 1.5V: now also C86.1, SB10.R1, SB10.R2
- net 12V: now also R45.2; no longer L12V.A
- net 3.3V: now also C51.1, C70.1, C71.1, C72.1, C73.1, R17.2, SB7.L1, SB8.R2; no longer JP2.4, LPWR.A, U$14.038, U$14.039, U$14.042, U$7.011
- net 3.3V_U: now also SB8.L1, SB8.L2; no longer C51.1
- net AVCC: now also SB11.R1, SB11.R2
- net AVCC_U: now also SB11.L1, SB11.L2; no longer U$14.012
- net GND: now also C70.2, C74.2, C85.2, C86.2, C87.2, L10.C, L11.C, L12V.C, L3V3.C, SW_UBOOT.1, S_RESET.1, U$1.P$10, U$1.P$11, U$1.P$12, U$1.P$13; no longer C69.1, C70.1, C74.1, C77.2, JP2.1, R17.1, R31.2, R32.2, R33.2, R35.1, R45.1, S2.1, SB7.L1, SB7.L2, SB9.L1, U$14.009, U$14.016, U$14.022, U$14.046, U$14.P$1, U$14.P$2, U$14.P$3, U$14.P$4, U$14.P$5, U$14.P$6, U$14.P$7, U$14.P$8, U$14.P$9, U$14.PAD
- net N$74: no longer SB2.L1, SB2.L2
- net N$75: no longer SB2.R1, SB2.R2
- net N$78: now also CONN9.P, U$7.014; no longer SB12.R1, SB12.R2, U$14.008
- net N$79: now also L10.A, R31.1; no longer SB13.R1, SB13.R2, U$14.010
- net N$82: now also L12V.A, R45.1; no longer LPWR.C, R17.2
- net N$84: now also L11.A, R32.1; no longer C69.2, U$14.024
- net NMI_N: now also CONN14.P; no longer U$14.048
- net RESET_N: now also C87.1, CONN17.P, S_RESET.4; no longer SB10.R1, U$14.025
- net SD_CLK: now also RA13.1; no longer RA13.4
- net SD_CMD: now also RA13.2; no longer RA13.3
- net SD_D2: now also RA13.4; no longer RA13.1
- net SD_D3: now also RA13.3; no longer RA13.2
- net SVR_ID0: now also RA14.4, U$1.120; no longer RA14.1
- net SVR_ID1: now also RA14.3, U$1.121; no longer RA14.2
- net SVR_ID2: now also RA14.2, U$1.122; no longer RA14.3
- net SVR_ID3: now also RA14.1, U$1.123; no longer RA14.4
- net SVR_ID4: now also U$1.124
- net TWI0-SCK: now also CONN16.P; no longer U$14.002
- net TWI0-SDA: now also CONN15.P; no longer U$14.001
- net UART1_RX: now also CONN18.P; no longer JP2.2
- net UART1_TX: now also CONN10.P; no longer JP2.3
- net UBOOT: now also SW_UBOOT.4; no longer S2.4
- net USBOTG_VBUSDRV: now also U$1.015
- net VCPU_SW: no longer SB12.L1, SB12.L2
- net VCPU_U: now also SB9.L1, SB9.L2; no longer SB13.L1, SB13.L2
- net VDDR_SW: no longer SB16.L1, SB16.L2
- net VDDR_U: now also SB10.L1, SB10.L2; no longer SB17.L1, SB17.L2
- net VDD_CPU: now also C74.1, C75.1, C76.1, SB9.R1, SB9.R2
- net VDD_INT: now also C85.1, SB12.R1, SB12.R2
- net VINT_SW: no longer SB14.L1, SB14.L2
- net VINT_U: now also SB12.L1, SB12.L2; no longer SB15.L1, SB15.L2
Routing:
- net GND: track 0.00 -> 544.8 mm, vias 0 -> 107
- net 3.3V: track 0.00 -> 168.6 mm, vias 0 -> 35
- net VDD_CPU: track 0.00 -> 98.1 mm, vias 0 -> 10
- net VDD_INT: track 0.00 -> 96.8 mm, vias 0 -> 8
- net 1.5V: track 0.00 -> 89.3 mm, vias 0 -> 26
- net TWI2_SDA: track 0.00 -> 83.8 mm, vias 0 -> 2
- net UART1_TX: track 0.00 -> 83.4 mm, vias 0 -> 2
- net TWI2_SCK: track 0.00 -> 82.3 mm, vias 0 -> 2
- net UART1_RX: track 0.00 -> 81.9 mm, vias 0 -> 2
- net SPI0_CS: track 0.00 -> 77.5 mm, vias 0 -> 2
- net SPI0_CLK: track 0.00 -> 76.8 mm, vias 0 -> 2
- net SPI0_MOSI: track 0.00 -> 76.6 mm, vias 0 -> 2
- net SPI0_MISO: track 0.00 -> 76.2 mm, vias 0 -> 2
- net USBOTG_VBUSDRV: track 0.00 -> 73.1 mm, vias 0 -> 3
- net USBOTG_VBUSDET: track 0.00 -> 66.4 mm, vias 0 -> 2
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- added copper zone on layer 15, net 1.5V
- added copper zone on layer 15, net 3.3V
- added copper zone on layer 1, net GND
- added copper zone on layer 16, net GND
- added copper zone on layer 2, net GND
- added copper zone on layer 15, net VDD_CPU
- added copper zone on layer 15, net VDD_INT
Other:
- board size 51 x 62 mm -> 56 x 62 mm
- board text added: "24/12"
- board text added: "24/18"
- board text added: "24/8"
- board text added: "30/12"
- board text added: "30/8"
- board text added: "36/12"
- board text added: "Coven A13 card v0.1 7-3-14"
- board text added: "LINK"
- board text added: "RESET"
- board text added: "UBOOT"

Commit message: working on more coven boards
Parts:
- Q1: value BSS84 -> 2N7002
- R44: value DNP(100k) -> 100k
- R47: value 100k -> 330k
- R48: value 100k -> DNP
Changed lines of the file:
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@@
 <?xml version="1.0" encoding="utf-8"?>
 <!DOCTYPE eagle SYSTEM "eagle.dtd">
-<eagle version="6.5.0">
+<eagle version="6.4">
 <drawing>
 <settings>
@@
 <setting verticaltext="up"/>
 </settings>
-<grid distance="1" unitdist="mm" unit="mm" style="lines" multiple="1" display="yes" altdistance="0.01" altunitdist="mm" altunit="mm"/>
+<grid distance="0.5" unitdist="mm" unit="mm" style="lines" multiple="1" display="yes" altdistance="0.01" altunitdist="mm" altunit="mm"/>
 <layers>
-<layer number="1" name="Top" color="4" fill="1" visible="no" active="yes"/>
+<layer number="1" name="Top" color="4" fill="1" visible="yes" active="yes"/>
 <layer number="2" name="Route2" color="20" fill="1" visible="no" active="yes"/>
 <layer number="3" name="Route3" color="4" fill="3" visible="no" active="no"/>
@@
 <layer number="19" name="Unrouted" color="6" fill="1" visible="yes" active="yes"/>
 <layer number="20" name="Dimension" color="15" fill="1" visible="yes" active="yes"/>
-<layer number="21" name="tPlace" color="16" fill="1" visible="no" active="yes"/>
+<layer number="21" name="tPlace" color="16" fill="1" visible="yes" active="yes"/>
 <layer number="22" name="bPlace" color="14" fill="1" visible="yes" active="yes"/>
-<layer number="23" name="tOrigins" color="15" fill="1" visible="no" active="yes"/>
+<layer number="23" name="tOrigins" color="15" fill="1" visible="yes" active="yes"/>
 <layer number="24" name="bOrigins" color="15" fill="1" visible="yes" active="yes"/>
-<layer number="25" name="tNames" color="7" fill="1" visible="no" active="yes"/>
+<layer number="25" name="tNames" color="7" fill="1" visible="yes" active="yes"/>
 <layer number="26" name="bNames" color="7" fill="1" visible="yes" active="yes"/>
-<layer number="27" name="tValues" color="7" fill="1" visible="no" active="yes"/>
+<layer number="27" name="tValues" color="7" fill="1" visible="yes" active="yes"/>
 <layer number="28" name="bValues" color="7" fill="1" visible="yes" active="yes"/>
 <layer number="29" name="tStop" color="7" fill="3" visible="no" active="yes"/>
-<layer number="30" name="bStop" color="7" fill="6" visible="yes" active="yes"/>
+<layer number="30" name="bStop" color="7" fill="6" visible="no" active="yes"/>
 <layer number="31" name="tCream" color="7" fill="4" visible="no" active="yes"/>
 <layer number="32" name="bCream" color="7" fill="5" visible="no" active="yes"/>
@@
 <layer number="37" name="tTest" color="7" fill="1" visible="no" active="yes"/>
 <layer number="38" name="bTest" color="7" fill="1" visible="no" active="yes"/>
-<layer number="39" name="tKeepout" color="4" fill="11" visible="no" active="yes"/>
+<layer number="39" name="tKeepout" color="4" fill="11" visible="yes" active="yes"/>
 <layer number="40" name="bKeepout" color="1" fill="11" visible="yes" active="yes"/>
-<layer number="41" name="tRestrict" color="4" fill="10" visible="no" active="yes"/>
+<layer number="41" name="tRestrict" color="4" fill="10" visible="yes" active="yes"/>
 <layer number="42" name="bRestrict" color="1" fill="10" visible="yes" active="yes"/>
 <layer number="43" name="vRestrict" color="2" fill="10" visible="yes" active="yes"/>
@@
 <layer number="49" name="Reference" color="7" fill="1" visible="yes" active="yes"/>
 <layer number="50" name="dxf" color="7" fill="1" visible="no" active="no"/>
-<layer number="51" name="tDocu" color="6" fill="1" visible="no" active="yes"/>
+<layer number="51" name="tDocu" color="6" fill="1" visible="yes" active="yes"/>
 <layer number="52" name="bDocu" color="7" fill="1" visible="yes" active="yes"/>
 <layer number="53" name="tGND_GNDA" color="7" fill="9" visible="no" active="no"/>
@@
 <layer number="220" name="220bmp" color="21" fill="1" visible="no" active="no"/>
 <layer number="221" name="221bmp" color="22" fill="1" visible="no" active="no"/>
-<layer number="222" name="222bmp" color="23" fill="1" visible="no" active="no"/>
 <layer number="223" name="223bmp" color="24" fill="1" visible="no" active="no"/>
 <layer number="224" name="224bmp" color="25" fill="1" visible="no" active="no"/>
@@
 </element>
 <element name="D1" library="kmod-discretesemi" package="SOD-523" value="RB521S30" x="14.16" y="36.5"/>
-<element name="R44" library="kmod-passives" package="0603-RES" value="DNP(100k)" x="12.98" y="12.9" rot="R180">
+<element name="R44" library="kmod-passives" package="0603-RES" value="100k" x="12.98" y="12.9" rot="R180">
 <attribute name="PACKAGE" value="0603" x="12.98" y="12.9" size="1.778" layer="27" rot="R180" display="off"/>
 </element>
@@
 <element name="L0" library="kmod-passives" package="0603_LED" value="WHT" x="3.1" y="49.9" rot="MR90"/>
 <element name="U$17" library="kmod-ics" package="SOT23-3" value="RT9818C-29GV" x="14.16" y="40.28"/>
-<element name="R47" library="kmod-passives" package="0603-RES" value="100k" x="7.1" y="14.7" rot="R270">
+<element name="R47" library="kmod-passives" package="0603-RES" value="330k" x="7.1" y="14.7" rot="R270">
 <attribute name="PACKAGE" value="0603" x="7.1" y="14.7" size="1.778" layer="27" rot="R270" display="off"/>
 </element>
-<element name="Q1" library="SparkFun-DiscreteSemi" package="SOT23-3" value="BSS84" x="9.9" y="14.7" rot="R270"/>
-<element name="R48" library="kmod-passives" package="0603-RES" value="100k" x="16.8" y="15.8" rot="R180">
+<element name="Q1" library="SparkFun-DiscreteSemi" package="SOT23-3" value="2N7002" x="9.9" y="14.7" rot="R270"/>
+<element name="R48" library="kmod-passives" package="0603-RES" value="DNP" x="16.8" y="15.8" rot="R180">
 <attribute name="PACKAGE" value="0603" x="16.8" y="15.8" size="1.778" layer="27" rot="R180" display="off"/>
 </element>
@@
 </signal>
 </signals>
-<errors>
-</errors>
 </board>
 </drawing>
