File: coven/a13_v0.1/board.brd (EAGLE design)
At the start: 56 x 62 mm, 209 parts, among them IC1 256/512 x 8bit, Q1 2N7002, Y1 24MHz, Y2 25MHz

Commit message: More work on coven boards (mostly old stuff I forgot to check in)
Parts:
- C43, C44, C50, C58, C59, C60, C79: device kmod-passives:0805 -> kmod-passives:0805-CAP
- L3V3: value YLW -> GRN
- R16, R46: value 680R -> 1k
- R17: value 330R -> 680R
- R45: value 2.2k -> 4.7k
Changed lines of the file:
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@@
 <?xml version="1.0" encoding="utf-8"?>
 <!DOCTYPE eagle SYSTEM "eagle.dtd">
-<eagle version="6.4">
+<eagle version="6.5.0">
 <drawing>
 <settings>
@@
 <grid distance="0.5" unitdist="mm" unit="mm" style="lines" multiple="1" display="yes" altdistance="0.01" altunitdist="mm" altunit="mm"/>
 <layers>
-<layer number="1" name="Top" color="4" fill="1" visible="yes" active="yes"/>
+<layer number="1" name="Top" color="4" fill="1" visible="no" active="yes"/>
 <layer number="2" name="Route2" color="20" fill="1" visible="no" active="yes"/>
 <layer number="3" name="Route3" color="4" fill="3" visible="no" active="no"/>
@@
 <layer number="19" name="Unrouted" color="6" fill="1" visible="yes" active="yes"/>
 <layer number="20" name="Dimension" color="15" fill="1" visible="yes" active="yes"/>
-<layer number="21" name="tPlace" color="16" fill="1" visible="yes" active="yes"/>
+<layer number="21" name="tPlace" color="16" fill="1" visible="no" active="yes"/>
 <layer number="22" name="bPlace" color="14" fill="1" visible="yes" active="yes"/>
-<layer number="23" name="tOrigins" color="15" fill="1" visible="yes" active="yes"/>
+<layer number="23" name="tOrigins" color="15" fill="1" visible="no" active="yes"/>
 <layer number="24" name="bOrigins" color="15" fill="1" visible="yes" active="yes"/>
-<layer number="25" name="tNames" color="7" fill="1" visible="yes" active="yes"/>
+<layer number="25" name="tNames" color="7" fill="1" visible="no" active="yes"/>
 <layer number="26" name="bNames" color="7" fill="1" visible="yes" active="yes"/>
-<layer number="27" name="tValues" color="7" fill="1" visible="yes" active="yes"/>
+<layer number="27" name="tValues" color="7" fill="1" visible="no" active="yes"/>
 <layer number="28" name="bValues" color="7" fill="1" visible="yes" active="yes"/>
 <layer number="29" name="tStop" color="7" fill="3" visible="no" active="yes"/>
@@
 <layer number="37" name="tTest" color="7" fill="1" visible="no" active="yes"/>
 <layer number="38" name="bTest" color="7" fill="1" visible="no" active="yes"/>
-<layer number="39" name="tKeepout" color="4" fill="11" visible="yes" active="yes"/>
+<layer number="39" name="tKeepout" color="4" fill="11" visible="no" active="yes"/>
 <layer number="40" name="bKeepout" color="1" fill="11" visible="yes" active="yes"/>
-<layer number="41" name="tRestrict" color="4" fill="10" visible="yes" active="yes"/>
+<layer number="41" name="tRestrict" color="4" fill="10" visible="no" active="yes"/>
 <layer number="42" name="bRestrict" color="1" fill="10" visible="yes" active="yes"/>
 <layer number="43" name="vRestrict" color="2" fill="10" visible="yes" active="yes"/>
@@
 <layer number="49" name="Reference" color="7" fill="1" visible="yes" active="yes"/>
 <layer number="50" name="dxf" color="7" fill="1" visible="no" active="no"/>
-<layer number="51" name="tDocu" color="6" fill="1" visible="yes" active="yes"/>
+<layer number="51" name="tDocu" color="6" fill="1" visible="no" active="yes"/>
 <layer number="52" name="bDocu" color="7" fill="1" visible="yes" active="yes"/>
 <layer number="53" name="tGND_GNDA" color="7" fill="9" visible="no" active="no"/>
@@
 <layer number="220" name="220bmp" color="21" fill="1" visible="no" active="no"/>
 <layer number="221" name="221bmp" color="22" fill="1" visible="no" active="no"/>
+<layer number="222" name="222bmp" color="23" fill="1" visible="no" active="no"/>
 <layer number="223" name="223bmp" color="24" fill="1" visible="no" active="no"/>
 <layer number="224" name="224bmp" color="25" fill="1" visible="no" active="no"/>
@@
 </element>
 <element name="LLNK" library="kmod-passives" package="0603_LED" value="GRN" x="54.6" y="27.8" rot="R180"/>
-<element name="R16" library="kmod-passives" package="0603-RES" value="680R" x="3.3" y="48.3">
+<element name="R16" library="kmod-passives" package="0603-RES" value="1k" x="3.3" y="48.3">
 <attribute name="PACKAGE" value="0603" x="3.3" y="48.3" size="1.778" layer="27" display="off"/>
 </element>
@@
 <attribute name="VALUE" x="33.8" y="27.6" size="0.6096" layer="21" ratio="12" rot="R90" align="bottom-center"/>
 </element>
-<element name="R17" library="kmod-passives" package="0603-RES" value="330R" x="7.06" y="30.7">
+<element name="R17" library="kmod-passives" package="0603-RES" value="680R" x="7.06" y="30.7">
 <attribute name="PACKAGE" value="0603" x="7.06" y="30.7" size="1.778" layer="27" display="off"/>
 </element>
-<element name="L3V3" library="kmod-passives" package="0603_LED" value="YLW" x="3.08" y="30.74" rot="R90"/>
+<element name="L3V3" library="kmod-passives" package="0603_LED" value="GRN" x="3.08" y="30.74" rot="R90"/>
 <element name="U$10" library="kmod-testing" package="HTSOP8" value="BD9D321EFJ" x="12.3" y="19.8" rot="R90"/>
-<element name="C43" library="kmod-passives" package="0805" value="10uF" x="3.5" y="18.3" rot="R180">
+<element name="C43" library="kmod-passives" package="0805-CAP" value="10uF" x="3.5" y="18.3" rot="R180">
 <attribute name="VOLTAGE" value="25V" x="3.5" y="18.3" size="1.778" layer="27" rot="R180" display="off"/>
 <attribute name="PACKAGE" value="0805" x="3.5" y="18.3" size="1.778" layer="27" rot="R180" display="off"/>
 </element>
-<element name="C44" library="kmod-passives" package="0805" value="10uF" x="3.5" y="20.3" rot="R180">
+<element name="C44" library="kmod-passives" package="0805-CAP" value="10uF" x="3.5" y="20.3" rot="R180">
 <attribute name="VOLTAGE" value="25V" x="3.5" y="20.3" size="1.778" layer="27" rot="R180" display="off"/>
 <attribute name="PACKAGE" value="0805" x="3.5" y="20.3" size="1.778" layer="27" rot="R180" display="off"/>
@@
 <attribute name="PACKAGE" value="0603" x="14.5" y="24.5" size="1.778" layer="27" display="off"/>
 </element>
-<element name="C50" library="kmod-passives" package="0805" value="22uF" x="10.5" y="24.5">
+<element name="C50" library="kmod-passives" package="0805-CAP" value="22uF" x="10.5" y="24.5">
 <attribute name="VOLTAGE" value="6.3V" x="10.5" y="24.5" size="1.778" layer="27" display="off"/>
 <attribute name="PACKAGE" value="0805" x="10.5" y="24.5" size="1.778" layer="27" display="off"/>
@@
 <variant name="test" populate="no"/>
 </element>
-<element name="C58" library="kmod-passives" package="0805" value="22uF" x="9.5" y="18.5" rot="MR270">
+<element name="C58" library="kmod-passives" package="0805-CAP" value="22uF" x="9.5" y="18.5" rot="MR270">
 <attribute name="VOLTAGE" value="6.3V" x="9.5" y="18.5" size="1.778" layer="28" rot="MR270" display="off"/>
 <attribute name="PACKAGE" value="0805" x="9.5" y="18.5" size="1.778" layer="28" rot="MR270" display="off"/>
 </element>
-<element name="C59" library="kmod-passives" package="0805" value="22uF" x="27.5" y="19" rot="MR270">
+<element name="C59" library="kmod-passives" package="0805-CAP" value="22uF" x="27.5" y="19" rot="MR270">
 <attribute name="VOLTAGE" value="6.3V" x="27.5" y="19" size="1.778" layer="28" rot="MR270" display="off"/>
 <attribute name="PACKAGE" value="0805" x="27.5" y="19" size="1.778" layer="28" rot="MR270" display="off"/>
 </element>
-<element name="C60" library="kmod-passives" package="0805" value="22uF" x="9.28" y="31.62" rot="MR270">
+<element name="C60" library="kmod-passives" package="0805-CAP" value="22uF" x="9.28" y="31.62" rot="MR270">
 <attribute name="VOLTAGE" value="6.3V" x="9.28" y="31.62" size="1.778" layer="28" rot="MR270" display="off"/>
 <attribute name="PACKAGE" value="0805" x="9.28" y="31.62" size="1.778" layer="28" rot="MR270" display="off"/>
@@
 <attribute name="PACKAGE" value="0603" x="34.3" y="51.54" size="1.778" layer="28" rot="MR0" display="off"/>
 </element>
-<element name="C79" library="kmod-passives" package="0805" value="22uF" x="31.971271875" y="54.341621875" rot="MR0">
+<element name="C79" library="kmod-passives" package="0805-CAP" value="22uF" x="31.971271875" y="54.341621875" rot="MR0">
 <attribute name="PACKAGE" value="0805" x="31.971271875" y="54.341621875" size="1.778" layer="28" rot="MR0" display="off"/>
 <attribute name="VOLTAGE" value="6.3V" x="31.971271875" y="54.341621875" size="1.778" layer="28" rot="MR0" display="off"/>
@@
 <attribute name="PACKAGE" value="0603" x="12.98" y="12.9" size="1.778" layer="27" rot="R180" display="off"/>
 </element>
-<element name="R45" library="kmod-passives" package="0603-RES" value="2.2k" x="3.1" y="15.5" rot="R90">
+<element name="R45" library="kmod-passives" package="0603-RES" value="4.7k" x="3.1" y="15.5" rot="R90">
 <attribute name="PACKAGE" value="0603" x="-0.9" y="15.5" size="1.778" layer="27" rot="R90" display="off"/>
 </element>
 <element name="L12V" library="kmod-passives" package="0603_LED" value="YLW" x="1.6" y="15.5"/>
 <element name="D2" library="kmod-discretesemi" package="SOD-523" value="RB521S30" x="11.54" y="32.8"/>
-<element name="R46" library="kmod-passives" package="0603-RES" value="680R" x="3.1" y="48.1" rot="MR180">
+<element name="R46" library="kmod-passives" package="0603-RES" value="1k" x="3.1" y="48.1" rot="MR180">
 <attribute name="PACKAGE" value="0603" x="3.1" y="44.1" size="1.778" layer="28" rot="MR180" display="off"/>
 </element>
