File: coven/a13_v0.1/board.sch (EAGLE design)
At the start: 169 parts, among them IC1 256/512 x 8bit, Y1 24MHz, Y2 25MHz

Commit message: work continues on coven boards
Parts:
- added C77: 0.1uF, kmod-passives:CAP0402-CAP
- added C78: 10uF, kmod-passives:CAP0603
- added C79: 22uF, kmod-passives:CAP0805
- added D3: PMEG2010AEB, SparkFun-DiscreteSemi:DIODE-SCHOTTKY
- added L9: CIC10J601(750mA,600R), kmod-passives:INDUCTOR0603
- added R35: 330R, kmod-passives:RESISTOR0603
- added R36: 10k, kmod-passives:RESISTOR0603
- added R37, R38, R39: 47k, kmod-passives:RESISTOR0603
- added RA13: 47k, kmod-passives:RESISTOR_ARRAY0603_X4
- added SB12, SB13, SB14, SB15, SB16, SB17: SOLDER-BRIDGEOPEN, kmod-nonparts:SOLDER-BRIDGEOPEN
- added U$15: Molex 1050270001, kmod-connectors:MICROSDMOLEX-1050270001
Connections:
- removed net AXP209_IRQ: U$14.IRQ
- removed net AXP209_SCK: U$14.SCK
- removed net AXP209_SDA: U$14.SDA
- new net N$108: C78.1, C79.1, L9.2, U$15.VDD
- new net N$112: C77.1, R35.2, U$15.SHELL
- new net N$78: SB12.P$2, U$14.LX2
- new net N$89: SB15.P$2, SB17.P$2, U$14.DCDC3
- new net NMI_N: R39.1, U$1.158/NMI_N, U$14.IRQ
- new net SD_CD: R36.2, U$1.155/PG0/EINT0, U$15.SWITCH
- new net SD_CLK: RA13D.1, U$1.110/SDC0_CLK/PF2, U$15.CLK
- new net SD_CMD: RA13C.1, U$1.111/SDC0_CMD/PF3, U$15.CMD/DI
- new net SD_D0: R38.1, U$1.108/SDC0_D0/PF1, U$15.DAT0/DO
- new net SD_D1: R37.1, U$1.107/SDC0_D1/PF0, U$15.DAT1/RSV
- new net SD_D2: RA13A.1, U$1.113/SDC0_D2/PF5, U$15.DAT2/NC
- new net SD_D3: RA13B.1, U$1.112/SDC0_D3/PF4, U$15.CD/DAT3/CS
- new net TWI0-SCK: U$1.101/TWI0-SCK/PB0, U$14.SCK
- new net TWI0-SDA: U$1.102/TWI0-SDA/PB1, U$14.SDA
- new net VDDR_SW: L5.1, SB16.P$1, U$12.SW
- new net VDDR_U: C60.1, L5.2, R22.2, R26.2, SB17.P$1
- net 3.3V: now also L9.1, R37.2, R38.2, RA13A.2, RA13B.2, RA13C.2, RA13D.2
- net GND: now also C77.2, C78.2, C79.2, R35.1, R36.1, U$15.VSS
- net N$79: now also SB13.P$2, U$14.DCDC2; no longer L5.1, U$12.SW
- net N$88: now also SB14.P$2, SB16.P$2, U$14.LX3; no longer C60.1, L5.2, R22.2, R26.2
- net N$93: now also R39.2; no longer U$1.158/NMI_N
- net VCPU_SW: now also SB12.P$1; no longer U$14.LX2
- net VCPU_U: now also SB13.P$1; no longer U$14.DCDC2
- net VINT_SW: now also SB14.P$1; no longer U$14.LX3
- net VINT_U: now also SB15.P$1; no longer U$14.DCDC3
Other:
- note added: "Not sure if this can be grounded or if it needs to be"
- note added: "Pick one pair and close for AXP mode"
- note added: "close for AXP mode"
- moved on the sheet: C60, L5, R22, R23, R26, R34

Commit message: more work on coven
Parts:
- removed D3: PMEG2010AEB, SparkFun-DiscreteSemi:DIODE-SCHOTTKY
- removed JP1: M13X22X13, SparkFun-Connectors:M13X22X13
- added C80, C84: 0.1uF, kmod-passives:CAP0402-CAP
- added C81, C83: 10uF, kmod-passives:CAP0603
- added C82: 1uF, kmod-passives:CAP0402-CAP
- added CONN11: UBOOT, kmod-nonparts:CONNECTOR22AWG
- added CONN12: PWR_ON#, kmod-nonparts:CONNECTOR2MM
- added CONN13: PWR_EN, kmod-nonparts:CONNECTOR2MM
- added D2: RB521S30, kmod-discretesemi:DIODE-SCHOTTKYSOD523
- added D4: B5819WS, kmod-discretesemi:DIODE-SCHOTTKYSOD323
- added D6: PMEG2010AEB, kmod-discretesemi:DIODE-SCHOTTKYSOD523
- added L0: WHT, kmod-passives:LED0603
- added L12V: YLW, kmod-passives:LED0603
- added Q1: BSS84, SparkFun-DiscreteSemi:MOSFET-PCHANNELSMD
- added R40: 100k, kmod-passives:RESISTOR0603
- added R41: 200k 1%, kmod-passives:RESISTOR0402
- added R42: 10k, kmod-passives:RESISTOR0402
- added R44: DNP(100k), kmod-passives:RESISTOR0402
- added R45: 2.2k, kmod-passives:RESISTOR0603
- added R46: 470R, kmod-passives:RESISTOR0603
- added R47, R48: 100k, kmod-passives:RESISTOR0402
- added RA14: 10k, kmod-passives:RESISTOR_ARRAY0603_X4
- added S2: TAC_SWITCHPTH, kmod-mechanical:TAC_SWITCHPTH
- added U$16: CVN-V1EDGE, kmod-connectors:CVN-V1EDGE
- added U$17: RT9818C-29GV, kmod-ics:POR_ACTIVE_LOW
- C43, C44, C45: VOLTAGE (none) -> 25V
- C48: VOLTAGE (none) -> 10V
- C77: value 0.1uF -> 0.1uF/DNP
- D1: value PMEG2010AEB -> RB521S30; device SparkFun-DiscreteSemi:DIODE-SCHOTTKY -> kmod-discretesemi:DIODE-SCHOTTKYSOD523
- R35: value 330R -> 330R?/DNP
Connections:
- net N$91 renamed 3.3V_U
- new net N$103: L12V.C, R45.2
- new net N$109: L0.A, R46.1
- new net N$110: R46.2
- new net PRSNT#: U$16.GND/PRSNT2#, U$16.PRSNT#
- new net PWR_EN: CONN13.P, Q1.D, R48.2, U$10.EN
- new net PWR_ON#: CONN12.P, Q1.G, R44.2, R47.1, U$16.PWR_ON#
- new net SVR_ID0: RA14A.1, U$16.SVR_ID0
- new net SVR_ID1: RA14B.1, U$16.SVR_ID1
- new net SVR_ID2: RA14C.1, U$16.SVR_ID2
- new net SVR_ID3: RA14D.1, U$16.SVR_ID3
- new net SVR_ID4: R42.1, U$16.GND/SVR_ID4
- new net TWI2_SCK: U$1.160/TWI2_SCK/PB18, U$16.I2C_SCL
- new net TWI2_SDA: U$1.161/TWI2_SDA/PB17, U$16.I2C_SDA
- new net UBOOT: CONN11.P, D2.A, R40.1, S2.4, U$1.157/UBOOT
- new net USBOTG_IDDET: U$1.153/PG2/EINT2, U$16.L1_N
- new net USBOTG_VBUSDET: U$1.154/PG1/EINT1, U$16.L1_P
- new net USBOTG_VBUSDRV: U$16.L0_N
- new net VRA2: C83.1, C84.1, R41.2, U$1.082/VRA2
- net 12V: now also L12V.A, Q1.S, R47.2, U$16.12V@1, U$16.12V@2, U$16.12V@3, U$16.12V@4, U$16.12V@5; no longer JP1.4, JP1.6, U$10.EN
- net 3.3V: now also D4.A, D6.A, R40.2, R42.2, RA14A.2, RA14B.2, RA14C.2, RA14D.2, U$17.VDD; no longer D1.A
- net ETH_RXN: now also U$16.ETH0_RX_N; no longer JP1.10
- net ETH_RXP: now also U$16.ETH0_RX_P; no longer JP1.8
- net ETH_TXN: now also U$16.ETH0_TX_N; no longer JP1.13
- net ETH_TXP: now also U$16.ETH0_TX_P; no longer JP1.11
- net GND: now also C80.1, C81.1, C82.1, C83.2, C84.2, L0.C, R41.1, R44.1, R45.1, R48.1, S2.1, U$16.GND@1, U$16.GND@10, U$16.GND@11, U$16.GND@12, U$16.GND@13, U$16.GND@14, U$16.GND@15, U$16.GND@16, U$16.GND@17, U$16.GND@18, U$16.GND@19, U$16.GND@2, U$16.GND@20, U$16.GND@21, U$16.GND@22, U$16.GND@23, U$16.GND@24, U$16.GND@25, U$16.GND@26, U$16.GND@27, U$16.GND@28, U$16.GND@29, U$16.GND@3, U$16.GND@30, U$16.GND@31, U$16.GND@32, U$16.GND@33, U$16.GND@34, U$16.GND@35, U$16.GND@36, U$16.GND@37, U$16.GND@38, U$16.GND@39, U$16.GND@40, U$16.GND@5, U$16.GND@6, U$16.GND@7, U$16.GND@8, U$16.GND@9, U$17.GND
- net N$92: now also D1.C, U$16.SYS_RESET#; no longer U$1.157/UBOOT
- net N$93: now also D4.C
- net N$95: now also C80.2, C81.2
- net N$96: now also D2.C, U$16.L0_P; no longer U$1.082/VRA2
- net N$97: now also C82.2
- net N$98: now also D6.C; no longer D1.C
- net RESET_N: now also D1.A, U$17.N_RESET
- net UART1_RX: now also U$16.COM_RX; no longer JP1.5
- net UART1_TX: now also U$16.COM_TX; no longer JP1.3
- net USB2DM: now also U$16.USB_N; no longer JP1.21
- net USB2DP: now also U$16.USB_P; no longer JP1.19
- net USB3DM: no longer JP1.26
- net USB3DP: no longer JP1.24
- net USBOTG_DM: now also U$16.L3_N; no longer JP1.18
- net USBOTG_DP: now also U$16.L3_P; no longer JP1.16
Other:
- note added: "2.9V threshold, 220ms delay"
- moved on the sheet: C32, C33, C34, C35, C36, C43, C44, C45, JP2, R34, R39, S1

Commit message: Initial coven boards: A13 v0.1 card and test socket
Parts:
- removed C69: 1uF, kmod-passives:CAP0402-CAP
- removed C77: 0.1uF/DNP, kmod-passives:CAP0402-CAP
- removed JP2: (no value), SparkFun-Connectors:M04PTH
- removed LPWR: YLW, kmod-passives:LED0603
- removed R33: 10k, kmod-passives:RESISTOR0603
- removed R35: 330R?/DNP, kmod-passives:RESISTOR0603
- removed S1, S2: TAC_SWITCHPTH, kmod-mechanical:TAC_SWITCHPTH
- removed SB13, SB14, SB15, SB16, SB17, SB2: SOLDER-BRIDGEOPEN, kmod-nonparts:SOLDER-BRIDGEOPEN
- removed U$14: AXP209, kmod-testing:AXP209
- added C85, C86: 4.7uF, kmod-passives:CAP0603
- added C87: 0.1uF, kmod-passives:CAP0402-CAP
- added CONN14: !NMI, kmod-nonparts:CONNECTOR22AWG
- added CONN15: TWI0C, kmod-nonparts:CONNECTOR1.27
- added CONN16: TWI0D, kmod-nonparts:CONNECTOR1.27
- added CONN17: RST_N, kmod-nonparts:CONNECTOR22AWG
- added CONN18: RX, kmod-nonparts:CONNECTOR22AWG
- added L10: GRN, kmod-passives:LED0603
- added L11, L3V3: YLW, kmod-passives:LED0603
- added SW_UBOOT, S_RESET: TAC_SWITCHSMD_4.5X4.5, kmod-mechanical:TAC_SWITCHSMD_4.5X4.5
- C10, C11, C12, C13, C14, C15, C16, C17, C18, C19, C20, C22, C24, C26, C27, C28, C29, C30, C32, C33, C34, C35, C36, C45, C5, C53, C55, C57, C6, C61, C62, C63, C64, C65, C66, C67, C9: value 1uF/0.1uF -> 0.1uF
- C25, C31: value 1uF/0.1uF -> 1uF
- C39, C40, C41, C42: value 10pF -> 0.1uF; VOLTAGE (none) -> 10V
- C46: VOLTAGE (none) -> 10V
- C48: device kmod-passives:CAP0402-CAP -> kmod-passives:CAP0603
- C51: value 22uF -> 4.7uF; device kmod-passives:CAP0805 -> kmod-passives:CAP0603
- C70: value 1nF -> 0.1uF
- C71, C72, C73, C74: value 1uF -> 0.1uF
- C75: value 10uF -> 0.1uF; device kmod-passives:CAP0603 -> kmod-passives:CAP0402-CAP
- C76: value 1uF -> 4.7uF; device kmod-passives:CAP0402-CAP -> kmod-passives:CAP0603
- CONN10: value VBUS -> TX
- CONN12: device kmod-nonparts:CONNECTOR2MM -> kmod-nonparts:CONNECTOR1.27
- CONN13: value PWR_EN -> 3V3_EN
- CONN9: value ACIN -> PRTCTL
- DDR3_1: value (none) -> x16, 96FBGA: AS4C{64/128/256}M16D3
- L6: value 2A,120R@100MHz -> DNP(2A,120R@100MHz)
- R10, R11, R18, R19, R20, R21, R22, R23, R24, R25, R3, R4, R41, R42, R44, R47, R48, R5, R6, R7, R8, R9: device kmod-passives:RESISTOR0402 -> kmod-passives:RESISTOR0603
- R16, R46: value 470R -> 680R
- R31: value 100R -> 470R
- R32: value 200k 1% -> 470R
- SB1: value SOLDER-BRIDGEOPEN -> NMDIX
- SB10: value TRACE-CUT -> 1V5_CS; device kmod-nonparts:TRACE-CUT -> kmod-nonparts:SOLDER-BRIDGEOPEN-WIDE
- SB11: value SOLDER-BRIDGEOPEN -> AVCC_CS; device kmod-nonparts:SOLDER-BRIDGEOPEN -> kmod-nonparts:SOLDER-BRIDGEOPEN-WIDE
- SB12: value SOLDER-BRIDGEOPEN -> INT_CS; device kmod-nonparts:SOLDER-BRIDGEOPEN -> kmod-nonparts:SOLDER-BRIDGEOPEN-WIDE
- SB3: value SOLDER-BRIDGEOPEN -> NCLKEN
- SB4: value TRACE-CUT -> CLKEN
- SB5: value SOLDER-BRIDGEOPEN -> CLKOUT
- SB6: value SOLDER-BRIDGEOPEN -> DET13
- SB7: value SOLDER-BRIDGEOPEN -> DET3; device kmod-nonparts:SOLDER-BRIDGEOPEN -> kmod-nonparts:TRACE-CUT
- SB8: value TRACE-CUT -> 3V3_CS; device kmod-nonparts:TRACE-CUT -> kmod-nonparts:SOLDER-BRIDGEOPEN-WIDE
- SB9: value TRACE-CUT -> CPU_CS; device kmod-nonparts:TRACE-CUT -> kmod-nonparts:SOLDER-BRIDGEOPEN-WIDE
Connections:
- net N$80 renamed 3.3V_FB
- net N$95 renamed VRP
- net N$97 renamed VRA1
- net PWR_EN renamed 3V3_EN
- removed net AXP209_NOE: R33.1, SB11.P$1, U$14.N_OE
- removed net AXP209_VINT: C74.2, U$14.LDO1SET, U$14.VINT
- removed net IPSOUT: C71.1, C72.1, C73.1, C75.1, C76.1, SB6.P$2, U$14.APS, U$14.LDO24IN, U$14.LDO3IN, U$14.PS1, U$14.PS2, U$14.VIN1, U$14.VIN2, U$14.VIN3
- removed net N$100: CONN10.P, U$14.VBUS
- removed net N$101: R32.1, U$14.BIAS
- removed net N$102: C70.2, U$14.PWRON
- removed net N$103: L12V.C, R45.2
- removed net N$104: SB7.P$2, SB8.P$1, U$14.CHSENSE
- removed net N$110: R46.2
- removed net N$112: C77.1, R35.2, U$15.SHELL
- removed net N$67: R16.2
- removed net N$86: S1.1, SB6.P$1, SB9.P$2
- removed net N$87: S1.4, SB10.P$1, SB11.P$2
- removed net N$88: SB14.P$2, SB16.P$2, U$14.LX3
- removed net N$89: SB15.P$2, SB17.P$2, U$14.DCDC3
- removed net N$90: R31.1, U$14.TS
- removed net N$99: CONN9.P, U$14.ACIN1, U$14.ACIN2
- removed net USB3DM: U$7.USBDM3
- removed net USB3DP: U$7.USBDP3
- new net L0: R46.2, U$1.001/NRE/PC5
- new net L1: R31.2, U$1.012/PG9/VDD3_CPU/SPI1_CS0/UART3_TX/EINT9
- new net L2: R32.2, U$1.013/PG10/SPI1_CLK/UART3_RX/EINT10
- new net LAN_VBUSDET: SB6.P$2, SB7.P$2, U$7.VBUS_DET
- new net LIND: R16.2, U$1.002/NCE0/PC4
- new net N$80: L3V3.A, R17.1
- new net SPI0_CLK: U$1.006/NCLE/SPI0_CLK/PC2, U$16.L7_P
- new net SPI0_CS: U$1.003/NCE1/SPI0_CS0/PC3, U$16.L7_N
- new net SPI0_MISO: U$1.007/NALE/SPI0_MISO/PC1, U$16.L5_N
- new net SPI0_MOSI: U$1.008/NWE/SPI0_MOSI/PC0, U$16.L5_P
- new net USBH_VBUSDRV: SB6.P$1, U$1.014/PG11/SPI1_MOSI/UART3_CTS/EINT11
- net 1.5V: now also C86.1, SB10.P$2
- net 12V: now also R45.2; no longer L12V.A
- net 3.3V: now also C51.1, C70.1, C71.1, C72.1, C73.1, R17.2, SB7.P$1; no longer JP2.4, LPWR.A, U$14.BAT1, U$14.BAT2, U$14.BATSENSE, U$7.VBUS_DET
- net 3.3V_U: now also SB8.P$1; no longer C51.1
- net AVCC: now also SB11.P$2
- net AVCC_U: now also SB11.P$1; no longer U$14.LDO2
- net GND: now also C70.2, C74.2, C85.2, C86.2, C87.2, L10.C, L11.C, L12V.C, L3V3.C, SW_UBOOT.1, S_RESET.1; no longer C69.1, C70.1, C74.1, C77.2, JP2.1, R17.1, R31.2, R32.2, R33.2, R35.1, R45.1, S2.1, SB7.P$1, SB9.P$1, U$14.AGND, U$14.PGND1, U$14.PGND2, U$14.PGND3, U$14.THERMAL
- net N$74: no longer SB2.P$1
- net N$75: no longer SB2.P$2
- net N$78: now also CONN9.P, U$7.PRTCTL2; no longer SB12.P$2, U$14.LX2
- net N$79: now also L10.A, R31.1; no longer SB13.P$2, U$14.DCDC2
- net N$82: now also L12V.A, R45.1; no longer LPWR.C, R17.2
- net N$84: now also L11.A, R32.1; no longer C69.2, U$14.VREF
- net NMI_N: now also CONN14.P; no longer U$14.IRQ
- net RESET_N: now also C87.1, CONN17.P, S_RESET.4; no longer SB10.P$2, U$14.PWROK
- net SD_CLK: now also RA13A.1; no longer RA13D.1
- net SD_CMD: now also RA13B.1; no longer RA13C.1
- net SD_D2: now also RA13D.1; no longer RA13A.1
- net SD_D3: now also RA13C.1; no longer RA13B.1
- net SVR_ID0: now also RA14D.1, U$1.120/CSI_D2/SDC2_D2/PE6; no longer RA14A.1
- net SVR_ID1: now also RA14C.1, U$1.121/CSI_D3/SDC2_D3/PE7; no longer RA14B.1
- net SVR_ID2: now also RA14B.1, U$1.122/CSI_D4/SDC2_CMD/PE8; no longer RA14C.1
- net SVR_ID3: now also RA14A.1, U$1.123/CSI_D5/SDC2_CLK/PE9; no longer RA14D.1
- net SVR_ID4: now also U$1.124/CSI_D6/UART1_TX/PE10
- net TWI0-SCK: now also CONN16.P; no longer U$14.SCK
- net TWI0-SDA: now also CONN15.P; no longer U$14.SDA
- net UART1_RX: now also CONN18.P; no longer JP2.2
- net UART1_TX: now also CONN10.P; no longer JP2.3
- net UBOOT: now also SW_UBOOT.4; no longer S2.4
- net USBOTG_VBUSDRV: now also U$1.015/PG12/SPI1_MISO/UART3_RTS/EINT12
- net VCPU_SW: no longer SB12.P$1
- net VCPU_U: now also SB9.P$1; no longer SB13.P$1
- net VDDR_SW: no longer SB16.P$1
- net VDDR_U: now also SB10.P$1; no longer SB17.P$1
- net VDD_CPU: now also C74.1, C75.1, C76.1, SB9.P$2
- net VDD_INT: now also C85.1, SB12.P$2
- net VINT_SW: no longer SB14.P$1
- net VINT_U: now also SB12.P$1; no longer SB15.P$1
Other:
- note added: "(1A diode is overprovisioned; should be 200mA max and probably much less)"
- note added: "not 100% sure what the voltages need to be on these; I think 6.3V is ok"
- note removed: "(1A is overprovisioned; should be 200mA max and probably much less)"
- note removed: "(\!AXP209)"
- note removed: "Not sure if this can be grounded or if it needs to be"
- note removed: "Pick one pair and close for AXP mode"
- note removed: "To have the AXP209 handle resets, switch all 4 of these nodes"
- note removed: "close for AXP mode"
- moved on the sheet: C24, C25, C26, C27, C28, C29, C30, C31, C37, C38, C51, C70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

Commit message: working on more coven boards
Parts:
- Q1: value BSS84 -> 2N7002
- R44: value DNP(100k) -> 100k
- R47: value 100k -> 330k
- R48: value 100k -> DNP
Other:
- note added: "DNP R47 to have card default to on"
- note added: "This section is all wrong and requires the following modifications: - populate Q1 with 2N7002 N-channel instead of the P-channel as specified; make sure it is G-S-D pinout - instead of using R48 to pull down to ground, add a 100k resistor that pulls up to 12V -- another option is to connect R48 to 12V instead of GND but I think the extra resistor is easier"
- moved on the sheet: CONN12

Commit message: More work on coven boards (mostly old stuff I forgot to check in)
Parts:
- L3V3: value YLW -> GRN
- R16, R46: value 680R -> 1k
- R17: value 330R -> 680R
- R45: value 2.2k -> 4.7k
Changed lines of the file:
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@@
 <?xml version="1.0" encoding="utf-8"?>
 <!DOCTYPE eagle SYSTEM "eagle.dtd">
-<eagle version="6.4">
+<eagle version="6.5.0">
 <drawing>
 <settings>
@@
 <part name="LLNK" library="kmod-passives" deviceset="LED" device="0603" value="GRN"/>
 <part name="SUPPLY8" library="kmod-nonparts" deviceset="3.3V" device=""/>
-<part name="R16" library="kmod-passives" deviceset="RESISTOR" device="0603" value="680R"/>
+<part name="R16" library="kmod-passives" deviceset="RESISTOR" device="0603" value="1k"/>
 <part name="LIND" library="kmod-passives" deviceset="LED" device="0603" value="BLU"/>
 <part name="GND22" library="kmod-nonparts" deviceset="GND" device=""/>
@@
 <part name="SB5" library="kmod-nonparts" deviceset="SOLDER-BRIDGE" device="OPEN" value="CLKOUT"/>
 <part name="SUPPLY11" library="kmod-nonparts" deviceset="3.3V" device=""/>
-<part name="R17" library="kmod-passives" deviceset="RESISTOR" device="0603" value="330R"/>
-<part name="L3V3" library="kmod-passives" deviceset="LED" device="0603" value="YLW"/>
+<part name="R17" library="kmod-passives" deviceset="RESISTOR" device="0603" value="680R"/>
+<part name="L3V3" library="kmod-passives" deviceset="LED" device="0603" value="GRN"/>
 <part name="GND25" library="kmod-nonparts" deviceset="GND" device=""/>
 <part name="SUPPLY12" library="kmod-nonparts" deviceset="3.3V" device=""/>
@@
 <part name="R44" library="kmod-passives" deviceset="RESISTOR" device="0603" value="100k"/>
 <part name="GND70" library="kmod-nonparts" deviceset="GND" device=""/>
-<part name="R45" library="kmod-passives" deviceset="RESISTOR" device="0603" value="2.2k"/>
+<part name="R45" library="kmod-passives" deviceset="RESISTOR" device="0603" value="4.7k"/>
 <part name="L12V" library="kmod-passives" deviceset="LED" device="0603" value="YLW"/>
 <part name="GND71" library="kmod-nonparts" deviceset="GND" device=""/>
@@
 <part name="GND107" library="kmod-nonparts" deviceset="GND" device=""/>
 <part name="GND109" library="kmod-nonparts" deviceset="GND" device=""/>
-<part name="R46" library="kmod-passives" deviceset="RESISTOR" device="0603" value="680R"/>
+<part name="R46" library="kmod-passives" deviceset="RESISTOR" device="0603" value="1k"/>
 <part name="L0" library="kmod-passives" deviceset="LED" device="0603" value="WHT"/>
 <part name="GND110" library="kmod-nonparts" deviceset="GND" device=""/>
