File: coven/backplane_x5_v0.1/board.brd (EAGLE design)
At the start: 100 x 100 mm, 142 parts

Commit message: More work on coven boards (mostly old stuff I forgot to check in)
Parts:
- removed C20, C21: 0.1uF, kmod-passives:0402-CAP
- removed CONN10: RST, kmod-nonparts:TESTPAD-1.27
- removed CONN8: PWR, kmod-nonparts:TESTPAD-1.27
- removed CONN9: PRSNT, kmod-nonparts:TESTPAD-1.27
- removed LED3_4: YLW, kmod-passives:0603_LED
- removed R1, R11, R13, R14, R2, R3, R4, R5, R6, R7, R8, R9: 0.01R, kmod-passives:0603-RES
- removed U$1: DF40-90RCP, kmod-connectors:DF40-RCP-90
- removed U$16, U$4, U$5: M04X2, SparkFun-Connectors:2X4
- removed U$17: DF40-80RCP, kmod-connectors:DF40-RCP-80
- added C16: 1uF, kmod-passives:0603-CAP
- added C17: 10uF, kmod-passives:0603-CAP
- added C18, C19, C27, C29, C34, C35, C36, C37, C38, C39, C40, C41, C42, C43, C44: 10nF, kmod-passives:0402-CAP
- added C45: DNP(10nF), kmod-passives:0402-CAP
- added C46, C47, C48, C49, C50, C51, C52, C53: 0.1uF, kmod-passives:0402-CAP
- added CH1, CH2: SRF2012-900YA, kmod-passives:SRF2012A
- added JP1: 0, SparkFun-Connectors:1X08
- added JP2: 1, SparkFun-Connectors:1X08
- added JP3: 2, SparkFun-Connectors:1X08
- added JP4: 3, SparkFun-Connectors:1X08
- added JP5: 4, SparkFun-Connectors:1X08
- added JP6: 0_1, SparkFun-Connectors:1X08
- added LED4_1: YLW, kmod-passives:0603_LED
- added RA11: 100k, kmod-passives:0603-ARV
- added SB17: RXP, kmod-nonparts:SB-0402
- added SB18: RXN, kmod-nonparts:SB-0402
- added SB19: TXP, kmod-nonparts:SB-0402
- added SB20: TXN, kmod-nonparts:SB-0402
- added U$18: AP1117IE33G, kmod-ics:SOT223
- C13, C14, C15: value 0.1uF -> DNP(10nF)
- IC1, IC2, IC3, IC4, IC5: value (none) -> 74X3G34
- SB12: value HVB_CS -> TVB_CS
- SB13: value HVB_CS -> BVB_CS
- U$13: value (none) -> ATX-PWRVERT-NOPEGS; device kmod-connectors:ATX-24-VERT -> kmod-connectors:ATX-24-VERT-NOPEGS
- U$2: value M04X2 -> DF40-80RCP; device SparkFun-Connectors:2X4 -> kmod-connectors:DF40-RCP-80
- U$3: value M04X2 -> DF40-90RCP; device SparkFun-Connectors:2X4 -> kmod-connectors:DF40-RCP-90
- moved LED3_1 166.2 mm to (68.0, 41.0)
- moved R23 165.7 mm to (66.0, 44.0), flipped to the bottom
- moved R15 160.5 mm to (59.0, 24.0)
- moved LED3_2 157.8 mm to (66.0, 41.0)
- moved R16 148.1 mm to (47.0, 24.0)
- moved R21 146.4 mm to (47.0, 43.5), flipped to the bottom
- moved LED2_2 145.9 mm to (48.0, 41.0)
- moved LED2_1 140.9 mm to (46.0, 41.0)
- moved R24 138.3 mm to (66.5, 14.5)
- moved R25 136.4 mm to (66.5, 16.5)
- moved C26 127.7 mm to (61.0, 41.0)
- moved C25 126.6 mm to (61.0, 42.0)
- moved C24 125.3 mm to (61.0, 43.0)
- moved R19 124.1 mm to (26.0, 45.5), flipped to the bottom
- moved C23 123.3 mm to (61.0, 44.0)
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Connections:
- removed net N$39: C9.2, U$1.75
- removed net USB_N_2: SOCKET2.B10, U$15.TD-
- removed net USB_N_3: SOCKET3.B10, U$15.BD-
- removed net USB_P_2: SOCKET2.B9, U$15.TD+
- removed net USB_P_3: SOCKET3.B9, U$15.BD+
- new net 3.3VSB: C17.1, R28.2, RA1.5, RA1.6, RA1.7, RA1.8, RA11.5, RA11.6, RA11.7, RA11.8, RA3.5, RA3.6, RA3.7, RA3.8, RA5.5, RA5.6, RA5.7, RA5.8, RA7.5, RA7.6, RA7.7, RA7.8, RA9.5, RA9.6, RA9.7, RA9.8, U$18.2, U$18.4, U$2.1, U$2.2
- new net E0_RXN_C: C53.2, SB18.L1, SB18.L2, U$3.82
- new net E0_RXP_C: C52.2, SB17.L1, SB17.L2, U$3.83
- new net E0_TXN_C: C51.2, SB20.L1, SB20.L2, U$3.85
- new net E0_TXP_C: C50.2, SB19.L1, SB19.L2, U$3.86
- new net N$67: CH1.2, U$3.15
- new net N$68: C46.1, CH1.1
- new net N$69: C47.1, CH1.4
- new net N$70: C48.1, CH2.1
- new net N$71: C49.1, CH2.4
- new net N$73: C10.2, U$3.73
- new net PRSNT#_5: RA11.2, U$2.26
- new net PRSNT#_6: RA11.3, U$2.19
- new net PRSNT#_7: RA11.4, U$2.12
- new net USB_N_0: SOCKET1.B10, U$15.BD-
- new net USB_N_4: SOCKET5.B10, U$15.TD-
- new net USB_P_0: SOCKET1.B9, U$15.BD+
- new net USB_P_4: SOCKET5.B9, U$15.TD+
- net !PS_ON: now also U$2.6
- net 12V: no longer R1.1, R3.1, R5.1, R7.1, R9.1
- net 12V_0: now also JP6.8; no longer R1.2
- net 12V_1: no longer R3.2
- net 12V_2: no longer R5.2
- net 12V_3: no longer R7.2
- net 12V_4: no longer R9.2
- net 3.3V: now also LED4_1.A, U$3.1, U$3.2, U$3.89, U$3.90; no longer LED3_4.A, R28.2, RA1.5, RA1.6, RA1.7, RA1.8, RA3.5, RA3.6, RA3.7, RA3.8, RA5.5, RA5.6, RA5.7, RA5.8, RA7.5, RA7.6, RA7.7, RA7.8, RA9.5, RA9.6, RA9.7, RA9.8, U$1.1, U$1.2, U$1.89, U$1.90
- net 5VSB: now also C16.1, U$18.3, U$2.78, U$2.79, U$2.80
- net B_VBUS: no longer R13.1
- net COM_RX_0: now also JP6.6, U$2.67
- net COM_RX_1: now also U$2.60
- net COM_RX_2: now also U$2.53
- net COM_RX_3: now also U$2.46
- net COM_RX_4: now also U$2.35
- net COM_TX_0: now also JP6.5, U$2.68
- net COM_TX_1: now also U$2.61
- net COM_TX_2: now also U$2.54
- net COM_TX_3: now also U$2.47
- net COM_TX_4: now also U$2.34
- net E0_RXN: now also C53.1; no longer C5.1
- net E0_RXP: now also C52.1; no longer C4.1
- net E0_TXN: now also C51.1; no longer C21.1
- net E0_TXP: now also C50.1; no longer C20.1
- net E4_RXN: now also C49.2
- net E4_RXP: now also C48.2
- net E4_TXN: now also C47.2
- net E4_TXP: now also C46.2
- net EX_RXN: now also SB18.R1, SB18.R2, U$3.6; no longer U$1.6
- net EX_RXP: now also SB17.R1, SB17.R2, U$3.5; no longer U$1.5
- net EX_TXN: now also SB20.R1, SB20.R2, U$3.9; no longer U$1.9
- net EX_TXP: now also SB19.R1, SB19.R2, U$3.8; no longer U$1.8
- net GND: now also C16.2, C17.2, C18.2, C19.2, C27.2, C29.2, C34.2, C35.2, C36.2, C37.2, C38.2, C39.2, C4.1, C40.2, C41.2, C42.2, C43.2, C44.2, C45.2, C5.1, JP1.6, JP2.6, JP3.6, JP4.6, JP5.6, JP6.4, U$18.1, U$2.15, U$2.22, U$2.29, U$2.36, U$2.45, U$2.52, U$2.59, U$2.66, U$2.76, U$3.10, U$3.14, U$3.17, U$3.20, U$3.24, U$3.27, U$3.30, U$3.34, U$3.37, U$3.4, U$3.40, U$3.51, U$3.54, U$3.57, U$3.61, U$3.64, U$3.67, U$3.7, U$3.71, U$3.74, U$3.77, U$3.81, U$3.84, U$3.87; no longer U$1.10, U$1.14, U$1.17, U$1.20, U$1.24, U$1.27, U$1.30, U$1.34, U$1.37, U$1.4, U$1.40, U$1.51, U$1.54, U$1.57, U$1.61, U$1.64, U$1.67, U$1.7, U$1.71, U$1.74, U$1.77, U$1.81, U$1.84, U$1.87, U$16.5, U$3.5, U$4.5, U$5.5
- net HD_LED: now also U$2.7
- net HOST_VBUS_U: no longer R11.2
- net HOST_VBUS_U1: no longer R13.2
- net I2C_SCL_0: now also JP1.7; no longer U$2.8
- net I2C_SCL_1: now also JP2.7; no longer U$3.8
- net I2C_SCL_2: now also JP3.7; no longer U$4.8
- net I2C_SCL_3: now also JP4.7; no longer U$5.8
- net I2C_SCL_4: now also JP5.7; no longer U$16.8
- net I2C_SDA_0: now also JP1.8; no longer U$2.7
- net I2C_SDA_1: now also JP2.8; no longer U$3.7
- net I2C_SDA_2: now also JP3.8; no longer U$4.7
- net I2C_SDA_3: now also JP4.8; no longer U$5.7
- net I2C_SDA_4: now also JP5.8; no longer U$16.7
- net LED0_1: now also U$3.79; no longer U$1.79
- net LED0_2: now also U$3.80; no longer U$1.80
- net LED1_1: now also U$3.69; no longer U$1.69
- net LED1_2: now also U$3.70; no longer U$1.70
- net LED2_1: now also U$3.59; no longer U$1.32
- net LED2_2: now also U$3.60; no longer U$1.31
- net LED3_1: now also U$3.32; no longer U$1.22
- net LED3_2: now also U$3.31; no longer U$1.21
- net LED4_1: now also U$3.22; no longer LED3_4.C, R18.2
- net LED4_2: now also U$3.21
- net LEDX_1: now also U$3.12; no longer U$1.12
- net LEDX_2: now also U$3.11; no longer U$1.11
- net N$28: now also LED4_1.C, R18.2; no longer C11.2, U$1.72
- net N$29: now also C11.2, U$3.72; no longer C10.2, U$1.73
- net N$32: now also C5.2
- net N$33: now also C4.2
- net N$41: now also U$3.76; no longer U$1.76
- net N$43: now also CH2.3, U$3.19; no longer C5.2, U$1.82
- net N$44: now also C9.2, U$3.75; no longer C4.2, U$1.83
- net N$45: now also CH2.2, U$3.18; no longer C21.2, U$1.85
- net N$46: now also CH1.3, U$3.16; no longer C20.2, U$1.86
- net N$49: now also U$3.62; no longer U$1.29
- net N$50: now also U$3.63; no longer U$1.28
- net N$51: now also U$3.65; no longer U$1.26
- net N$52: now also U$3.66; no longer U$1.25
- net N$53: now also U$3.28; no longer U$1.18
- net N$54: now also U$3.26; no longer U$1.16
- net N$55: now also U$3.25; no longer U$1.15
- net N$96: now also U$3.29; no longer U$1.19
- net PRSNT#_0: now also C19.1, JP6.2, U$2.69; no longer CONN9.P
- net PRSNT#_1: now also C34.1, U$2.62
- net PRSNT#_2: now also C37.1, U$2.55
- net PRSNT#_3: now also C40.1, U$2.48
- net PRSNT#_4: now also C43.1, U$2.33
- net PWR2: no longer R14.1, R2.1, R4.1, R6.1, R8.1
- net PWR2_0: now also JP6.7; no longer R2.2
- net PWR2_1: no longer R4.2
- net PWR2_2: no longer R6.2
- net PWR2_3: no longer R8.2
- net PWR2_4: no longer R14.2
- net PWR_BUT: now also U$2.73
- net PWR_OK: now also C45.1, U$2.75
- net PWR_ON#_0: now also C27.1, JP6.3, U$2.71; no longer CONN8.P
- net PWR_ON#_1: now also C35.1, U$2.64
- net PWR_ON#_2: now also C38.1, U$2.57
- net PWR_ON#_3: now also C41.1, U$2.50
- net PWR_ON#_4: now also C44.1, U$2.31
- net RESET_BUT: now also U$2.74
- net SPI_CLK_0: now also JP1.3; no longer U$2.4
- net SPI_CLK_1: now also JP2.3; no longer U$3.4
- net SPI_CLK_2: now also JP3.3; no longer U$4.4
- net SPI_CLK_3: now also JP4.3; no longer U$5.4
- net SPI_CLK_4: now also JP5.3; no longer U$16.4
- net SPI_CS_0: now also JP1.5; no longer U$2.3
- net SPI_CS_1: now also JP2.5; no longer U$3.3
- net SPI_CS_2: now also JP3.5; no longer U$4.3
- net SPI_CS_3: now also JP4.5; no longer U$5.3
- net SPI_CS_4: now also JP5.5; no longer U$16.3
- net SPI_MISO_0: now also JP1.2; no longer U$2.2
- net SPI_MISO_1: now also JP2.2; no longer U$3.2
- net SPI_MISO_2: now also JP3.2; no longer U$4.2
- net SPI_MISO_3: now also JP4.2; no longer U$5.2
- net SPI_MISO_4: now also JP5.2; no longer U$16.2
- net SPI_MOSI_0: now also JP1.4; no longer U$2.1
- net SPI_MOSI_1: now also JP2.4; no longer U$3.1
- net SPI_MOSI_2: now also JP3.4; no longer U$4.1
- net SPI_MOSI_3: now also JP4.4; no longer U$5.1
- net SPI_MOSI_4: now also JP5.4; no longer U$16.1
- net SYS_RESET#_0: now also C18.1, JP6.1, U$2.70; no longer CONN10.P
- net SYS_RESET#_1: now also C29.1, U$2.63
- net SYS_RESET#_2: now also C36.1, U$2.56
- net SYS_RESET#_3: now also C39.1, U$2.49
- net SYS_RESET#_4: now also C42.1, U$2.32
- net T_VBUS: no longer R11.1
- net UBOOT_0: now also JP1.1; no longer U$2.6
- net UBOOT_1: now also JP2.1; no longer U$3.6
- net UBOOT_2: now also JP3.1; no longer U$4.6
- net UBOOT_3: now also JP4.1; no longer U$5.6
- net UBOOT_4: now also JP5.1; no longer U$16.6
Routing:
- added copper zone on layer 2, net GND
Other:
- board text added: "12V"
- board text added: "CLK"
- board text added: "CS"
- board text added: "GND"
- board text added: "MISO"
- board text added: "MOSI"
- board text added: "P2"
- board text added: "PNT"
- board text added: "PWR"
- board text added: "RST"
- board text added: "RX"
- board text added: "SCL"
- board text added: "SDA"
- board text added: "TX"
- board text added: "UBT"
