File: coven/supervisor_v0.1/board.brd (EAGLE design)
At the start: 40 x 20 mm, 72 parts, among them IC1 74HC151PW, IC3 STM6601D, IC4 74AC138MTCX, IC5 FT2232HL, U1 ATMEGA328P, Y1 12MHz, Y2 16MHz

Commit message: More work on coven boards (mostly old stuff I forgot to check in)
Parts:
- removed U$3: DF40-80HDR, kmod-connectors:DF40-HDR-80
- added CONN8, CONN9: (no value), kmod-nonparts:HOLE_22AWG
- added U$2: DF40-80HDR, kmod-connectors:DF40-HDR-80
- moved IC2 199.5 mm to (36.0, 27.0)
- moved R7 139.3 mm to (-20.0, -22.0)
- moved R8 139.3 mm to (-20.0, -26.0)
- moved JP3 130.0 mm to (30.0, -15.0)
- moved Y2 122.3 mm to (36.0, 9.00), turned to 90 degrees
- moved C24 107.9 mm to (14.0, -24.0)
- moved LMEG 107.9 mm to (2.00, -49.0)
- moved R6 107.9 mm to (6.00, -49.5)
- moved RA1 107.9 mm to (15.0, -20.0)
- moved SB4 107.9 mm to (6.00, -39.0)
- moved SB5 107.9 mm to (6.00, -42.0)
- moved SB6 107.9 mm to (6.00, -44.5)
- moved SB7 107.9 mm to (6.00, -47.0)
- moved SB8 107.9 mm to (3.00, -52.5)
- moved SB9 107.9 mm to (3.00, -55.0)
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Connections:
- new net 3.3VSB: U$2.1, U$2.2
- new net N$31: CONN9.P
- new net N$35: CONN8.P
- net !PS_ON: now also U$2.6; no longer U$3.6
- net 5VSB: now also U$2.78, U$2.79, U$2.80; no longer U$3.78, U$3.79, U$3.80
- net COM_RX_0: now also U$2.67; no longer U$3.14
- net COM_RX_1: now also U$2.60; no longer U$3.67
- net COM_RX_2: now also U$2.53; no longer U$3.21
- net COM_RX_3: now also U$2.46; no longer U$3.60
- net COM_RX_4: now also U$2.35; no longer U$3.28
- net COM_RX_5: now also U$2.28; no longer U$3.53
- net COM_RX_6: now also U$2.21; no longer U$3.35
- net COM_RX_7: now also U$2.14; no longer U$3.46
- net COM_TX_0: now also U$2.68; no longer U$3.13
- net COM_TX_1: now also U$2.61; no longer U$3.68
- net COM_TX_2: now also U$2.54; no longer U$3.20
- net COM_TX_3: now also U$2.47; no longer U$3.61
- net COM_TX_4: now also U$2.34; no longer U$3.27
- net COM_TX_5: now also U$2.27; no longer U$3.54
- net COM_TX_6: now also U$2.20; no longer U$3.34
- net COM_TX_7: now also U$2.13; no longer U$3.47
- net GND: now also IC2.25, IC2.PAD, IC2.PAD1, IC2.PAD2, IC2.PAD3, IC2.PAD4, IC2.PAD5, IC2.PAD6, IC2.PAD7, IC2.PAD8, IC2.PAD9, U$2.15, U$2.22, U$2.29, U$2.36, U$2.45, U$2.5, U$2.52, U$2.59, U$2.66, U$2.76; no longer U$3.15, U$3.22, U$3.29, U$3.36, U$3.45, U$3.5, U$3.52, U$3.59, U$3.66, U$3.76
- net HD_LED: now also U$2.7; no longer U$3.7
- net PRSNT#_0: now also IC2.17, U$2.69; no longer U$3.12
- net PRSNT#_1: now also IC2.18, U$2.62; no longer U$3.69
- net PRSNT#_2: now also IC2.19, U$2.55; no longer U$3.19
- net PRSNT#_3: now also IC2.20, U$2.48; no longer U$3.62
- net PRSNT#_4: now also IC2.21, U$2.33; no longer U$3.26
- net PRSNT#_5: now also IC2.22, U$2.26; no longer U$3.55
- net PRSNT#_6: now also IC2.23, U$2.19; no longer U$3.33
- net PRSNT#_7: now also IC2.24, U$2.12; no longer U$3.48
- net PWR_BUT: now also U$2.73; no longer U$3.73
- net PWR_OK: now also U$2.75; no longer U$3.75
- net PWR_ON#_0: now also IC2.1, U$2.71; no longer U$3.10
- net PWR_ON#_1: now also IC2.2, U$2.64; no longer U$3.71
- net PWR_ON#_2: now also IC2.3, U$2.57; no longer U$3.17
- net PWR_ON#_3: now also IC2.4, U$2.50; no longer U$3.64
- net PWR_ON#_4: now also IC2.5, U$2.31; no longer U$3.24
- net PWR_ON#_5: now also IC2.6, U$2.24; no longer U$3.57
- net PWR_ON#_6: now also IC2.7, U$2.17; no longer U$3.31
- net PWR_ON#_7: now also IC2.8, U$2.10; no longer U$3.50
- net RESET_BUT: now also U$2.74; no longer U$3.74
- net SYS_RESET#_0: now also IC2.9, U$2.70; no longer U$3.11
- net SYS_RESET#_1: now also IC2.10, U$2.63; no longer U$3.70
- net SYS_RESET#_2: now also IC2.11, U$2.56; no longer U$3.18
- net SYS_RESET#_3: now also IC2.12, U$2.49; no longer U$3.63
- net SYS_RESET#_4: now also IC2.13, U$2.32; no longer U$3.25
- net SYS_RESET#_5: now also IC2.14, U$2.25; no longer U$3.56
- net SYS_RESET#_6: now also IC2.15, U$2.18; no longer U$3.32
- net SYS_RESET#_7: now also IC2.16, U$2.11; no longer U$3.49
