File: vga/board_v0.3/board.brd (EAGLE design)
At the start: 55 x 52 mm, 126 parts, among them IC1 XC6S{9,16,25}LX-FT256, IC2 74LVC3G34, IC3 AS4C8M16D1, X2 

Commit message: Got the VGA board up and running!
The resistors had gotten mixed up due to pinswapping,
so fixed that up in the schematic.

Copied the code from v0.2, updated the ucf, and it works!
Parts:
- R10, R9: value 2k -> 8.06k
- R11: value 2k -> 4.02k
- R12, R13: value 4.02k -> 2k
- R14: value 4.02k -> 1k
- R15, R16: value 8.06k -> 499
- R3, R4: value 499 -> 4.02k
- R5: value 499 -> 2k
- R8: value 1k -> 499
Connections:
- net VB0: now also IC1.P5, R9.1; no longer IC1.N5, R15.1
- net VB1: now also IC1.P6, R3.1; no longer IC1.N6, R12.1
- net VB2: now also IC1.N6, R12.1; no longer IC1.P5, R9.1
- net VB4: now also IC1.N5, R15.1; no longer IC1.P6, R3.1
- net VG0: now also IC1.P8, R10.1; no longer IC1.T5, R16.1
- net VG1: now also IC1.R7, R4.1; no longer IC1.T6, R13.1
- net VG2: now also IC1.T6, R13.1; no longer IC1.P8, R10.1
- net VG4: now also IC1.T5, R16.1; no longer IC1.R7, R4.1
- net VR1: now also IC1.T7, R11.1; no longer IC1.P7, R14.1
- net VR2: now also IC1.L7, R5.1; no longer IC1.T7, R11.1
- net VR3: now also IC1.P7, R14.1; no longer IC1.M7, R8.1
- net VR4: now also IC1.M7, R8.1; no longer IC1.L7, R5.1
Routing:
- net VR2: track 9.08 -> 13.7 mm, vias 0 -> 2
- net VG0: track 4.26 -> 7.50 mm
- net VB0: track 13.7 -> 10.5 mm, vias 2 -> 0
- net VG2: track 7.50 -> 4.67 mm
- net VR3: track 12.7 -> 10.00 mm
- net VB2: track 10.5 -> 12.9 mm, vias 0 -> 2
- net VG4: track 6.29 -> 4.26 mm
- net VG1: track 4.67 -> 6.29 mm
- net VB4: track 12.5 -> 13.7 mm
- net VR4: track 13.7 -> 12.7 mm
- net VR1: track 10.00 -> 9.08 mm, vias 2 -> 0
Changed lines of the file:
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@@
 <layers>
 <layer number="1" name="Top" color="4" fill="1" visible="yes" active="yes"/>
-<layer number="2" name="Route2" color="20" fill="5" visible="yes" active="yes"/>
+<layer number="2" name="Route2" color="20" fill="5" visible="no" active="yes"/>
 <layer number="3" name="Route3" color="4" fill="3" visible="no" active="no"/>
 <layer number="4" name="Route4" color="1" fill="4" visible="no" active="no"/>
@@
 <layer number="13" name="Route13" color="4" fill="5" visible="no" active="no"/>
 <layer number="14" name="Route14" color="1" fill="6" visible="no" active="no"/>
-<layer number="15" name="Route15" color="5" fill="4" visible="yes" active="yes"/>
+<layer number="15" name="Route15" color="5" fill="4" visible="no" active="yes"/>
 <layer number="16" name="Bottom" color="1" fill="1" visible="yes" active="yes"/>
 <layer number="17" name="Pads" color="2" fill="1" visible="yes" active="yes"/>
@@
 <attribute name="OC_FARNELL" value="unknown" x="34.9" y="57" size="1.778" layer="27" rot="R180" display="off"/>
 </element>
-<element name="R3" library="kmod-passives" package="0603-RES" value="499" x="33.6" y="44.6" rot="R90"/>
-<element name="R4" library="kmod-passives" package="0603-RES" value="499" x="27" y="40.9" rot="R90"/>
-<element name="R5" library="kmod-passives" package="0603-RES" value="499" x="27.3" y="44.6" rot="R90"/>
+<element name="R3" library="kmod-passives" package="0603-RES" value="4.02k" x="33.6" y="44.6" rot="R90"/>
+<element name="R4" library="kmod-passives" package="0603-RES" value="4.02k" x="27" y="40.9" rot="R90"/>
+<element name="R5" library="kmod-passives" package="0603-RES" value="2k" x="27.3" y="44.6" rot="R90"/>
 <element name="R6" library="kmod-passives" package="0603-RES" value="1k" x="36.6" y="44.6" rot="R90"/>
 <element name="R7" library="kmod-passives" package="0603-RES" value="1k" x="30" y="40.9" rot="R90"/>
-<element name="R8" library="kmod-passives" package="0603-RES" value="1k" x="30.3" y="44.6" rot="R90"/>
-<element name="R9" library="kmod-passives" package="0603-RES" value="2k" x="32.1" y="44.6" rot="R90"/>
-<element name="R10" library="kmod-passives" package="0603-RES" value="2k" x="25.5" y="40.9" rot="R90"/>
-<element name="R11" library="kmod-passives" package="0603-RES" value="2k" x="25.8" y="44.6" rot="R90"/>
-<element name="R12" library="kmod-passives" package="0603-RES" value="4.02k" x="35.1" y="44.6" rot="R90"/>
-<element name="R13" library="kmod-passives" package="0603-RES" value="4.02k" x="28.5" y="40.9" rot="R90"/>
-<element name="R14" library="kmod-passives" package="0603-RES" value="4.02k" x="28.8" y="44.6" rot="R90"/>
-<element name="R15" library="kmod-passives" package="0603-RES" value="8.06k" x="38.1" y="44.6" rot="R90"/>
-<element name="R16" library="kmod-passives" package="0603-RES" value="8.06k" x="31.5" y="40.9" rot="R90"/>
+<element name="R8" library="kmod-passives" package="0603-RES" value="499" x="30.3" y="44.6" rot="R90"/>
+<element name="R9" library="kmod-passives" package="0603-RES" value="8.06k" x="32.1" y="44.6" rot="R90"/>
+<element name="R10" library="kmod-passives" package="0603-RES" value="8.06k" x="25.5" y="40.9" rot="R90"/>
+<element name="R11" library="kmod-passives" package="0603-RES" value="4.02k" x="25.8" y="44.6" rot="R90"/>
+<element name="R12" library="kmod-passives" package="0603-RES" value="2k" x="35.1" y="44.6" rot="R90"/>
+<element name="R13" library="kmod-passives" package="0603-RES" value="2k" x="28.5" y="40.9" rot="R90"/>
+<element name="R14" library="kmod-passives" package="0603-RES" value="1k" x="28.8" y="44.6" rot="R90"/>
+<element name="R15" library="kmod-passives" package="0603-RES" value="499" x="38.1" y="44.6" rot="R90"/>
+<element name="R16" library="kmod-passives" package="0603-RES" value="499" x="31.5" y="40.9" rot="R90"/>
 <element name="R17" library="kmod-passives" package="0603-RES" value="8.06k" x="24.3" y="44.6" rot="R90"/>
 <element name="C9" library="kmod-passives" package="0402-CAP" value="1uF" x="18" y="47" rot="MR0"/>
@@
 <wire x1="30.571" y1="45.721" x2="30.571" y2="48.46" width="0.1524" layer="1"/>
 </signal>
-<signal name="VB4">
+<signal name="VB1">
 <contactref element="R3" pad="1"/>
 <contactref element="IC1" pad="P6"/>
@@
 <wire x1="33.6" y1="43.4" x2="33.6" y2="43.75" width="0.1524" layer="1"/>
 </signal>
-<signal name="VG4">
+<signal name="VG1">
 <contactref element="R4" pad="1"/>
 <contactref element="IC1" pad="R7"/>
@@
 <wire x1="27" y1="39.3" x2="27" y2="40.05" width="0.1524" layer="1"/>
 </signal>
-<signal name="VR4">
+<signal name="VR2">
 <contactref element="R5" pad="1"/>
 <contactref element="IC1" pad="L7"/>
@@
 <wire x1="30" y1="37.8" x2="30" y2="40.05" width="0.1524" layer="1"/>
 </signal>
-<signal name="VR3">
+<signal name="VR4">
 <contactref element="R8" pad="1"/>
 <contactref element="IC1" pad="M7"/>
@@
 <wire x1="29" y1="33.7" x2="29" y2="33" width="0.1524" layer="16"/>
 </signal>
-<signal name="VB2">
+<signal name="VB0">
 <contactref element="R9" pad="1"/>
 <contactref element="IC1" pad="P5"/>
@@
 <wire x1="32.1" y1="43.7" x2="32.1" y2="43.75" width="0.1524" layer="1"/>
 </signal>
-<signal name="VG2">
+<signal name="VG0">
 <contactref element="R10" pad="1"/>
 <contactref element="IC1" pad="P8"/>
@@
 <wire x1="28.5" y1="34.9" x2="28.5" y2="36.8" width="0.1524" layer="1"/>
 </signal>
-<signal name="VR2">
+<signal name="VR1">
 <contactref element="R11" pad="1"/>
 <contactref element="IC1" pad="T7"/>
@@
 <wire x1="26.25" y1="43.3" x2="25.8" y2="43.75" width="0.1524" layer="1"/>
 </signal>
-<signal name="VB1">
+<signal name="VB2">
 <contactref element="R12" pad="1"/>
 <contactref element="IC1" pad="N6"/>
@@
 <wire x1="35.1" y1="40.6" x2="35.1" y2="42.7" width="0.1524" layer="16"/>
 </signal>
-<signal name="VG1">
+<signal name="VG2">
 <contactref element="R13" pad="1"/>
 <contactref element="IC1" pad="T6"/>
@@
 <wire x1="28.5" y1="38.5" x2="28.5" y2="40.05" width="0.1524" layer="1"/>
 </signal>
-<signal name="VR1">
+<signal name="VR3">
 <contactref element="R14" pad="1"/>
 <contactref element="IC1" pad="P7"/>
@@
 <wire x1="29" y1="34" x2="28.6" y2="34.4" width="0.1524" layer="1"/>
 </signal>
-<signal name="VB0">
+<signal name="VB4">
 <contactref element="R15" pad="1"/>
 <contactref element="IC1" pad="N5"/>
@@
 <wire x1="37.9" y1="42" x2="37.9" y2="42.7" width="0.1524" layer="16"/>
 </signal>
-<signal name="VG0">
+<signal name="VG4">
 <contactref element="R16" pad="1"/>
 <contactref element="IC1" pad="T5"/>
