File: vga/board_v0.3/board.sch (EAGLE design)
At the start: 130 parts, among them IC1 XC6S{9,16,25}LX-FT256, IC2 74LVC3G34, IC3 AS4C8M16D1

Commit message: vga board v0.3.  added keepout to a bunch of packages
Parts:
- removed C28, C50: 10uF, kmod-passives:CAP0603
- removed C29, C31, C32: 1uF, kmod-passives:CAP0402-CAP
- removed CONN6: INITB, kmod-nonparts:CONNECTOR1.27
- added R48: 100, kmod-passives:RESISTOR0603
- added S1: TAC_SWITCHPTH, kmod-mechanical:TAC_SWITCHPTH
- C23: value 10uF -> 22uF; device kmod-passives:CAP0603 -> kmod-passives:CAP0805
- C4: value 10uF -> 100uF; device kmod-passives:CAP0603 -> kmod-passives:CAP_POLPTH-5-2
- C5: value 1uF -> 0.1uF; device kmod-passives:CAP0402-CAP -> kmod-passives:CAP0201
- R23: device kmod-passives:RESISTOR0603 -> kmod-passives:RESISTOR0402
- X2: value (none) -> (none)
Connections:
- net N$12 renamed DDR3_ZQ
- net N$13 renamed DDR3_CS#
- new net N$17: IC1.IO_L1N_VREF_0, IC1.IO_L2N_0
- new net N$22: IC1.IO_L2P_0, IC1.IO_L4P_0
- new net N$24: IC1.IO_L3N_0, IC1.IO_L3P_0
- new net N$25: IC1.IO_L7N_0, IC1.IO_L7P_0
- new net N$26: IC1.IO_L38N_VREF_0, IC1.IO_L6P_0
- new net N$27: IC1.IO_L33P_0, IC1.IO_L34P_GCLK19_0
- new net N$28: IC1.IO_L37N_GCLK12_0, IC1.IO_L40N_0
- new net N$29: IC1.IO_L36N_GCLK14_0, IC1.IO_L38P_0
- new net N$31: IC1.IO_L36P_GCLK15_0, IC1.IO_L5N_0
- new net N$32: IC1.IO_L64N_SCP4_0, IC1.IO_L66P_SCP1_0
- new net N$35: R48.1, SB1.P$2, SB2.P$2
- net 1.2V: now also C20.+; no longer C4.1, C5.1
- net 1.5V: now also C4.+, C5.1, IC1.VCCO_3; no longer C20.+, C28.1, C29.1, C50.1, IC1.VCCO_1
- net 2.5V: now also IC1.VCCO_1; no longer C21.+, IC1.VCCO_3
- net 3.3V: now also C21.+
- net 50MHZ: now also IC1.IO_L34N_GCLK18_0
- net DDR1_A0: now also IC1.IO_L37P_A7_M1A0_1; no longer IC1.IO_L47P_M3A0_3
- net DDR1_A1: now also IC1.IO_L37N_A6_M1A1_1; no longer IC1.IO_L47N_M3A1_3
- net DDR1_A10: now also IC1.IO_L33P_A15_M1A10_1; no longer IC1.IO_L51P_M3A10_3
- net DDR1_A11: now also IC1.IO_L30N_A20_M1A11_1; no longer IC1.IO_L54N_M3A11_3
- net DDR1_A12: now also IC1.IO_L31N_A18_M1A12_1; no longer IC1.IO_L53N_M3A12_3
- net DDR1_A2: now also IC1.IO_L35N_A10_M1A2_1; no longer IC1.IO_L49N_M3A2_3
- net DDR1_A3: now also IC1.IO_L39P_M1A3_1; no longer IC1.IO_L45P_M3A3_3
- net DDR1_A4: now also IC1.IO_L33N_A14_M1A4_1; no longer IC1.IO_L51N_M3A4_3
- net DDR1_A5: now also IC1.IO_L40P_GCLK11_M1A5_1; no longer IC1.IO_L44P_GCLK21_M3A5_3
- net DDR1_A6: now also IC1.IO_L40N_GCLK10_M1A6_1; no longer IC1.IO_L44N_GCLK20_M3A6_3
- net DDR1_A7: now also IC1.IO_L35P_A11_M1A7_1; no longer IC1.IO_L49P_M3A7_3
- net DDR1_A8: now also IC1.IO_L32P_A17_M1A8_1; no longer IC1.IO_L52P_M3A8_3
- net DDR1_A9: now also IC1.IO_L32N_A16_M1A9_1; no longer IC1.IO_L52N_M3A9_3
- net DDR1_BA0: now also IC1.IO_L36P_A9_M1BA0_1; no longer IC1.IO_L48P_M3BA0_3
- net DDR1_BA1: now also IC1.IO_L36N_A8_M1BA1_1; no longer IC1.IO_L48N_M3BA1_3
- net DDR1_CAS#: now also IC1.IO_L41N_GCLK8_M1CASN_1; no longer IC1.IO_L43N_GCLK22_IRDY2_M3CASN_3
- net DDR1_CK: now also IC1.IO_L38P_A5_M1CLK_1; no longer IC1.IO_L46P_M3CLK_3
- net DDR1_CK#: now also IC1.IO_L38N_A4_M1CLKN_1; no longer IC1.IO_L46N_M3CLKN_3
- net DDR1_CKE: now also IC1.IO_L31P_A19_M1CKE_1; no longer IC1.IO_L53P_M3CKE_3
- net DDR1_DML: now also IC1.IO_L42N_GCLK6_TRDY1_M1LDM_1; no longer IC1.IO_L42N_GCLK24_M3LDM_3
- net DDR1_DMU: now also IC1.IO_L42P_GCLK7_M1UDM_1; no longer IC1.IO_L42P_GCLK25_TRDY2_M3UDM_3
- net DDR1_DQ0: now also IC1.IO_L47P_FWE_B_M1DQ0_1; no longer IC1.IO_L37P_M3DQ0_3
- net DDR1_DQ1: now also IC1.IO_L47N_LDC_M1DQ1_1; no longer IC1.IO_L37N_M3DQ1_3
- net DDR1_DQ10: now also IC1.IO_L49P_M1DQ10_1; no longer IC1.IO_L35P_M3DQ10_3
- net DDR1_DQ11: now also IC1.IO_L49N_M1DQ11_1; no longer IC1.IO_L35N_M3DQ11_3
- net DDR1_DQ12: now also IC1.IO_L51P_M1DQ12_1; no longer IC1.IO_L33P_M3DQ12_3
- net DDR1_DQ13: now also IC1.IO_L51N_M1DQ13_1; no longer IC1.IO_L33N_M3DQ13_3
- net DDR1_DQ14: now also IC1.IO_L52P_M1DQ14_1; no longer IC1.IO_L32P_M3DQ14_3
- net DDR1_DQ15: now also IC1.IO_L52N_M1DQ15_1; no longer IC1.IO_L32N_M3DQ15_3
- net DDR1_DQ2: now also IC1.IO_L46P_FCS_B_M1DQ2_1; no longer IC1.IO_L38P_M3DQ2_3
- net DDR1_DQ3: now also IC1.IO_L46N_FOE_B_M1DQ3_1; no longer IC1.IO_L38N_M3DQ3_3
- net DDR1_DQ4: now also IC1.IO_L43P_GCLK5_M1DQ4_1; no longer IC1.IO_L41P_GCLK27_M3DQ4_3
- net DDR1_DQ5: now also IC1.IO_L43N_GCLK4_M1DQ5_1; no longer IC1.IO_L41N_GCLK26_M3DQ5_3
- net DDR1_DQ6: now also IC1.IO_L44P_A3_M1DQ6_1; no longer IC1.IO_L40P_M3DQ6_3
- net DDR1_DQ7: now also IC1.IO_L44N_A2_M1DQ7_1; no longer IC1.IO_L40N_M3DQ7_3
- net DDR1_DQ8: now also IC1.IO_L48P_HDC_M1DQ8_1; no longer IC1.IO_L36P_M3DQ8_3
- net DDR1_DQ9: now also IC1.IO_L48N_M1DQ9_1; no longer IC1.IO_L36N_M3DQ9_3
- net DDR1_DQSL: now also IC1.IO_L45P_A1_M1LDQS_1; no longer IC1.IO_L39P_M3LDQS_3
- net DDR1_DQSU: now also IC1.IO_L50P_M1UDQS_1; no longer IC1.IO_L34P_M3UDQS_3
- net DDR1_RAS#: now also IC1.IO_L41P_GCLK9_IRDY1_M1RASN_1; no longer IC1.IO_L43P_GCLK23_M3RASN_3
- net DDR1_WE#: now also IC1.IO_L34P_A13_M1WE_1; no longer IC1.IO_L50P_M3WE_3
- net DDR3_A0: now also IC1.IO_L47P_M3A0_3; no longer IC1.IO_L37P_A7_M1A0_1
- net DDR3_A1: now also IC1.IO_L47N_M3A1_3; no longer IC1.IO_L37N_A6_M1A1_1
- net DDR3_A10: now also IC1.IO_L51P_M3A10_3; no longer IC1.IO_L33P_A15_M1A10_1
- net DDR3_A11: now also IC1.IO_L54N_M3A11_3; no longer IC1.IO_L30N_A20_M1A11_1
- net DDR3_A12: now also IC1.IO_L53N_M3A12_3; no longer IC1.IO_L31N_A18_M1A12_1
- net DDR3_A13: now also IC1.IO_L55P_M3A13_3; no longer IC1.IO_L29P_A23_M1A13_1
- net DDR3_A14: now also IC1.IO_L55N_M3A14_3; no longer IC1.IO_L29N_A22_M1A14_1
- net DDR3_A2: now also IC1.IO_L49N_M3A2_3; no longer IC1.IO_L35N_A10_M1A2_1
- net DDR3_A3: now also IC1.IO_L45P_M3A3_3; no longer IC1.IO_L39P_M1A3_1
- net DDR3_A4: now also IC1.IO_L51N_M3A4_3; no longer IC1.IO_L33N_A14_M1A4_1
- net DDR3_A5: now also IC1.IO_L44P_GCLK21_M3A5_3; no longer IC1.IO_L40P_GCLK11_M1A5_1
- net DDR3_A6: now also IC1.IO_L44N_GCLK20_M3A6_3; no longer IC1.IO_L40N_GCLK10_M1A6_1
- net DDR3_A7: now also IC1.IO_L49P_M3A7_3; no longer IC1.IO_L35P_A11_M1A7_1
- net DDR3_A8: now also IC1.IO_L52P_M3A8_3; no longer IC1.IO_L32P_A17_M1A8_1
- net DDR3_A9: now also IC1.IO_L52N_M3A9_3; no longer IC1.IO_L32N_A16_M1A9_1
- net DDR3_BA0: now also IC1.IO_L48P_M3BA0_3; no longer IC1.IO_L36P_A9_M1BA0_1
- net DDR3_BA1: now also IC1.IO_L48N_M3BA1_3; no longer IC1.IO_L36N_A8_M1BA1_1
- net DDR3_BA2: now also IC1.IO_L50N_M3BA2_3; no longer IC1.IO_L34N_A12_M1BA2_1
- net DDR3_CAS#: now also IC1.IO_L43N_GCLK22_IRDY2_M3CASN_3; no longer IC1.IO_L41N_GCLK8_M1CASN_1
- net DDR3_CK: now also IC1.IO_L46P_M3CLK_3; no longer IC1.IO_L38P_A5_M1CLK_1
- net DDR3_CK#: now also IC1.IO_L46N_M3CLKN_3; no longer IC1.IO_L38N_A4_M1CLKN_1
- net DDR3_CKE: now also IC1.IO_L53P_M3CKE_3; no longer IC1.IO_L31P_A19_M1CKE_1
- net DDR3_DML: now also IC1.IO_L42N_GCLK24_M3LDM_3; no longer IC1.IO_L42N_GCLK6_TRDY1_M1LDM_1
- net DDR3_DMU: now also IC1.IO_L42P_GCLK25_TRDY2_M3UDM_3; no longer IC1.IO_L42P_GCLK7_M1UDM_1
- net DDR3_DQ0: now also IC1.IO_L37P_M3DQ0_3; no longer IC1.IO_L47P_FWE_B_M1DQ0_1
- net DDR3_DQ1: now also DDR3_0.DQ2, IC1.IO_L37N_M3DQ1_3; no longer DDR3_0.DQ1, IC1.IO_L47N_LDC_M1DQ1_1
- net DDR3_DQ10: now also DDR3_0.DQ15, IC1.IO_L35P_M3DQ10_3; no longer DDR3_0.DQ10, IC1.IO_L49P_M1DQ10_1
- net DDR3_DQ11: now also DDR3_0.DQ13, IC1.IO_L35N_M3DQ11_3; no longer DDR3_0.DQ11, IC1.IO_L49N_M1DQ11_1
- net DDR3_DQ12: now also DDR3_0.DQ10, IC1.IO_L33P_M3DQ12_3; no longer DDR3_0.DQ12, IC1.IO_L51P_M1DQ12_1
- net DDR3_DQ13: now also DDR3_0.DQ8, IC1.IO_L33N_M3DQ13_3; no longer DDR3_0.DQ13, IC1.IO_L51N_M1DQ13_1
- net DDR3_DQ14: now also IC1.IO_L32P_M3DQ14_3; no longer IC1.IO_L52P_M1DQ14_1
- net DDR3_DQ15: now also DDR3_0.DQ12, IC1.IO_L32N_M3DQ15_3; no longer DDR3_0.DQ15, IC1.IO_L52N_M1DQ15_1
- net DDR3_DQ2: now also DDR3_0.DQ1, IC1.IO_L38P_M3DQ2_3; no longer DDR3_0.DQ2, IC1.IO_L46P_FCS_B_M1DQ2_1
- net DDR3_DQ3: now also IC1.IO_L38N_M3DQ3_3; no longer IC1.IO_L46N_FOE_B_M1DQ3_1
- net DDR3_DQ4: now also IC1.IO_L41P_GCLK27_M3DQ4_3; no longer IC1.IO_L43P_GCLK5_M1DQ4_1
- net DDR3_DQ5: now also IC1.IO_L41N_GCLK26_M3DQ5_3; no longer IC1.IO_L43N_GCLK4_M1DQ5_1
- net DDR3_DQ6: now also IC1.IO_L40P_M3DQ6_3; no longer IC1.IO_L44P_A3_M1DQ6_1
- net DDR3_DQ7: now also IC1.IO_L40N_M3DQ7_3; no longer IC1.IO_L44N_A2_M1DQ7_1
- net DDR3_DQ8: now also DDR3_0.DQ11, IC1.IO_L36P_M3DQ8_3; no longer DDR3_0.DQ8, IC1.IO_L48P_HDC_M1DQ8_1
- net DDR3_DQ9: now also IC1.IO_L36N_M3DQ9_3; no longer IC1.IO_L48N_M1DQ9_1
- net DDR3_DQSL: now also IC1.IO_L39P_M3LDQS_3; no longer IC1.IO_L45P_A1_M1LDQS_1
- net DDR3_DQSL#: now also IC1.IO_L39N_M3LDQSN_3; no longer IC1.IO_L45N_A0_M1LDQSN_1
- net DDR3_DQSU: now also IC1.IO_L34P_M3UDQS_3; no longer IC1.IO_L50P_M1UDQS_1
- net DDR3_DQSU#: now also IC1.IO_L34N_M3UDQSN_3; no longer IC1.IO_L50N_M1UDQSN_1
- net DDR3_ODT: now also IC1.IO_L45N_M3ODT_3; no longer IC1.IO_L39N_M1ODT_1
- net DDR3_RAS#: now also IC1.IO_L43P_GCLK23_M3RASN_3; no longer IC1.IO_L41P_GCLK9_IRDY1_M1RASN_1
- net DDR3_RESET#: now also IC1.IO_L54P_M3RESET_3; no longer IC1.IO_L30P_A21_M1RESET_1
- net DDR3_WE#: now also IC1.IO_L50P_M3WE_3; no longer IC1.IO_L34P_A13_M1WE_1
- net GND: now also C4.-, S1.3, U$3.C0, U$3.C1, U$3.D0, U$3.D1, U$3.E0, U$3.E1, U$3.E2, U$3.E3; no longer C28.2, C29.2, C31.2, C32.2, C4.2, C50.2
- net HSYNC: now also IC1.IO_L63N_2; no longer IC1.IO_L35N_GCLK16_0
- net INIT_B: no longer CONN6.P
- net L0: now also IC1.IO_L33N_0
- net L1: now also IC1.IO_L6N_0
- net L2: now also IC1.IO_L4N_0
- net MB_A0: now also IC1.IO_L62N_VREF_0; no longer IC1.IO_L31P_GCLK31_D14_2, SB2.P$1
- net MB_A1: now also IC1.IO_L66N_SCP0_0; no longer IC1.IO_L30P_GCLK1_D13_2
- net MB_A2: now also IC1.IO_L39P_0; no longer IC1.IO_L23P_2
- net MB_A3: now also SB2.P$1; no longer IC1.IO_L14N_D12_2
- net MB_B0: now also IC1.IO_L62P_0; no longer IC1.IO_L47N_2
- net MB_B1: now also IC1.IO_L39N_0; no longer IC1.IO_L32N_GCLK28_2
- net MB_B2: now also IC1.IO_L35N_GCLK16_0; no longer IC1.IO_L30N_GCLK0_USERCCLK_2
- net MB_B3: now also IC1.IO_L35P_GCLK17_0; no longer IC1.IO_L23N_2
- net MB_C2: now also IC1.IO_L65N_SCP2_0; no longer IC1.IO_L48P_D7_2
- net MB_C3: now also IC1.IO_L63P_SCP7_0; no longer IC1.IO_L32P_GCLK29_2
- net MB_D2: now also IC1.IO_L65P_SCP3_0; no longer IC1.IO_L63N_2
- net MB_D3: now also IC1.IO_L63N_SCP6_0; no longer IC1.IO_L48N_RDWR_B_VREF_2
- net PROGRAM: now also R48.2, S1.2; no longer SB1.P$2, SB2.P$2
- net USB_CLK: now also IC1.IO_L37P_GCLK13_0; no longer IC1.IO_L33N_0
- net USB_DATA0: now also IC1.IO_L16N_VREF_2; no longer IC1.IO_L2P_0
- net USB_DATA1: now also IC1.IO_L14P_D11_2; no longer IC1.IO_L2N_0
- net USB_DATA2: now also IC1.IO_L16P_2; no longer IC1.IO_L3P_0
- net USB_DATA3: now also IC1.IO_L14N_D12_2; no longer IC1.IO_L3N_0
- net USB_DATA4: now also IC1.IO_L29P_GCLK3_2; no longer IC1.IO_L4P_0
- net USB_DATA5: now also IC1.IO_L23P_2; no longer IC1.IO_L4N_0
- net USB_DATA6: now also IC1.IO_L23N_2; no longer IC1.IO_L6P_0
- net USB_DATA7: now also IC1.IO_L29N_GCLK2_2; no longer IC1.IO_L6N_0
- net USB_DIR: now also IC1.IO_L62P_D5_2; no longer IC1.IO_L7N_0
- net USB_NXT: now also IC1.IO_L13N_D10_2; no longer IC1.IO_L7P_0
- net USB_RESET: now also IC1.IO_L2P_CMPCLK_2; no longer IC1.IO_L1N_VREF_0
- net USB_STP: now also IC1.IO_L2N_CMPMOSI_2; no longer IC1.IO_L33P_0
- net VB0: now also IC1.IO_L49P_D3_2; no longer IC1.IO_L65N_SCP2_0
- net VB1: now also IC1.IO_L64N_D9_2; no longer IC1.IO_L66P_SCP1_0
- net VB2: now also IC1.IO_L49N_D4_2; no longer IC1.IO_L66N_SCP0_0
- net VB3: now also IC1.IO_L64P_D8_2; no longer IC1.IO_L34P_GCLK19_0
- net VB4: now also IC1.IO_L47P_2; no longer IC1.IO_L34N_GCLK18_0
- net VG0: now also IC1.IO_L48N_RDWR_B_VREF_2; no longer IC1.IO_L63P_SCP7_0
- net VG1: now also IC1.IO_L47N_2; no longer IC1.IO_L63N_SCP6_0
- net VG2: now also IC1.IO_L30P_GCLK1_D13_2; no longer IC1.IO_L64P_SCP5_0
- net VG3: now also IC1.IO_L48P_D7_2; no longer IC1.IO_L64N_SCP4_0
- net VG4: now also IC1.IO_L32P_GCLK29_2; no longer IC1.IO_L65P_SCP3_0
- net VR0: now also IC1.IO_L30N_GCLK0_USERCCLK_2; no longer IC1.IO_L39N_0
- net VR1: now also IC1.IO_L31P_GCLK31_D14_2; no longer IC1.IO_L40P_0
- net VR2: now also IC1.IO_L32N_GCLK28_2; no longer IC1.IO_L40N_0
- net VR3: now also IC1.IO_L31N_GCLK30_D15_2; no longer IC1.IO_L62P_0
- net VR4: now also IC1.IO_L62N_D6_2; no longer IC1.IO_L62N_VREF_0
- net VREF_DDR1: now also IC1.IO_L1N_A24_VREF_1, IC1.IO_L53N_VREF_1; no longer C32.1, IC1.IO_L1N_VREF_3, IC1.IO_L83N_VREF_3
- net VREF_DDR3: now also IC1.IO_L1N_VREF_3, IC1.IO_L83N_VREF_3; no longer C31.1, IC1.IO_L1N_A24_VREF_1, IC1.IO_L53N_VREF_1
- net VSYNC: now also IC1.IO_L63P_2; no longer IC1.IO_L37N_GCLK12_0
Other:
- moved on the sheet: C1, C2, C20, C21, C34, C35, C36, C37, C38, C39, C40, C41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

Commit message: Initial coven boards: A13 v0.1 card and test socket
Parts:
- R12, R13, R14: value 3.9k -> 4.02k
- R15, R16, R17: value 8.2k -> 8.06k
- R26: value 10k DNP -> 10k
- R27: value 10k DNP -> DNP(10k)
- R28: value 2.4k -> 10k
- R3, R4, R5: value 510 -> 499
- U$14: value MCP1700-2502 -> MCP1700T-2502

Commit message: Got the VGA board up and running!
The resistors had gotten mixed up due to pinswapping,
so fixed that up in the schematic.

Copied the code from v0.2, updated the ucf, and it works!
Parts:
- R10, R9: value 2k -> 8.06k
- R11: value 2k -> 4.02k
- R12, R13: value 4.02k -> 2k
- R14: value 4.02k -> 1k
- R15, R16: value 8.06k -> 499
- R3, R4: value 499 -> 4.02k
- R5: value 499 -> 2k
- R8: value 1k -> 499
Connections:
- net VB0: now also IC1.IO_L49N_D4_2, R9.1; no longer IC1.IO_L49P_D3_2, R15.1
- net VB1: now also IC1.IO_L47P_2, R3.1; no longer IC1.IO_L64N_D9_2, R12.1
- net VB2: now also IC1.IO_L64N_D9_2, R12.1; no longer IC1.IO_L49N_D4_2, R9.1
- net VB4: now also IC1.IO_L49P_D3_2, R15.1; no longer IC1.IO_L47P_2, R3.1
- net VG0: now also IC1.IO_L30P_GCLK1_D13_2, R10.1; no longer IC1.IO_L48N_RDWR_B_VREF_2, R16.1
- net VG1: now also IC1.IO_L32P_GCLK29_2, R4.1; no longer IC1.IO_L47N_2, R13.1
- net VG2: now also IC1.IO_L47N_2, R13.1; no longer IC1.IO_L30P_GCLK1_D13_2, R10.1
- net VG4: now also IC1.IO_L48N_RDWR_B_VREF_2, R16.1; no longer IC1.IO_L32P_GCLK29_2, R4.1
- net VR1: now also IC1.IO_L32N_GCLK28_2, R11.1; no longer IC1.IO_L31P_GCLK31_D14_2, R14.1
- net VR2: now also IC1.IO_L62N_D6_2, R5.1; no longer IC1.IO_L32N_GCLK28_2, R11.1
- net VR3: now also IC1.IO_L31P_GCLK31_D14_2, R14.1; no longer IC1.IO_L31N_GCLK30_D15_2, R8.1
- net VR4: now also IC1.IO_L31N_GCLK30_D15_2, R8.1; no longer IC1.IO_L62N_D6_2, R5.1
Other:
- moved on the sheet: R10, R12, R13, R14, R15, R16, R17, R3, R4, R5, R6, R7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
