File: modboard/pwrboard_v1.1/board.sch (EAGLE design)
At the start: 36 parts, among them J2 POWER_JACKPTH, Q1 IRFML8244

Commit message: man made a number of mistakes
Parts:
- C7: value 10uF -> 22uF
- L3: value NR5040T4R7N -> NR6028T4R7M
- R6: value 6.7k -> 6.8k
Changed lines of the file:
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@@
 <part name="GND8" library="kmod-nonparts" deviceset="GND" device=""/>
 <part name="C6" library="kmod-passives" deviceset="CAP" device="0805" value="10uF"/>
-<part name="C7" library="kmod-passives" deviceset="CAP" device="0805" value="10uF"/>
+<part name="C7" library="kmod-passives" deviceset="CAP" device="0805" value="22uF"/>
 <part name="SUPPLY7" library="kmod-nonparts" deviceset="1.8V" device=""/>
 <part name="U$9" library="kmod-ics" deviceset="VREG" device="SOT223" value="NCP1117"/>
@@
 <part name="SB1" library="kmod-nonparts" deviceset="SOLDER-BRIDGE" device="0603" value="12V_CS"/>
 <part name="Q1" library="SparkFun-DiscreteSemi" deviceset="MOSFET-NCHANNEL" device="BSS138" value="IRFML8244"/>
-<part name="R6" library="kmod-passives" deviceset="RESISTOR" device="0603" value="6.7k"/>
+<part name="R6" library="kmod-passives" deviceset="RESISTOR" device="0603" value="6.8k"/>
 <part name="L2" library="kmod-passives" deviceset="LED" device="0603" value="RED"/>
 <part name="D1" library="SparkFun-DiscreteSemi" deviceset="DIODE" device="SOD" value="1N4148"/>
@@
 <part name="GND28" library="kmod-nonparts" deviceset="GND" device=""/>
 <part name="C49" library="kmod-passives" deviceset="CAP" device="0402-CAP" value="5pF-100pF;optional"/>
-<part name="L3" library="kmod-passives" deviceset="INDUCTOR" device="NR60XX" value="NR5040T4R7N"/>
+<part name="L3" library="kmod-passives" deviceset="INDUCTOR" device="NR60XX" value="NR6028T4R7M"/>
 <part name="R18" library="kmod-passives" deviceset="RESISTOR" device="0603" value="33k 1%"/>
 <part name="R19" library="kmod-passives" deviceset="RESISTOR" device="0603" value="10k 1%"/>
